File: ll-tester.brd (EAGLE design)
At the start: 120.6 x 145.7 mm, 97 parts, among them IC1 BMA490L, IC2 TCAN330GD, IC4 CAT4238TD-GT3, U1 PIC32MK0512MCJ048T-I/Y8XTQFP4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, U2 MAX6126B30

Commit message: up
Parts:
- added C24, C25, C26, C27: 0.1uf, rcl:C0805
- added LS1: CMI-9705-0380-SMT-TR, CMI-9705-0380-SMT-TR:CMI97050380SMTTR
- moved C20 35.6 mm to (44.5, 20.3)
- moved C21 35.6 mm to (49.5, 20.3)
- moved C19 35.6 mm to (39.4, 20.3)
- moved C22 33.0 mm to (54.6, 20.3)
- moved 3.3VDC 31.9 mm to (45.7, 27.9)
Connections:
- net PWM1EN: now also C24.1
- net PWM1ER: now also C25.1
- net PWM1L: now also LS1.1
- net PWM4H: now also C27.1
- net PWM4L: now also C26.1
- net VSS: now also C24.2, C25.2, C26.2, C27.2, LS1.2
Routing:
- net VSS: track 303.8 -> 237.1 mm, vias 8 -> 15
- net PWM1L: track 22.5 -> 79.3 mm, vias 0 -> 1
- net VDD: track 578.2 -> 612.8 mm, vias 6 -> 4
- net SDI2: track 21.2 -> 52.3 mm
- net SDO1: track 227.0 -> 195.9 mm, vias 2 -> 3
- net SCK1: track 212.5 -> 237.1 mm
- net PGC_C1RX: track 123.6 -> 103.4 mm, vias 2 -> 3
- net DIS_RESET: track 196.1 -> 209.6 mm, vias 3 -> 2
- net QEB2: track 90.0 -> 103.2 mm, vias 4 -> 2
- net EXT_INT2: track 14.8 -> 27.8 mm
- net PWM4H: track 69.4 -> 81.9 mm, vias 0 -> 1
- net N$3: track 37.4 -> 24.9 mm
- net DIS_CS: track 184.0 -> 171.9 mm, vias 2 -> 3
- net MCLR_SIG: track 64.2 -> 75.8 mm
- net PWM4L: track 110.3 -> 99.3 mm, vias 1 -> 2
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
Commit message: up
Parts:
- added SV3: MISC0, con-lstb:MA10-1
Connections:
- net AN0: now also SV3.2
- net AN1: now also SV3.3
- net DAC1: now also SV3.4
- net EXT_SW2: now also SV3.9
- net INDX2: now also SV3.7
- net PWM4EN: now also SV3.6
- net PWM4ER: now also SV3.8
- net VDD: now also SV3.10
- net VSS: now also SV3.1
Routing:
- net VDD: track 612.8 -> 865.1 mm, vias 4 -> 13
- net PWM1ER: track 115.0 -> 339.7 mm, vias 1 -> 0
- net DAC1: track 0.00 -> 190.0 mm
- net N$66: track 54.7 -> 166.6 mm, vias 3 -> 0
- net DIS_MODE: track 188.6 -> 295.3 mm, vias 3 -> 4
- net QEA2: track 65.6 -> 165.0 mm, vias 1 -> 0
- net PWM4EN: track 0.00 -> 94.7 mm
- net INDX2: track 0.00 -> 89.3 mm
- net VSS: track 237.1 -> 320.6 mm, vias 15 -> 20
- net AN0: track 0.00 -> 73.2 mm, vias 0 -> 2
- net AN1: track 0.00 -> 60.0 mm, vias 0 -> 2
- net PWM4ER: track 0.00 -> 58.1 mm, vias 0 -> 1
- net MCLR_SIG: track 75.8 -> 126.2 mm, vias 1 -> 2
- net EXT_SW2: track 0.00 -> 48.8 mm, vias 0 -> 1
- net DIS_CS: track 171.9 -> 219.2 mm
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
Commit message: up
Routing:
- net VDD: track 865.1 -> 592.9 mm, vias 13 -> 5
- net PWM1ER: track 339.7 -> 120.1 mm, vias 0 -> 2
- net N$66: track 166.6 -> 54.2 mm, vias 0 -> 1
- net DAC1: track 190.0 -> 86.9 mm, vias 0 -> 2
- net QEA2: track 165.0 -> 84.9 mm, vias 0 -> 2
- net VSS: track 320.6 -> 253.1 mm, vias 20 -> 16
- net DIS_MODE: track 295.3 -> 232.5 mm, vias 4 -> 2
- net MCLR_SIG: track 126.2 -> 82.7 mm, vias 2 -> 1
- net PWM4EN: track 94.7 -> 62.3 mm, vias 0 -> 1
- net SDI2: track 58.9 -> 27.1 mm
- net RED_LED: track 61.0 -> 30.7 mm, vias 2 -> 3
- net EXT_INT2: track 47.9 -> 19.5 mm
- net INDX2: track 89.3 -> 60.9 mm, vias 0 -> 1
- net QEB2: track 103.8 -> 79.2 mm, vias 2 -> 3
- net PWM4H: track 107.3 -> 82.8 mm, vias 2 -> 1
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
Commit message: up
Parts:
- removed SV4, SV5: ETHG, con-lstb:MA03-1
- added C28: 0.1uf, rcl:C0805
- added C29: 10uf, rcl:C0805
- added I/O_MON: IOMON, con-lstb:MA10-1
- added IC3: EM14R0D-R20-L064S, EM14R0D-R20-L064S:EM14R0DR20L064S
- moved LS1 14.0 mm to (45.7, 43.2)
Connections:
- net PWM1EN renamed RD8
- net PWM1ER renamed RB8
- net PWM1L renamed RB15
- net PWM4EN renamed RB11
- net PWM4L renamed RA7
- removed net PWM1H: SV1.1, U1.2
- removed net PWM4ER: SV3.8, U1.23
- removed net PWM4H: C27.1, S5.2, U1.48
- new net RA10: C27.1, IC3.2, S5.2, U1.48
- new net U2RX: I/O_MON.6, SV3.8, U1.23
- new net U2TX: I/O_MON.7, SV1.1, U1.2
- net AN0: now also I/O_MON.9
- net AN1: now also I/O_MON.10
- net MCLR_SIG: now also SV3.5
- net QEA2: now also IC3.A1
- net QEB2: now also IC3.B1
- net U1RX: now also I/O_MON.2
- net U1TX: now also I/O_MON.3
- net VDD: now also C28.1, C29.1, I/O_MON.4, I/O_MON.8, IC3.3
- net VSS: now also C28.2, C29.2, I/O_MON.1, I/O_MON.5, IC3.1, IC3.4, IC3.MH1, IC3.MH2; no longer SV4.1, SV4.2, SV4.3, SV5.1, SV5.2, SV5.3
Routing:
- net U2RX: track 0.00 -> 91.3 mm, vias 0 -> 1
- net RA10: track 0.00 -> 91.3 mm, vias 0 -> 1
- net PWM4H: track 82.8 -> 0.00 mm, vias 1 -> 0
- net U2TX: track 0.00 -> 81.0 mm
- net QEB2: track 79.2 -> 136.3 mm, vias 3 -> 2
- net PWM4ER: track 56.3 -> 0.00 mm, vias 1 -> 0
- net U1RX: track 53.9 -> 106.8 mm, vias 1 -> 2
- net VDD: track 592.9 -> 639.9 mm, vias 5 -> 12
- net MCLR_SIG: track 82.7 -> 126.0 mm, vias 1 -> 4
- net VSS: track 253.1 -> 296.0 mm, vias 16 -> 13
- net SDO1: track 201.9 -> 238.1 mm, vias 3 -> 2
- net AN1: track 60.4 -> 95.1 mm, vias 1 -> 0
- net U1TX: track 48.6 -> 83.2 mm, vias 1 -> 2
- net RA7: track 102.0 -> 125.9 mm, vias 2 -> 1
- net PWM1H: track 23.1 -> 0.00 mm
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
Commit message: up
Parts:
- moved LS1 6.35 mm to (45.7, 49.5)
Routing:
- net VDD: track 639.9 -> 667.8 mm, vias 12 -> 11
- net VSS: track 296.0 -> 276.9 mm, vias 13 -> 14
- net AN1: track 95.1 -> 80.3 mm, vias 0 -> 1
- net QEA2: track 100.6 -> 114.8 mm, vias 1 -> 0
- net BMA_INT2: track 40.5 -> 26.9 mm, vias 1 -> 2
- net SDO1: track 238.1 -> 227.3 mm
- net SCK1: track 209.6 -> 220.2 mm, vias 4 -> 3
- net RB11: track 68.3 -> 58.2 mm, vias 0 -> 2
- net DIS_RESET: track 218.0 -> 209.0 mm, vias 2 -> 3
- net DAC1: track 92.2 -> 83.5 mm, vias 2 -> 0
- net U2TX: track 81.0 -> 72.8 mm, vias 0 -> 2
- net IMU_CS: track 35.1 -> 27.5 mm, vias 2 -> 3
- net RD8: track 125.1 -> 117.5 mm, vias 1 -> 2
- net CAN_P: track 58.9 -> 65.3 mm
- net DIS_MODE: track 240.1 -> 246.5 mm, vias 3 -> 2
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
Commit message: up
Parts:
- added R7: 10k, rcl:M0805
Connections:
- net RB8: now also R7.1
- net VDD: now also R7.2
Routing:
- net VDD: track 667.8 -> 710.0 mm
- net RB8: track 117.2 -> 121.8 mm
Other:
- board text added: "PIC32MK-CANFD HID V1.0"
- board text removed: "PIC32MK-CANFD HOST V1.7"
Changed lines of the file:
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@@
 <wire x1="62.21" y1="163.5" x2="-58.42" y2="163.5" width="0" layer="20"/>
 <wire x1="-58.42" y1="163.5" x2="-58.42" y2="162.23" width="0" layer="20"/>
-<text x="21.59" y="20.32" size="1.016" layer="1" font="vector" ratio="17" distance="77" rot="R180">PIC32MK-CANFD HOST V1.7</text>
+<text x="21.59" y="20.32" size="1.016" layer="1" font="vector" ratio="17" distance="77" rot="R180">PIC32MK-CANFD HID V1.0</text>
 <hole x="-55.88" y="20.32" drill="2.54"/>
 <hole x="-55.88" y="58.42" drill="2.54"/>
@@
 <attribute name="VALUE" x="-43.18" y="59.69" size="1.27" layer="27"/>
 </element>
+<element name="R7" library="rcl" library_urn="urn:adsk.eagle:library:334" package="M0805" package3d_urn="urn:adsk.eagle:package:23556/2" value="10k" x="-45.72" y="123.19" smashed="yes" rot="MR180">
+<attribute name="NAME" x="-46.99" y="121.92" size="1.27" layer="26" rot="MR180"/>
+<attribute name="POPULARITY" value="45" x="-45.72" y="123.19" size="1.778" layer="28" rot="MR180" display="off"/>
+<attribute name="SPICEPREFIX" value="R" x="-45.72" y="123.19" size="1.778" layer="28" rot="MR180" display="off"/>
+<attribute name="VALUE" x="-46.99" y="125.73" size="1.27" layer="28" rot="MR180"/>
+</element>
 </elements>
 <signals>
@@
 <via x="12.0396" y="25.146" extent="1-16" drill="0.35"/>
 <via x="40.3098" y="21.6408" extent="1-16" drill="0.35"/>
+<contactref element="R7" pad="2"/>
+<wire x1="-44.7294" y1="123.444" x2="-44.7294" y2="123.2154" width="0.3048" layer="16"/>
+<wire x1="-24.9174" y1="143.256" x2="-44.7294" y2="123.444" width="0.3048" layer="16"/>
+<wire x1="-12.4206" y1="143.256" x2="-24.9174" y2="143.256" width="0.3048" layer="16"/>
+<wire x1="-11.43" y1="142.2654" x2="-12.4206" y2="143.256" width="0.3048" layer="16"/>
+<wire x1="-44.7294" y1="123.2154" x2="-44.77" y2="123.19" width="0.3048" layer="16"/>
+<wire x1="-11.43" y1="142.2654" x2="-11.43" y2="142.24" width="0.3048" layer="16"/>
 </signal>
 <signal name="VSS" class="2">
@@
 <contactref element="C25" pad="1"/>
 <wire x1="-43.5102" y1="113.4618" x2="-43.5102" y2="110.49" width="0.1524" layer="16"/>
-<wire x1="-53.34" y1="123.2916" x2="-43.5102" y2="113.4618" width="0.1524" layer="16"/>
+<wire x1="-53.34" y1="123.2916" x2="-49.9491" y2="119.9007" width="0.1524" layer="16"/>
+<wire x1="-49.9491" y1="119.9007" x2="-43.5102" y2="113.4618" width="0.1524" layer="16"/>
 <wire x1="-43.5102" y1="110.49" x2="-43.5" y2="110.49" width="0.1524" layer="16"/>
 <wire x1="-53.34" y1="123.2916" x2="-53.34" y2="123.34" width="0.1524" layer="16"/>
@@
 <wire x1="23.3934" y1="44.7294" x2="23.3299" y2="44.66" width="0.1524" layer="1"/>
 <via x="23.8506" y="53.8734" extent="1-16" drill="0.35"/>
+<contactref element="R7" pad="1"/>
+<wire x1="-49.9491" y1="119.9007" x2="-46.7106" y2="123.1392" width="0.1524" layer="16"/>
+<wire x1="-46.7106" y1="123.1392" x2="-46.67" y2="123.19" width="0.1524" layer="16"/>
 </signal>
 <signal name="RB11">

Commit message: up
Connections:
- net INDX2: now also SJ5.3
- net QEB2: no longer SJ5.3
Routing:
- net INDX2: track 49.8 -> 76.4 mm, vias 2 -> 4
- net QEB2: track 135.5 -> 129.1 mm
Changed lines of the file:
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@@
 <contactref element="U1" pad="47"/>
 <contactref element="SV2" pad="10"/>
-<contactref element="SJ5" pad="3"/>
 <contactref element="IC3" pad="B1"/>
 <wire x1="16.8402" y1="49.8348" x2="16.8402" y2="46.2534" width="0.1524" layer="1"/>
 <wire x1="17.3736" y1="50.3682" x2="16.8402" y2="49.8348" width="0.1524" layer="1"/>
-<wire x1="17.3736" y1="53.0352" x2="17.3736" y2="50.3682" width="0.1524" layer="15"/>
-<wire x1="24.4602" y1="60.1218" x2="17.3736" y2="53.0352" width="0.1524" layer="15"/>
-<wire x1="24.4602" y1="63.3222" x2="24.4602" y2="60.1218" width="0.1524" layer="1"/>
-<wire x1="28.194" y1="67.056" x2="24.4602" y2="63.3222" width="0.1524" layer="1"/>
-<wire x1="28.194" y1="67.31" x2="28.194" y2="67.056" width="0.1524" layer="1"/>
 <wire x1="16.8402" y1="46.2534" x2="16.8" y2="46.1899" width="0.1524" layer="1"/>
-<wire x1="42.291" y1="66.9036" x2="46.9392" y2="62.2554" width="0.1524" layer="1"/>
-<wire x1="28.1178" y1="66.9036" x2="42.291" y2="66.9036" width="0.1524" layer="1"/>
-<wire x1="46.9392" y1="62.2554" x2="46.99" y2="62.23" width="0.1524" layer="1"/>
-<wire x1="28.1178" y1="66.9036" x2="28.194" y2="67.31" width="0.1524" layer="1"/>
 <wire x1="3.2004" y1="21.6408" x2="-24.0792" y2="21.6408" width="0.1524" layer="15"/>
 <wire x1="21.6408" y1="40.0812" x2="3.2004" y2="21.6408" width="0.1524" layer="15"/>
@@
 <wire x1="46.9392" y1="62.1792" x2="46.99" y2="62.23" width="0.1524" layer="15"/>
 <via x="17.3736" y="50.3682" extent="1-16" drill="0.35"/>
-<via x="24.4602" y="60.1218" extent="1-16" drill="0.35"/>
+<wire x1="17.3736" y1="52.1208" x2="17.3736" y2="50.3682" width="0.1524" layer="15"/>
+<wire x1="23.5458" y1="58.293" x2="17.3736" y2="52.1208" width="0.1524" layer="15"/>
+<via x="23.5458" y="58.293" extent="1-16" drill="0.35"/>
+<wire x1="26.8986" y1="58.293" x2="23.5458" y2="58.293" width="0.1524" layer="1"/>
+<wire x1="31.6992" y1="63.0936" x2="26.8986" y2="58.293" width="0.1524" layer="1"/>
+<wire x1="46.0248" y1="63.0936" x2="31.6992" y2="63.0936" width="0.1524" layer="1"/>
+<wire x1="46.863" y1="62.2554" x2="46.0248" y2="63.0936" width="0.1524" layer="1"/>
+<wire x1="46.863" y1="62.2554" x2="46.99" y2="62.23" width="0.1524" layer="1"/>
 </signal>
 <signal name="INDX2">
@@
 <wire x1="17.0688" y1="45.1866" x2="17.2974" y2="45.4152" width="0.1524" layer="1"/>
 <wire x1="16.002" y1="45.1866" x2="17.0688" y2="45.1866" width="0.1524" layer="1"/>
-<wire x1="14.9352" y1="46.2534" x2="16.002" y2="45.1866" width="0.1524" layer="1"/>
+<wire x1="14.9352" y1="46.2534" x2="14.9733" y2="46.2153" width="0.1524" layer="1"/>
+<wire x1="14.9733" y1="46.2153" x2="16.002" y2="45.1866" width="0.1524" layer="1"/>
 <wire x1="11.1252" y1="46.2534" x2="14.9352" y2="46.2534" width="0.1524" layer="1"/>
 <wire x1="-1.905" y1="46.2534" x2="11.1252" y2="46.2534" width="0.1524" layer="15"/>
@@
 <via x="11.1252" y="46.2534" extent="1-16" drill="0.35"/>
 <via x="-2.2098" y="46.5582" extent="1-16" drill="0.35"/>
+<contactref element="SJ5" pad="3"/>
+<wire x1="28.0416" y1="67.2846" x2="28.194" y2="67.2846" width="0.1524" layer="1"/>
+<wire x1="27.5082" y1="66.7512" x2="28.0416" y2="67.2846" width="0.1524" layer="1"/>
+<wire x1="27.5082" y1="65.3034" x2="27.5082" y2="66.7512" width="0.1524" layer="1"/>
+<wire x1="22.5552" y1="60.3504" x2="27.5082" y2="65.3034" width="0.1524" layer="1"/>
+<wire x1="22.5552" y1="57.7596" x2="22.5552" y2="60.3504" width="0.1524" layer="15"/>
+<wire x1="15.3924" y1="50.5968" x2="22.5552" y2="57.7596" width="0.1524" layer="15"/>
+<wire x1="15.3924" y1="49.6062" x2="15.3924" y2="50.5968" width="0.1524" layer="1"/>
+<wire x1="15.0114" y1="49.2252" x2="15.3924" y2="49.6062" width="0.1524" layer="1"/>
+<wire x1="15.0114" y1="46.2534" x2="15.0114" y2="49.2252" width="0.1524" layer="1"/>
+<wire x1="28.194" y1="67.2846" x2="28.194" y2="67.31" width="0.1524" layer="1"/>
+<wire x1="15.0114" y1="46.2534" x2="14.9733" y2="46.2153" width="0.1524" layer="1"/>
+<via x="22.5552" y="60.3504" extent="1-16" drill="0.35"/>
+<via x="15.3924" y="50.5968" extent="1-16" drill="0.35"/>
 </signal>
 <signal name="RB15">

Commit message: up
Parts:
- moved 3.3VDC 14.0 mm to (45.7, 41.9)
Routing:
- net DC_INPUT: track 29.5 -> 40.4 mm, vias 0 -> 2
- net VDD: track 710.0 -> 716.4 mm
Changed lines of the file:
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@@
 <attribute name="VALUE" x="-2.54" y="25.4" size="1.27" layer="27"/>
 </element>
-<element name="3.3VDC" library="linear" library_urn="urn:adsk.eagle:library:262" package="TO220V" package3d_urn="urn:adsk.eagle:package:16417/2" value="3.3 Vreg" x="45.72" y="27.94" smashed="yes">
-<attribute name="NAME" x="44.45" y="21.8948" size="1.27" layer="25" ratio="10"/>
-<attribute name="POPULARITY" value="57" x="45.72" y="27.94" size="1.778" layer="27" display="off"/>
-<attribute name="VALUE" x="40.64" y="20.32" size="1.27" layer="27" ratio="10"/>
+<element name="3.3VDC" library="linear" library_urn="urn:adsk.eagle:library:262" package="TO220V" package3d_urn="urn:adsk.eagle:package:16417/2" value="3.3 Vreg" x="45.72" y="41.91" smashed="yes">
+<attribute name="NAME" x="44.45" y="35.8648" size="1.27" layer="25" ratio="10"/>
+<attribute name="POPULARITY" value="57" x="45.72" y="41.91" size="1.778" layer="27" display="off"/>
+<attribute name="VALUE" x="40.64" y="34.29" size="1.27" layer="27" ratio="10"/>
 </element>
 <element name="C19" library="rcl" library_urn="urn:adsk.eagle:library:334" package="C0805" package3d_urn="urn:adsk.eagle:package:23617/2" value="0.1uf" x="39.37" y="20.32" smashed="yes" rot="MR0">
@@
 <wire x1="5.7912" y1="25.146" x2="5.715" y2="25.0698" width="0.3048" layer="1"/>
 <wire x1="31.4706" y1="23.5458" x2="28.2702" y2="20.3454" width="0.3048" layer="1"/>
-<wire x1="46.4058" y1="23.5458" x2="40.3098" y2="23.5458" width="0.3048" layer="1"/>
 <wire x1="40.3098" y1="23.5458" x2="31.4706" y2="23.5458" width="0.3048" layer="1"/>
-<wire x1="48.26" y1="25.4" x2="46.4058" y2="23.5458" width="0.3048" layer="1"/>
 <wire x1="28.2702" y1="20.3454" x2="28.26" y2="20.32" width="0.3048" layer="1"/>
 <wire x1="40.3098" y1="21.6408" x2="40.3098" y2="20.3454" width="0.3048" layer="16"/>
@@
 <wire x1="52.8828" y1="19.2024" x2="54.483" y2="19.2024" width="0.3048" layer="16"/>
 <wire x1="51.435" y1="20.6502" x2="52.8828" y2="19.2024" width="0.3048" layer="16"/>
-<wire x1="51.435" y1="22.2504" x2="51.435" y2="20.6502" width="0.3048" layer="16"/>
-<wire x1="48.3108" y1="25.3746" x2="51.435" y2="22.2504" width="0.3048" layer="16"/>
 <wire x1="55.5498" y1="20.2692" x2="55.56" y2="20.32" width="0.3048" layer="16"/>
-<wire x1="48.3108" y1="25.3746" x2="48.26" y2="25.4" width="0.3048" layer="16"/>
 <wire x1="45.72" y1="49.53" x2="45.72" y2="62.23" width="0.3048" layer="16"/>
-<wire x1="57.15" y1="38.1" x2="45.72" y2="49.53" width="0.3048" layer="16"/>
-<wire x1="48.3108" y1="29.2608" x2="48.3108" y2="25.527" width="0.3048" layer="1"/>
-<wire x1="57.15" y1="38.1" x2="48.3108" y2="29.2608" width="0.3048" layer="1"/>
-<wire x1="48.3108" y1="25.527" x2="48.26" y2="25.4" width="0.3048" layer="1"/>
+<wire x1="57.15" y1="38.1" x2="52.0827" y2="43.1673" width="0.3048" layer="16"/>
+<wire x1="52.0827" y1="43.1673" x2="45.72" y2="49.53" width="0.3048" layer="16"/>
 <wire x1="29.718" y1="30.7086" x2="21.717" y2="30.7086" width="0.3048" layer="16"/>
 <wire x1="38.7096" y1="21.717" x2="29.718" y2="30.7086" width="0.3048" layer="16"/>
@@
 <wire x1="-44.7294" y1="123.2154" x2="-44.77" y2="123.19" width="0.3048" layer="16"/>
 <wire x1="-11.43" y1="142.2654" x2="-11.43" y2="142.24" width="0.3048" layer="16"/>
+<wire x1="52.0827" y1="43.1673" x2="48.3108" y2="39.3954" width="0.3048" layer="16"/>
+<wire x1="48.3108" y1="39.3954" x2="48.26" y2="39.37" width="0.3048" layer="16"/>
+<wire x1="51.435" y1="21.2598" x2="51.435" y2="20.6502" width="0.3048" layer="16"/>
+<wire x1="50.673" y1="22.0218" x2="51.435" y2="21.2598" width="0.3048" layer="16"/>
+<wire x1="40.6908" y1="22.0218" x2="50.673" y2="22.0218" width="0.3048" layer="16"/>
+<wire x1="40.3098" y1="21.6408" x2="40.6908" y2="22.0218" width="0.3048" layer="16"/>
+<wire x1="57.2262" y1="37.7952" x2="57.2262" y2="38.0238" width="0.3048" layer="16"/>
+<wire x1="58.9788" y1="36.0426" x2="57.2262" y2="37.7952" width="0.3048" layer="16"/>
+<wire x1="58.9788" y1="23.622" x2="58.9788" y2="36.0426" width="0.3048" layer="16"/>
+<wire x1="55.7022" y1="20.3454" x2="58.9788" y2="23.622" width="0.3048" layer="16"/>
+<wire x1="57.2262" y1="38.0238" x2="57.15" y2="38.1" width="0.3048" layer="16"/>
+<wire x1="55.7022" y1="20.3454" x2="55.56" y2="20.32" width="0.3048" layer="16"/>
 </signal>
 <signal name="VSS" class="2">
@@
 <wire x1="26.67" y1="24.13" x2="26.67" y2="20.0406" width="0.3048" layer="1"/>
 <wire x1="30.099" y1="20.2692" x2="30.16" y2="20.32" width="0.3048" layer="1"/>
-<wire x1="48.5394" y1="22.5552" x2="48.5394" y2="20.3454" width="0.3048" layer="16"/>
-<wire x1="45.72" y1="25.3746" x2="48.5394" y2="22.5552" width="0.3048" layer="16"/>
 <wire x1="48.5394" y1="20.3454" x2="48.58" y2="20.32" width="0.3048" layer="16"/>
-<wire x1="45.72" y1="25.3746" x2="45.72" y2="25.4" width="0.3048" layer="16"/>
 <wire x1="53.721" y1="20.6502" x2="53.721" y2="20.3454" width="0.3048" layer="16"/>
 <wire x1="57.15" y1="24.0792" x2="53.721" y2="20.6502" width="0.3048" layer="16"/>
@@
 <via x="-1.6764" y="29.2608" extent="1-16" drill="0.35"/>
 <via x="13.4112" y="42.672" extent="1-16" drill="0.35"/>
+<wire x1="48.1584" y1="20.3454" x2="48.387" y2="20.3454" width="0.3048" layer="16"/>
+<wire x1="46.9392" y1="21.5646" x2="48.1584" y2="20.3454" width="0.3048" layer="16"/>
+<wire x1="44.7294" y1="21.5646" x2="46.9392" y2="21.5646" width="0.3048" layer="16"/>
+<wire x1="43.5864" y1="20.4216" x2="44.7294" y2="21.5646" width="0.3048" layer="16"/>
+<wire x1="48.387" y1="20.3454" x2="48.58" y2="20.32" width="0.3048" layer="16"/>
+<wire x1="43.5864" y1="20.4216" x2="43.5" y2="20.32" width="0.3048" layer="16"/>
 </signal>
 <signal name="AVDD" class="2">
@@
 <contactref element="C21" pad="1"/>
 <contactref element="R6" pad="1"/>
-<wire x1="45.339" y1="23.241" x2="45.339" y2="20.3454" width="0.3048" layer="16"/>
-<wire x1="43.18" y1="25.4" x2="45.339" y2="23.241" width="0.3048" layer="16"/>
 <wire x1="45.339" y1="20.3454" x2="45.4" y2="20.32" width="0.3048" layer="16"/>
 <wire x1="49.3776" y1="19.2024" x2="50.4444" y2="20.2692" width="0.3048" layer="16"/>
@@
 <wire x1="50.4444" y1="20.2692" x2="50.48" y2="20.32" width="0.3048" layer="16"/>
 <wire x1="45.4914" y1="20.193" x2="45.4" y2="20.32" width="0.3048" layer="16"/>
-<wire x1="32.9946" y1="32.6136" x2="32.9946" y2="33.147" width="0.3048" layer="16"/>
-<wire x1="31.6992" y1="31.3182" x2="32.9946" y2="32.6136" width="0.3048" layer="16"/>
-<wire x1="31.6992" y1="29.4132" x2="31.6992" y2="31.3182" width="0.3048" layer="16"/>
-<wire x1="35.6616" y1="25.4508" x2="31.6992" y2="29.4132" width="0.3048" layer="16"/>
-<wire x1="43.053" y1="25.4508" x2="35.6616" y2="25.4508" width="0.3048" layer="16"/>
-<wire x1="32.9946" y1="33.147" x2="33.02" y2="33.15" width="0.3048" layer="16"/>
-<wire x1="43.053" y1="25.4508" x2="43.18" y2="25.4" width="0.3048" layer="16"/>
+<wire x1="37.719" y1="37.8714" x2="33.0708" y2="33.2232" width="0.3048" layer="16"/>
+<wire x1="41.6814" y1="37.8714" x2="37.719" y2="37.8714" width="0.3048" layer="15"/>
+<wire x1="43.18" y1="39.37" x2="41.6814" y2="37.8714" width="0.3048" layer="15"/>
+<wire x1="33.0708" y1="33.2232" x2="33.02" y2="33.15" width="0.3048" layer="16"/>
+<wire x1="46.6344" y1="20.8788" x2="45.7962" y2="20.0406" width="0.3048" layer="16"/>
+<wire x1="46.6344" y1="35.8902" x2="46.6344" y2="20.8788" width="0.3048" layer="1"/>
+<wire x1="43.2054" y1="39.3192" x2="46.6344" y2="35.8902" width="0.3048" layer="1"/>
+<wire x1="45.7962" y1="20.0406" x2="45.4" y2="20.32" width="0.3048" layer="16"/>
+<wire x1="43.2054" y1="39.3192" x2="43.18" y2="39.37" width="0.3048" layer="1"/>
+<via x="37.719" y="37.8714" extent="1-16" drill="0.35"/>
+<via x="46.6344" y="20.8788" extent="1-16" drill="0.35"/>
 </signal>
 <signal name="DC_IN" class="1">
