File: ll-tester.brd (EAGLE design)
At the start: 120.6 x 145.7 mm, 106 parts, among them IC1 BMA490L, IC2 TCAN330GD, IC3 EM14R0D-R20-L064S, IC4 CAT4238TD-GT3, U1 PIC32MK0512MCJ048T-I/Y8XTQFP4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, U2 MAX6126B30

Commit message: up
Parts:
- added C30, C31: 0.1uf, rcl:C0805
- added OS2: OSC-OE-IQXO-793, IQD-Frequency-Products:2.5X2-4-PAD
- added U3: BNO080, BNO080:IC_BNO080
Connections:
- new net 32KHZ: OS2.3, U3.27
- new net N$14: C30.1, U3.9
- net BMA_INT2: now also U3.14
- net IMU_CS: now also U3.18
- net SCK2: now also U3.19
- net SDI2: now also U3.20
- net SDO2: now also U3.17
- net VDD: now also C31.1, OS2.1, OS2.4, U3.10, U3.26, U3.28, U3.3
- net VSS: now also C30.2, C31.2, OS2.2, U3.2, U3.25

Commit message: up
Parts:
- added C32: 0.1uf, rcl:C0805
- added OSCI1: PTR1PAD1-13, testpad:P1-13
- added R8, R9: 10k, rcl:M0805
- added SJ3: BOOT_ON, jumper:SJ
- added SJ4: IMU_RESET, jumper:SJ
Connections:
- net RB15 renamed BUZZER1
- removed net BMA_INT2: IC1.6, TP3.TP, U1.11, U3.14
- new net N$16: R8.1, SJ3.2, U3.4
- new net N$17: C32.1, R9.1, SJ4.2, U3.11
- new net TP3_SIG_WAKE: IC1.6, TP3.TP, U1.11, U3.6
- net 32KHZ: now also OSCI1.TP
- net EXT_INT2: now also U3.14
- net VDD: now also R8.2, R9.2, U3.5
- net VSS: now also C32.2, SJ3.1, SJ4.1
Routing:
- net VSS: track 276.8 -> 326.9 mm, vias 14 -> 10
- net TP3_SIG_WAKE: track 0.00 -> 47.6 mm
- net N$17: track 0.00 -> 46.5 mm
- net VDD: track 716.4 -> 755.5 mm, vias 11 -> 10
- net IMU_CS: track 27.5 -> 64.7 mm, vias 3 -> 4
- net QEB2: track 129.1 -> 95.1 mm, vias 2 -> 4
- net SDI2: track 25.0 -> 55.0 mm, vias 3 -> 4
- net BMA_INT2: track 26.9 -> 0.00 mm, vias 2 -> 0
- net DIS_MODE: track 246.5 -> 220.8 mm
- net PGD_C1TX: track 132.8 -> 109.1 mm, vias 1 -> 3
- net SCK2: track 16.8 -> 37.5 mm, vias 1 -> 4
- net U1RX: track 109.7 -> 89.3 mm
- net SDO2: track 12.0 -> 31.9 mm, vias 2 -> 4
- net RA7: track 121.9 -> 103.4 mm, vias 2 -> 4
- net N$14: track 0.00 -> 15.2 mm
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Other:
- board text added: "PIC32MK-CANFD HID V1.1"
- board text removed: "PIC32MK-CANFD HID V1.0"

Commit message: p
Parts:
- added DISP_SIGS: DISP-SIG, pinhead:1X02
- added GLORY: GLORY, pinhead:1X02
- added SJ7: IMU_R_SIG, jumper:SJ
- SV3: value MISC0 -> MISC_SIG
Connections:
- new net MISC_0: DISP_SIGS.1, SJ5.3
- net DIS_RESET: now also DISP_SIGS.2, SJ7.2
- net INDX2: no longer SJ5.3
- net N$17: now also SJ7.1
- net VDD: now also GLORY.1, GLORY.2
Routing:
- net MISC_0: track 0.00 -> 81.7 mm, vias 0 -> 1
- net VDD: track 755.5 -> 768.3 mm
- net DIS_RESET: track 205.7 -> 217.7 mm, vias 2 -> 3
- net N$17: track 46.5 -> 56.7 mm, vias 0 -> 2
- net INDX2: track 78.6 -> 70.9 mm
Changed lines of the file:
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@@
 <attribute name="VALUE" x="45.72" y="49.53" size="1.27" layer="27" align="center"/>
 </element>
-<element name="SV3" library="con-lstb" library_urn="urn:adsk.eagle:library:162" package="MA10-1" package3d_urn="urn:adsk.eagle:package:8346/1" value="MISC0" x="-31.75" y="40.64" smashed="yes">
+<element name="SV3" library="con-lstb" library_urn="urn:adsk.eagle:library:162" package="MA10-1" package3d_urn="urn:adsk.eagle:package:8346/1" value="MISC_SIG" x="-31.75" y="40.64" smashed="yes">
 <attribute name="MF" value="" x="-31.75" y="40.64" size="1.778" layer="27" display="off"/>
 <attribute name="MPN" value="" x="-31.75" y="40.64" size="1.778" layer="27" display="off"/>
@@
 <attribute name="VALUE" x="19.9199" y="57.15" size="0.02" layer="28" rot="MR0"/>
 </element>
+<element name="SJ7" library="jumper" library_urn="urn:adsk.eagle:library:252" package="SJ" package3d_urn="urn:adsk.eagle:package:15471/1" value="IMU_R_SIG" x="26.67" y="72.39" smashed="yes" rot="MR0">
+<attribute name="NAME" x="28.321" y="73.533" size="1.27" layer="26" ratio="10" rot="MR0"/>
+<attribute name="POPULARITY" value="33" x="26.67" y="72.39" size="1.778" layer="28" rot="MR0" display="off"/>
+<attribute name="VALUE" x="26.2699" y="72.39" size="0.02" layer="28" rot="MR0"/>
+</element>
+<element name="DISP_SIGS" library="pinhead" library_urn="urn:adsk.eagle:library:325" package="1X02" package3d_urn="urn:adsk.eagle:package:22435/2" value="DISP-SIG" x="-34.29" y="50.8" smashed="yes">
+<attribute name="NAME" x="-36.9062" y="52.6288" size="1.27" layer="25" ratio="10"/>
+<attribute name="POPULARITY" value="98" x="-34.29" y="50.8" size="1.778" layer="27" display="off"/>
+<attribute name="VALUE" x="-36.83" y="47.625" size="1.27" layer="27"/>
+</element>
+<element name="GLORY" library="pinhead" library_urn="urn:adsk.eagle:library:325" package="1X02" package3d_urn="urn:adsk.eagle:package:22435/2" value="GLORY" x="34.29" y="48.26" smashed="yes">
+<attribute name="NAME" x="31.6738" y="50.0888" size="1.27" layer="25" ratio="10"/>
+<attribute name="POPULARITY" value="98" x="34.29" y="48.26" size="1.778" layer="27" display="off"/>
+<attribute name="VALUE" x="31.75" y="45.085" size="1.27" layer="27"/>
+</element>
 </elements>
 <signals>
@@
 <wire x1="57.15" y1="38.1" x2="58.9788" y2="36.2712" width="0.3048" layer="16"/>
 <wire x1="55.626" y1="20.3454" x2="55.56" y2="20.32" width="0.3048" layer="16"/>
-<wire x1="45.72" y1="41.91" x2="45.72" y2="62.23" width="0.3048" layer="15"/>
+<wire x1="45.72" y1="41.91" x2="45.72" y2="48.3108" width="0.3048" layer="15"/>
+<wire x1="45.72" y1="48.3108" x2="45.72" y2="62.23" width="0.3048" layer="15"/>
 <wire x1="48.26" y1="39.37" x2="45.72" y2="41.91" width="0.3048" layer="15"/>
 <wire x1="49.4538" y1="38.1762" x2="57.0738" y2="38.1762" width="0.3048" layer="16"/>
@@
 <via x="12.0396" y="43.2816" extent="1-16" drill="0.35"/>
 <wire x1="14.7066" y1="42.1386" x2="14.7701" y2="42.16" width="0.3048" layer="1"/>
+<contactref element="GLORY" pad="1"/>
+<contactref element="GLORY" pad="2"/>
+<wire x1="35.5092" y1="48.3108" x2="33.0708" y2="48.3108" width="0.3048" layer="1"/>
+<wire x1="33.0708" y1="48.3108" x2="33.02" y2="48.26" width="0.3048" layer="1"/>
+<wire x1="35.5092" y1="48.3108" x2="35.56" y2="48.26" width="0.3048" layer="1"/>
+<wire x1="45.72" y1="48.3108" x2="35.5854" y2="48.3108" width="0.3048" layer="15"/>
+<wire x1="35.5854" y1="48.3108" x2="35.56" y2="48.26" width="0.3048" layer="15"/>
 </signal>
 <signal name="VSS" class="2">
@@
 <wire x1="17.526" y1="75.2856" x2="-9.8298" y2="102.6414" width="0.1524" layer="15"/>
 <wire x1="17.526" y1="74.9808" x2="17.526" y2="75.2856" width="0.1524" layer="1"/>
-<wire x1="25.146" y1="67.3608" x2="17.526" y2="74.9808" width="0.1524" layer="1"/>
+<wire x1="25.146" y1="67.3608" x2="23.9649" y2="68.5419" width="0.1524" layer="1"/>
+<wire x1="23.9649" y1="68.5419" x2="17.526" y2="74.9808" width="0.1524" layer="1"/>
 <wire x1="-16.4592" y1="142.2654" x2="-16.51" y2="142.24" width="0.1524" layer="15"/>
 <wire x1="25.146" y1="67.3608" x2="25.146" y2="67.31" width="0.1524" layer="1"/>
@@
 <wire x1="-32.004" y1="39.0144" x2="-34.29" y2="36.7284" width="0.1524" layer="15"/>
 <wire x1="-32.004" y1="41.4528" x2="-32.004" y2="39.0144" width="0.1524" layer="1"/>
-<wire x1="-12.4206" y1="61.0362" x2="-32.004" y2="41.4528" width="0.1524" layer="1"/>
+<wire x1="-12.4206" y1="61.0362" x2="-27.8511" y2="45.6057" width="0.1524" layer="1"/>
+<wire x1="-27.8511" y1="45.6057" x2="-32.004" y2="41.4528" width="0.1524" layer="1"/>
 <wire x1="0.9906" y1="61.0362" x2="-12.4206" y2="61.0362" width="0.1524" layer="1"/>
 <wire x1="2.4384" y1="62.484" x2="0.9906" y2="61.0362" width="0.1524" layer="1"/>
@@
 <via x="17.526" y="75.2856" extent="1-16" drill="0.35"/>
 <via x="-32.004" y="39.0144" extent="1-16" drill="0.35"/>
+<contactref element="SJ7" pad="2"/>
+<contactref element="DISP_SIGS" pad="2"/>
+<wire x1="25.908" y1="70.485" x2="25.908" y2="72.39" width="0.1524" layer="16"/>
+<wire x1="24.003" y1="68.58" x2="25.908" y2="70.485" width="0.1524" layer="16"/>
+<wire x1="24.003" y1="68.58" x2="23.9649" y2="68.5419" width="0.1524" layer="1"/>
+<wire x1="-32.9946" y1="50.7492" x2="-27.8511" y2="45.6057" width="0.1524" layer="1"/>
+<wire x1="-32.9946" y1="50.7492" x2="-33.02" y2="50.8" width="0.1524" layer="1"/>
+<via x="24.003" y="68.58" extent="1-16" drill="0.35"/>
 </signal>
 <signal name="SDI1">
@@
 <contactref element="U1" pad="46"/>
 <contactref element="SV3" pad="7"/>
-<contactref element="SJ5" pad="3"/>
 <wire x1="17.3736" y1="47.8536" x2="17.3736" y2="46.2534" width="0.1524" layer="1"/>
 <wire x1="17.0688" y1="48.1584" x2="17.3736" y2="47.8536" width="0.1524" layer="1"/>
@@
 <wire x1="-27.94" y1="40.64" x2="-25.6794" y2="42.9006" width="0.1524" layer="15"/>
 <wire x1="17.3736" y1="46.2534" x2="17.3" y2="46.1899" width="0.1524" layer="1"/>
-<wire x1="28.194" y1="59.5884" x2="28.194" y2="67.31" width="0.1524" layer="1"/>
 <wire x1="20.1168" y1="51.5112" x2="28.194" y2="59.5884" width="0.1524" layer="15"/>
 <wire x1="19.05" y1="51.5112" x2="20.1168" y2="51.5112" width="0.1524" layer="16"/>
@@
 <wire x1="4.572" y1="68.6562" x2="1.8288" y2="65.913" width="0.1524" layer="16"/>
 <wire x1="17.3736" y1="68.6562" x2="4.572" y2="68.6562" width="0.1524" layer="16"/>
-<wire x1="21.2598" y1="64.77" x2="17.3736" y2="68.6562" width="0.1524" layer="16"/>
+<wire x1="21.2598" y1="64.77" x2="20.2311" y2="65.7987" width="0.1524" layer="16"/>
+<wire x1="20.2311" y1="65.7987" x2="17.3736" y2="68.6562" width="0.1524" layer="16"/>
 <wire x1="4.8006" y1="55.5498" x2="4.83" y2="55.5875" width="0.1524" layer="16"/>
 <wire x1="21.2598" y1="64.77" x2="21.2598" y2="60.96" width="0.1524" layer="16"/>
@@
 <wire x1="19.5834" y1="57.15" x2="19.558" y2="57.15" width="0.1524" layer="16"/>
 <wire x1="21.2598" y1="60.96" x2="21.27" y2="60.96" width="0.1524" layer="16"/>
+<contactref element="SJ7" pad="1"/>
+<wire x1="27.432" y1="71.9328" x2="27.432" y2="72.39" width="0.1524" layer="16"/>
+<wire x1="26.5176" y1="71.0184" x2="27.432" y2="71.9328" width="0.1524" layer="16"/>
+<wire x1="25.4508" y1="71.0184" x2="26.5176" y2="71.0184" width="0.1524" layer="15"/>
+<wire x1="20.574" y1="66.1416" x2="25.4508" y2="71.0184" width="0.1524" layer="15"/>
+<wire x1="20.2311" y1="65.7987" x2="20.574" y2="66.1416" width="0.1524" layer="16"/>
+<via x="26.5176" y="71.0184" extent="1-16" drill="0.35"/>
+<via x="20.574" y="66.1416" extent="1-16" drill="0.35"/>
+</signal>
+<signal name="MISC_0">
+<contactref element="SJ5" pad="3"/>
+<contactref element="DISP_SIGS" pad="1"/>
+<wire x1="28.194" y1="68.1228" x2="28.194" y2="67.31" width="0.1524" layer="1"/>
+<wire x1="20.1168" y1="76.2" x2="28.194" y2="68.1228" width="0.1524" layer="1"/>
+<wire x1="20.1168" y1="76.6572" x2="20.1168" y2="76.2" width="0.1524" layer="1"/>
+<wire x1="19.5072" y1="77.2668" x2="20.1168" y2="76.6572" width="0.1524" layer="1"/>
+<wire x1="16.8402" y1="77.2668" x2="19.5072" y2="77.2668" width="0.1524" layer="1"/>
+<wire x1="14.859" y1="75.2856" x2="16.8402" y2="77.2668" width="0.1524" layer="1"/>
+<wire x1="-14.7066" y1="75.2856" x2="14.859" y2="75.2856" width="0.1524" layer="15"/>
+<wire x1="-35.5092" y1="54.483" x2="-14.7066" y2="75.2856" width="0.1524" layer="15"/>
+<wire x1="-35.5092" y1="50.8254" x2="-35.5092" y2="54.483" width="0.1524" layer="15"/>
+<wire x1="-35.5092" y1="50.8254" x2="-35.56" y2="50.8" width="0.1524" layer="15"/>
+<via x="14.859" y="75.2856" extent="1-16" drill="0.35"/>
 </signal>
 </signals>

Commit message: up
Parts:
- added R10, R11: 10k, rcl:M0805
- added SV4: IMU_SIG, con-lstb:MA10-1
Connections:
- new net BNO_CHIP_RESET: C32.1, R9.1, SJ4.2, SJ7.1, SV4.8, U3.11
- new net N$18: R11.2, U3.15
- net 32KHZ: now also SV4.9
- net EXT_INT2: now also SV4.6
- net IMU_CS: now also SV4.2
- net N$17: now also R10.2, U3.16; no longer C32.1, R9.1, SJ4.2, SJ7.1, U3.11
- net RED_LED: now also SV4.7
- net SCK2: now also SV4.3
- net SDI2: now also SV4.4
- net SDO2: now also SV4.5
- net TP3_SIG_WAKE: now also SV4.10
- net VDD: now also R10.1, R11.1
- net VSS: now also SV4.1
Routing:
- net BNO_CHIP_RESET: track 0.00 -> 114.3 mm, vias 0 -> 4
- net RED_LED: track 29.8 -> 89.3 mm, vias 4 -> 5
- net SDO2: track 31.9 -> 82.9 mm, vias 4 -> 5
- net 32KHZ: track 11.6 -> 62.0 mm
- net N$17: track 56.7 -> 10.4 mm, vias 2 -> 0
- net SDI2: track 55.0 -> 100.0 mm, vias 4 -> 5
- net TP3_SIG_WAKE: track 47.6 -> 92.0 mm
- net EXT_INT2: track 38.8 -> 81.3 mm, vias 3 -> 5
- net SCK2: track 37.5 -> 78.7 mm, vias 4 -> 5
- net IMU_CS: track 64.7 -> 93.7 mm
- net MISC_0: track 81.7 -> 99.6 mm
- net VDD: track 768.3 -> 774.1 mm
- net N$14: track 15.2 -> 19.4 mm, vias 0 -> 2
- net N$18: track 0.00 -> 3.57 mm
Other:
- board text added: "PIC32MK-CANFD HID V1.2-fixes"
- board text removed: "PIC32MK-CANFD HID V1.1"

Commit message: up
Parts:
- added PS1: MYRBP500080B21RE, MYRBP500080B21RE:MYRBP500080B21RE
- added PS2: MYRLP330015F21RE, MYRLP330015F21RE:MYRLP330015F21RE
Changed lines of the file:
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@@
 <attribute name="VALUE" x="-2.54" y="57.15" size="1.27" layer="28" rot="MR180"/>
+</element>
+<element name="PS1" library="MYRBP500080B21RE" package="MYRBP500080B21RE" value="MYRBP500080B21RE" x="54.61" y="57.15" smashed="yes" rot="MR0">
+<attribute name="DESCRIPTION" value="Non-Isolated DC/DC Converters" x="54.61" y="57.15" size="1.778" layer="28" rot="MR0" display="off"/>
+<attribute name="HEIGHT" value="1.04mm" x="54.61" y="57.15" size="1.778" layer="28" rot="MR0" display="off"/>
+<attribute name="MANUFACTURER_NAME" value="Murata Electronics" x="54.61" y="57.15" size="1.778" layer="28" rot="MR0" display="off"/>
+<attribute name="MANUFACTURER_PART_NUMBER" value="MYRBP500080B21RE" x="54.61" y="57.15" size="1.778" layer="28" rot="MR0" display="off"/>
+<attribute name="MOUSER_PART_NUMBER" value="81-MYRBP500080B21RE" x="54.61" y="57.15" size="1.778" layer="28" rot="MR0" display="off"/>
+<attribute name="MOUSER_PRICE-STOCK" value="https://www.mouser.co.uk/ProductDetail/Murata-Electronics/MYRBP500080B21RE?qs=hd1VzrDQEGi2HKFlO8%252BP9Q%3D%3D" x="54.61" y="57.15" size="1.778" layer="28" rot="MR0" display="off"/>
+<attribute name="NAME" x="55.88" y="58.42" size="1.27" layer="26" rot="MR0" align="center"/>
+<attribute name="VALUE" x="54.61" y="57.15" size="1.27" layer="28" rot="MR0" align="center"/>
+</element>
+<element name="PS2" library="MYRLP330015F21RE" package="MYRLP330015F21RE" value="MYRLP330015F21RE" x="54.61" y="52.07" smashed="yes" rot="MR0">
+<attribute name="DESCRIPTION" value="Non-Isolated DC/DC Converters 150mA 1.8-6.0Vin 3.30Vout -40 to 85degC PWM" x="54.61" y="52.07" size="1.778" layer="28" rot="MR0" display="off"/>
+<attribute name="HEIGHT" value="1.04mm" x="54.61" y="52.07" size="1.778" layer="28" rot="MR0" display="off"/>
+<attribute name="MANUFACTURER_NAME" value="Murata Electronics" x="54.61" y="52.07" size="1.778" layer="28" rot="MR0" display="off"/>
+<attribute name="MANUFACTURER_PART_NUMBER" value="MYRLP330015F21RE" x="54.61" y="52.07" size="1.778" layer="28" rot="MR0" display="off"/>
+<attribute name="MOUSER_PART_NUMBER" value="580-MYRLP330015F21RE" x="54.61" y="52.07" size="1.778" layer="28" rot="MR0" display="off"/>
+<attribute name="MOUSER_PRICE-STOCK" value="https://www.mouser.co.uk/ProductDetail/Murata-Power-Solutions/MYRLP330015F21RE?qs=vvQtp7zwQdNOX7V%2FydgWKA%3D%3D" x="54.61" y="52.07" size="1.778" layer="28" rot="MR0" display="off"/>
+<attribute name="NAME" x="55.88" y="52.07" size="1.27" layer="26" rot="MR0" align="center"/>
+<attribute name="VALUE" x="54.61" y="52.07" size="1.27" layer="28" rot="MR0" align="center"/>
 </element>
 </elements>

Commit message: up
Parts:
- added +5VDC: +5VDC, pinhead:1X02
- added C33, C44: 10uf, rcl:C0805
- added SJ8: BLANK_ON, jumper:SJ
- moved PS1 18.0 mm to (41.9, 69.8)
- moved PS2 1.80 mm to (55.9, 53.3)
Connections:
- removed net DC_INPUT: 3.3VDC.1, C20.1, C21.1, R6.1
- new net +5V: +5VDC.1, +5VDC.2, C33.1, IC3.3, PS1.6
- new net N$20: PS2.1, PS2.7
- new net N$23: PS1.5, PS1.8
- new net V+: 3.3VDC.1, C20.1, C21.1, PS2.4, PS2.6, R6.1
- net MISC_0: now also SJ8.1
- net RB11: now also SJ8.2
- net VDD: now also C44.1, PS1.1, PS1.3, PS1.7, PS2.3, PS2.8; no longer IC3.3
- net VSS: now also C33.2, C44.2, PS1.2, PS1.4, PS1.9, PS2.2, PS2.5, PS2.9
Routing:
- net V+: track 0.00 -> 58.8 mm, vias 0 -> 2
- net VDD: track 774.1 -> 823.3 mm, vias 10 -> 11
- net +5V: track 0.00 -> 40.2 mm
- net DC_INPUT: track 35.8 -> 0.00 mm, vias 2 -> 0
- net VSS: track 326.9 -> 357.3 mm, vias 10 -> 11
- net MISC_0: track 99.6 -> 108.4 mm
- net N$23: track 0.00 -> 4.82 mm
- net RB11: track 68.9 -> 72.2 mm, vias 0 -> 2
- net N$20: track 0.00 -> 1.31 mm
- added copper zone on layer 16, net N$20
- added copper zone on layer 16, net N$23

Commit message: up
Parts:
- added C45, C46: 0.1uf, rcl:C0805
- added C47: 10uf, rcl:C0805
- added U4: BME280, BME280:PSON65P250X250X100-8N
- added U5: VCNL4040M3OE, VCNL4040M3OE:VISHAY_VCNL4040_4X2X1.1
- moved PS1 43.8 mm to (49.5, 26.7)
- moved C33 33.6 mm to (47.0, 31.8)
- moved C44 33.4 mm to (52.1, 31.8)
- moved PS2 31.4 mm to (39.4, 26.7)
Connections:
- removed net N$17: R10.2, U3.16
- removed net N$18: R11.2, U3.15
- new net BSCL: R11.2, U3.15, U4.4, U5.8
- new net BSDA: R10.2, U3.16, U4.3, U5.7
- new net N$22: U5.2, U5.5
- net VDD: now also C45.1, C46.1, C47.1, U4.2, U4.6, U4.8, U5.3, U5.4
- net VSS: now also C45.2, C46.2, C47.2, U4.1, U4.7, U5.1
Routing:
- net VDD: track 823.3 -> 745.9 mm, vias 11 -> 7
- net BSDA: track 0.00 -> 71.4 mm, vias 0 -> 5
- net BSCL: track 0.00 -> 49.6 mm, vias 0 -> 4
- net VSS: track 357.3 -> 398.2 mm, vias 11 -> 14
- net +5V: track 40.2 -> 68.0 mm
- net DIS_RESET: track 217.7 -> 243.2 mm, vias 3 -> 2
- net SCK1: track 216.7 -> 242.2 mm, vias 1 -> 4
- net RED_LED: track 89.3 -> 111.1 mm, vias 5 -> 2
- net MISC_0: track 108.4 -> 89.6 mm
- net QEB2: track 95.1 -> 113.6 mm, vias 4 -> 3
- net IMU_CS: track 93.7 -> 76.6 mm, vias 4 -> 5
- net SDO1: track 228.8 -> 245.9 mm, vias 2 -> 1
- net SDO2: track 82.9 -> 67.6 mm, vias 5 -> 3
- net RB8: track 133.2 -> 118.1 mm, vias 1 -> 2
- net SDI2: track 100.0 -> 85.3 mm, vias 5 -> 4
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- removed copper zone on layer 16, net N$20
- removed copper zone on layer 16, net N$23

Commit message: up
Parts:
- moved C31 20.8 mm to (12.7, 49.5), turned to 0 degrees
- moved C4 20.4 mm to (26.7, 49.5)
- moved C30 15.5 mm to (12.7, 53.3), turned to 0 degrees
- moved OS2 14.2 mm to (19.1, 64.8)
- moved U3 14.2 mm to (19.1, 59.7)
- moved R10 14.0 mm to (6.35, 58.4)
- moved R11 10.8 mm to (6.35, 62.2)
- moved C45 8.89 mm to (26.7, 53.3)
- moved C10 6.48 mm to (12.7, 34.3), turned to 0 degrees
- moved IC1 6.48 mm to (19.1, 49.5)
- moved U4 6.48 mm to (19.1, 54.6)
- moved R6 6.48 mm to (39.4, 33.0)
- moved C32 6.35 mm to (26.7, 61.0)
- moved R9 6.35 mm to (26.7, 64.8)
- moved SJ4 6.35 mm to (26.7, 57.1)
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Routing:
- net VDD: track 745.9 -> 697.1 mm, vias 7 -> 5
- net DIS_RESET: track 243.2 -> 204.7 mm, vias 2 -> 5
- net BSDA: track 71.4 -> 33.2 mm, vias 5 -> 4
- net VSS: track 398.2 -> 366.7 mm, vias 14 -> 18
- net SDI2: track 85.3 -> 114.8 mm
- net RB8: track 118.1 -> 145.1 mm
- net 32KHZ: track 56.9 -> 82.8 mm, vias 0 -> 2
- net PGC_C1RX: track 105.7 -> 131.4 mm, vias 2 -> 3
- net BNO_CHIP_RESET: track 106.3 -> 84.1 mm
- net RED_LED: track 111.1 -> 90.5 mm, vias 2 -> 3
- net IMU_CS: track 76.6 -> 95.4 mm, vias 5 -> 4
- net RA10: track 102.0 -> 120.8 mm, vias 1 -> 2
- net DIS_CS: track 216.8 -> 234.1 mm, vias 1 -> 2
- net RA7: track 111.9 -> 129.0 mm
- net PGD_C1TX: track 107.4 -> 124.5 mm, vias 2 -> 3
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Other:
- board text added: "PIC32MK-CANFD HID V1.3"
- board text removed: "PIC32MK-CANFD HID V1.2-fixes"
