File: ll-tester.brd (EAGLE design)
At the start: 120.6 x 145.7 mm, 133 parts, among them IC1 BMA490L, IC2 TCAN330GD, IC3 EM14R0D-R20-L064S, IC4 CAT4238TD-GT3, U1 PIC32MK0512MCJ048T-I/Y8XTQFP4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, U2 MAX6126B30, U3 BNO086, U4 BME280, U5 VCNL4040M3OE

Commit message: up
Parts:
- added R12, R13: 0 ohms, rcl:R0805
- added R21, R22: 1k, rcl:R0805
- added SJ9: QEI_PWR, jumper:SJ_2
Connections:
- new net CHANA: IC3.A1, R12.1
- new net CHANB: IC3.B1, R13.1
- new net CHANP: IC3.3, SJ9.2
- net +5V: now also SJ9.3; no longer IC3.3
- net QEA2: now also R12.2, R22.1; no longer IC3.A1
- net QEB2: now also R13.2, R21.2; no longer IC3.B1
- net VDD: now also SJ9.1
- net VSS: now also R21.1, R22.2
Routing:
- net VSS: track 416.0 -> 384.2 mm, vias 15 -> 17
- net CHANB: track 0.00 -> 28.1 mm
- net VDD: track 706.7 -> 731.7 mm, vias 12 -> 13
- net SCK1: track 252.3 -> 227.3 mm, vias 4 -> 3
- net RA10: track 99.8 -> 122.4 mm, vias 3 -> 2
- net N$7: track 12.3 -> 34.3 mm, vias 2 -> 0
- net EXT_INT2: track 77.9 -> 99.5 mm, vias 4 -> 5
- net DIS_CS: track 199.2 -> 219.9 mm
- net DIS_MODE: track 233.7 -> 253.7 mm, vias 4 -> 2
- net RA7: track 107.3 -> 127.2 mm, vias 2 -> 3
- net U1RX: track 103.6 -> 86.1 mm, vias 1 -> 2
- net CHANA: track 0.00 -> 17.0 mm
- net RB11: track 78.7 -> 62.5 mm, vias 0 -> 3
- net +5V: track 78.6 -> 62.8 mm, vias 0 -> 1
- net N$14: track 24.4 -> 9.10 mm, vias 2 -> 0
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
Commit message: up
Parts:
- moved IC1 6.35 mm to (22.9, 54.6)
- moved GLORY 2.84 mm to (36.8, 49.5), turned to 90 degrees
- moved C12 2.54 mm to (29.2, 45.7)
- moved C4 2.54 mm to (29.2, 49.5)
- moved C45 2.54 mm to (29.2, 53.3)
- moved R8 2.54 mm to (29.2, 57.1)
- moved U4 1.27 mm to (17.8, 54.6)
Connections:
- removed net N$66: IC4.3, PAD8.1, R19.1
- removed net N$67: C43.1, D2.C, PAD7.1
- removed net N$68: PAD10.1, PAD9.1
- removed net N$69: PAD11.1, PAD12.1
- new net CA1: C43.1, D2.C, LCD2.1, PAD7.1
- new net CA2: LCD2.18, LCD2.2, PAD10.1, PAD9.1
- new net CA3: LCD2.19, LCD2.3, PAD11.1, PAD12.1
- new net CA6: IC4.3, LCD2.20, PAD8.1, R19.1
Routing:
- net VDD: track 731.7 -> 0.00 mm, vias 13 -> 0
- net VSS: track 384.2 -> 0.00 mm, vias 17 -> 0
- net DIS_MODE: track 253.7 -> 0.00 mm, vias 2 -> 0
- net SDO1: track 238.1 -> 0.00 mm, vias 3 -> 0
- net SCK1: track 227.3 -> 0.00 mm, vias 3 -> 0
- net DIS_CS: track 219.9 -> 0.00 mm, vias 2 -> 0
- net DIS_RESET: track 200.4 -> 0.00 mm, vias 4 -> 0
- net RA7: track 127.2 -> 0.00 mm, vias 3 -> 0
- net RD8: track 124.9 -> 0.00 mm, vias 3 -> 0
- net QEA2: track 122.9 -> 0.00 mm, vias 4 -> 0
- net RA10: track 122.4 -> 0.00 mm, vias 2 -> 0
- net MCLR_SIG: track 121.3 -> 0.00 mm, vias 2 -> 0
- net RB8: track 120.7 -> 0.00 mm, vias 2 -> 0
- net PGD_C1TX: track 119.5 -> 0.00 mm, vias 2 -> 0
- net PGC_C1RX: track 117.6 -> 0.00 mm, vias 2 -> 0
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
Commit message: up
Routing:
- net VDD: track 0.00 -> 745.9 mm, vias 0 -> 14
- net VSS: track 0.00 -> 379.8 mm, vias 0 -> 18
- net SCK1: track 0.00 -> 259.1 mm
- net DIS_MODE: track 0.00 -> 243.9 mm, vias 0 -> 2
- net SDO1: track 0.00 -> 240.3 mm, vias 0 -> 1
- net DIS_RESET: track 0.00 -> 233.6 mm, vias 0 -> 4
- net DIS_CS: track 0.00 -> 207.5 mm, vias 0 -> 2
- net RD8: track 0.00 -> 145.2 mm, vias 0 -> 2
- net RB8: track 0.00 -> 134.6 mm, vias 0 -> 3
- net MCLR_SIG: track 0.00 -> 127.1 mm, vias 0 -> 5
- net QEA2: track 0.00 -> 125.0 mm, vias 0 -> 5
- net IMU_CS: track 0.00 -> 118.4 mm, vias 0 -> 4
- net PGC_C1RX: track 0.00 -> 117.2 mm, vias 0 -> 3
- net PGD_C1TX: track 0.00 -> 108.5 mm, vias 0 -> 2
- net SDI2: track 0.00 -> 104.3 mm, vias 0 -> 5
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
Commit message: up
Routing:
- net TP3_SIG_WAKE: track 97.3 -> 99.8 mm, vias 4 -> 3
Changed lines of the file:
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@@
 <vertex x="17.78" y="66.04"/>
 </polygon>
+<polygon width="0.1524" layer="43">
+<vertex x="21.59" y="55.88"/>
+<vertex x="24.13" y="55.88"/>
+<vertex x="24.13" y="53.34"/>
+<vertex x="21.59" y="53.34"/>
+</polygon>
 </plain>
 <attributes>
@@
 <contactref element="U3" pad="6"/>
 <contactref element="SV4" pad="10"/>
-<wire x1="22.7076" y1="54.7878" x2="22.098" y2="54.7878" width="0.1524" layer="16"/>
-<wire x1="22.86" y1="54.6354" x2="22.7076" y2="54.7878" width="0.1524" layer="16"/>
-<wire x1="21.9456" y1="55.5498" x2="22.86" y2="54.6354" width="0.1524" layer="15"/>
-<wire x1="21.8694" y1="55.5498" x2="21.9456" y2="55.5498" width="0.1524" layer="15"/>
-<wire x1="21.336" y1="56.0832" x2="21.8694" y2="55.5498" width="0.1524" layer="15"/>
-<wire x1="21.336" y1="56.9976" x2="21.336" y2="56.0832" width="0.1524" layer="15"/>
 <wire x1="21.336" y1="58.0644" x2="21.336" y2="56.9976" width="0.1524" layer="16"/>
-<wire x1="22.098" y1="54.7878" x2="22.085" y2="54.86" width="0.1524" layer="16"/>
 <wire x1="21.336" y1="58.0644" x2="21.3" y2="58.1275" width="0.1524" layer="16"/>
 <wire x1="10.8966" y1="39.624" x2="14.7066" y2="39.624" width="0.1524" layer="1"/>
@@
 <wire x1="14.7066" y1="39.624" x2="14.7701" y2="39.66" width="0.1524" layer="1"/>
 <wire x1="-1.2192" y1="52.0446" x2="-1.27" y2="52.07" width="0.1524" layer="15"/>
-<wire x1="22.7838" y1="52.1208" x2="22.7838" y2="54.6354" width="0.1524" layer="15"/>
-<wire x1="21.717" y1="51.054" x2="22.7838" y2="52.1208" width="0.1524" layer="15"/>
-<wire x1="21.717" y1="49.8348" x2="21.717" y2="51.054" width="0.1524" layer="15"/>
-<wire x1="17.8308" y1="45.9486" x2="21.717" y2="49.8348" width="0.1524" layer="15"/>
 <wire x1="13.6398" y1="45.9486" x2="17.8308" y2="45.9486" width="0.1524" layer="15"/>
 <wire x1="8.763" y1="41.0718" x2="13.6398" y2="45.9486" width="0.1524" layer="15"/>
-<wire x1="22.7838" y1="54.6354" x2="22.86" y2="54.6354" width="0.1524" layer="15"/>
 <wire x1="8.763" y1="41.0718" x2="8.763" y2="40.9956" width="0.1524" layer="15"/>
 <wire x1="-42.8244" y1="55.8546" x2="-43.1292" y2="55.8546" width="0.1524" layer="1"/>
@@
 <wire x1="-43.1292" y1="55.8546" x2="-43.18" y2="55.88" width="0.1524" layer="1"/>
 <wire x1="-1.2954" y1="52.1208" x2="-1.27" y2="52.07" width="0.1524" layer="15"/>
-<via x="22.86" y="54.6354" extent="1-16" drill="0.35"/>
 <via x="21.336" y="56.9976" extent="1-16" drill="0.35"/>
 <via x="8.763" y="40.9956" extent="1-16" drill="0.35"/>
 <via x="-4.2672" y="52.197" extent="1-16" drill="0.35"/>
+<wire x1="21.2598" y1="54.864" x2="22.0218" y2="54.864" width="0.1524" layer="16"/>
+<wire x1="20.1168" y1="56.007" x2="21.2598" y2="54.864" width="0.1524" layer="16"/>
+<wire x1="20.1168" y1="56.6166" x2="20.1168" y2="56.007" width="0.1524" layer="16"/>
+<wire x1="20.4978" y1="56.9976" x2="20.1168" y2="56.6166" width="0.1524" layer="16"/>
+<wire x1="21.336" y1="56.9976" x2="20.4978" y2="56.9976" width="0.1524" layer="16"/>
+<wire x1="22.0218" y1="54.864" x2="22.085" y2="54.86" width="0.1524" layer="16"/>
+<wire x1="21.336" y1="54.102" x2="21.336" y2="56.9976" width="0.1524" layer="15"/>
+<wire x1="21.717" y1="53.721" x2="21.336" y2="54.102" width="0.1524" layer="15"/>
+<wire x1="21.717" y1="49.8348" x2="21.717" y2="53.721" width="0.1524" layer="15"/>
+<wire x1="17.8308" y1="45.9486" x2="21.717" y2="49.8348" width="0.1524" layer="15"/>
 </signal>
 <signal name="N$6">

Commit message: up
Parts:
- added I2C: I2C, pinhead:1X02
Connections:
- net BSCL: now also I2C.1
- net BSDA: now also I2C.2
Routing:
- net BSCL: track 39.1 -> 64.3 mm, vias 4 -> 5
- net BSDA: track 60.9 -> 71.6 mm
Other:
- board text added: "C D"
- board text added: "CAN-FD"
- board text added: "ICSP"
- board text added: "IMU I2C"
- board text added: "PIC32MK-CANFD HID V1.4"
- board text removed: "PIC32MK-CANFD HID V1.3"
Changed lines of the file:
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@@
 <wire x1="62.21" y1="163.5" x2="-58.42" y2="163.5" width="0" layer="20"/>
 <wire x1="-58.42" y1="163.5" x2="-58.42" y2="162.23" width="0" layer="20"/>
-<text x="25.4" y="20.32" size="1.016" layer="1" font="vector" ratio="17" distance="77" rot="R180">PIC32MK-CANFD HID V1.3</text>
+<text x="25.4" y="20.32" size="1.016" layer="1" font="vector" ratio="17" distance="77" rot="R180">PIC32MK-CANFD HID V1.4</text>
 <hole x="-55.88" y="20.32" drill="2.54"/>
 <hole x="-55.88" y="58.42" drill="2.54"/>
@@
 <vertex x="21.59" y="53.34"/>
 </polygon>
+<text x="-3.81" y="73.66" size="1.778" layer="1" font="vector" ratio="15">IMU I2C</text>
+<text x="6.35" y="71.12" size="1.778" layer="1" font="vector" ratio="15">C D</text>
+<text x="53.34" y="31.75" size="1.778" layer="1" font="vector" ratio="15">ICSP</text>
+<text x="-54.61" y="36.83" size="1.778" layer="1" font="vector" ratio="15" rot="R90">CAN-FD</text>
 </plain>
 <attributes>
@@
 <attribute name="VALUE" x="59.69" y="65.405" size="1.27" layer="27" rot="R90"/>
 </element>
+<element name="I2C" library="pinhead" library_urn="urn:adsk.eagle:library:325" package="1X02" package3d_urn="urn:adsk.eagle:package:22435/2" value="I2C" x="8.89" y="74.93" smashed="yes" rot="MR180">
+<attribute name="NAME" x="6.2738" y="73.1012" size="1.27" layer="26" ratio="10" rot="MR180"/>
+<attribute name="POPULARITY" value="98" x="8.89" y="74.93" size="1.778" layer="28" rot="MR180" display="off"/>
+<attribute name="VALUE" x="6.35" y="78.105" size="1.27" layer="28" rot="MR180"/>
+</element>
 </elements>
 <signals>
@@
 <via x="18.7452" y="69.8754" extent="1-16" drill="0.35"/>
 <via x="8.5344" y="58.5216" extent="1-16" drill="0.35"/>
+<contactref element="I2C" pad="2"/>
+<wire x1="13.716" y1="74.9046" x2="10.2108" y2="74.9046" width="0.1524" layer="15"/>
+<wire x1="18.7452" y1="69.8754" x2="13.716" y2="74.9046" width="0.1524" layer="15"/>
+<wire x1="10.2108" y1="74.9046" x2="10.16" y2="74.93" width="0.1524" layer="15"/>
 </signal>
 <signal name="BSCL">
@@
 <via x="23.8506" y="64.8462" extent="1-16" drill="0.35"/>
 <via x="12.3444" y="64.008" extent="1-16" drill="0.35"/>
+<contactref element="I2C" pad="1"/>
+<wire x1="8.763" y1="74.9808" x2="7.62" y2="74.9808" width="0.1524" layer="15"/>
+<wire x1="9.7536" y1="75.9714" x2="8.763" y2="74.9808" width="0.1524" layer="15"/>
+<wire x1="15.3924" y1="75.9714" x2="9.7536" y2="75.9714" width="0.1524" layer="15"/>
+<wire x1="19.6596" y1="71.7042" x2="15.3924" y2="75.9714" width="0.1524" layer="15"/>
+<wire x1="18.1356" y1="70.1802" x2="19.6596" y2="71.7042" width="0.1524" layer="1"/>
+<wire x1="18.1356" y1="68.6562" x2="18.1356" y2="70.1802" width="0.1524" layer="1"/>
+<wire x1="21.9456" y1="64.8462" x2="18.1356" y2="68.6562" width="0.1524" layer="1"/>
+<wire x1="23.8506" y1="64.8462" x2="21.9456" y2="64.8462" width="0.1524" layer="1"/>
+<wire x1="7.62" y1="74.9808" x2="7.62" y2="74.93" width="0.1524" layer="15"/>
+<via x="19.6596" y="71.7042" extent="1-16" drill="0.35"/>
 </signal>
 <signal name="N$20" class="1">
