File: ll-tester.sch (EAGLE design)
At the start: 105 parts, among them IC1 BMA490L, IC2 TCAN330GD, IC3 EM14R0D-R20-L064S, IC4 CAT4238TD-GT3, U1 PIC32MK0512MCJ048T-I/Y8XTQFP4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, U2 MAX6126B30

Commit message: up
Parts:
- added R7: 10k, rcl:R-US_M0805
Connections:
- net RB8: now also R7.1
- net VDD: now also R7.2
Changed lines of the file:
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@@
 <part name="C29" library="rcl" library_urn="urn:adsk.eagle:library:334" deviceset="C-US" device="C0805" package3d_urn="urn:adsk.eagle:package:23617/2" value="10uf"/>
 <part name="VSS59" library="supply1" library_urn="urn:adsk.eagle:library:371" deviceset="VSS" device=""/>
+<part name="R7" library="rcl" library_urn="urn:adsk.eagle:library:334" deviceset="R-US_" device="M0805" package3d_urn="urn:adsk.eagle:package:23556/2" value="10k"/>
+<part name="VDD18" library="supply1" library_urn="urn:adsk.eagle:library:371" deviceset="VDD" device=""/>
 </parts>
 <sheets>
@@
 <instance part="VSS59" gate="G$1" x="-71.12" y="-35.56" smashed="yes">
 <attribute name="VALUE" x="-73.66" y="-40.64" size="1.778" layer="96" rot="R90"/>
+</instance>
+<instance part="R7" gate="G$1" x="-81.28" y="-81.28" smashed="yes" rot="R90">
+<attribute name="NAME" x="-82.7786" y="-85.09" size="1.778" layer="95" rot="R90"/>
+<attribute name="VALUE" x="-77.978" y="-85.09" size="1.778" layer="96" rot="R90"/>
+</instance>
+<instance part="VDD18" gate="G$1" x="-83.82" y="-76.2" smashed="yes" rot="R90">
+<attribute name="VALUE" x="-81.28" y="-78.74" size="1.778" layer="96" rot="R180"/>
 </instance>
 </instances>
@@
 <pinref part="C29" gate="G$1" pin="1"/>
 <junction x="-78.74" y="-33.02"/>
+</segment>
+<segment>
+<pinref part="R7" gate="G$1" pin="2"/>
+<pinref part="VDD18" gate="G$1" pin="VDD"/>
+<junction x="-81.28" y="-76.2"/>
 </segment>
 </net>
@@
 <pinref part="C25" gate="G$1" pin="1"/>
 <junction x="-66.04" y="-86.36"/>
-</segment>
-</net>
+<pinref part="R7" gate="G$1" pin="1"/>
+</segment>
+</net>

Commit message: up
Connections:
- net INDX2: now also SJ5.3
- net QEB2: no longer SJ5.3
Changed lines of the file:
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@@
-</segment>
-<segment>
-<wire x1="30.48" y1="-111.76" x2="43.18" y2="-111.76" width="0.1524" layer="91"/>
-<wire x1="43.18" y1="-111.76" x2="78.74" y2="-111.76" width="0.1524" layer="91"/>
-<wire x1="78.74" y1="-111.76" x2="78.74" y2="-170.18" width="0.1524" layer="91"/>
-<wire x1="78.74" y1="-170.18" x2="106.68" y2="-170.18" width="0.1524" layer="91"/>
-<wire x1="106.68" y1="-170.18" x2="106.68" y2="-172.72" width="0.1524" layer="91"/>
-<pinref part="SJ5" gate="G$1" pin="3"/>
-<wire x1="106.68" y1="-172.72" x2="111.76" y2="-172.72" width="0.1524" layer="91"/>
-<junction x="111.76" y="-172.72"/>
-<label x="15.24" y="-111.76" size="1.778" layer="95"/>
-<label x="73.66" y="-111.76" size="1.778" layer="95"/>
-<junction x="43.18" y="-111.76"/>
-<junction x="30.48" y="-111.76"/>
 </segment>
 <segment>
@@
 <junction x="-43.18" y="0"/>
 </segment>
+<segment>
+<pinref part="SJ5" gate="G$1" pin="3"/>
+<wire x1="111.76" y1="-172.72" x2="104.14" y2="-172.72" width="0.1524" layer="91"/>
+<wire x1="104.14" y1="-172.72" x2="104.14" y2="-170.18" width="0.1524" layer="91"/>
+<wire x1="104.14" y1="-170.18" x2="78.74" y2="-170.18" width="0.1524" layer="91"/>
+<wire x1="78.74" y1="-170.18" x2="78.74" y2="-111.76" width="0.1524" layer="91"/>
+<wire x1="78.74" y1="-111.76" x2="43.18" y2="-111.76" width="0.1524" layer="91"/>
+<junction x="43.18" y="-111.76"/>
+<wire x1="30.48" y1="-111.76" x2="43.18" y2="-111.76" width="0.1524" layer="91"/>
+<junction x="30.48" y="-111.76"/>
+<label x="15.24" y="-111.76" size="1.778" layer="95"/>
+<label x="88.9" y="-170.18" size="1.778" layer="95"/>
+<junction x="111.76" y="-172.72"/>
+</segment>
 </net>

Commit message: up
Parts:
- added C30, C31: 0.1uf, rcl:C-USC0805
- added OS2: OSC-OE-IQXO-793, IQD-Frequency-Products:OSC-OE-IQXO-793
- added U3: BNO080, BNO080:BNO080
Connections:
- new net 32KHZ: OS2.OUT, U3.XIN32
- new net N$14: C30.1, U3.CAP
- net BMA_INT2: now also U3.!H_INT
- net IMU_CS: now also U3.!H_CS
- net SCK2: now also U3.H_SCL/SCK/RX
- net SDI2: now also U3.H_SDA/H_MISO/TX
- net SDO2: now also U3.SA0/H_MOSI
- net VDD: now also C31.1, OS2.CON, OS2.VDD, U3.CLKSEL0, U3.VDD, U3.VDDIO, U3.XOUT32/CLKSEL1
- net VSS: now also C30.2, C31.2, OS2.VSS, U3.GND, U3.GNDIO
Changed lines of the file:
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@@
 <part name="R7" library="rcl" library_urn="urn:adsk.eagle:library:334" deviceset="R-US_" device="M0805" package3d_urn="urn:adsk.eagle:package:23556/2" value="10k"/>
 <part name="VDD18" library="supply1" library_urn="urn:adsk.eagle:library:371" deviceset="VDD" device=""/>
+<part name="U3" library="BNO080" deviceset="BNO080" device=""/>
+<part name="C30" library="rcl" library_urn="urn:adsk.eagle:library:334" deviceset="C-US" device="C0805" package3d_urn="urn:adsk.eagle:package:23617/2" value="0.1uf"/>
+<part name="VSS60" library="supply1" library_urn="urn:adsk.eagle:library:371" deviceset="VSS" device=""/>
+<part name="OS2" library="IQD-Frequency-Products" library_urn="urn:adsk.eagle:library:90" deviceset="OSC-OE" device="-IQXO-793" package3d_urn="urn:adsk.eagle:package:3371/1"/>
+<part name="C31" library="rcl" library_urn="urn:adsk.eagle:library:334" deviceset="C-US" device="C0805" package3d_urn="urn:adsk.eagle:package:23617/2" value="0.1uf"/>
 </parts>
 <sheets>
@@
 <instance part="VDD18" gate="G$1" x="-83.82" y="-76.2" smashed="yes" rot="R90">
 <attribute name="VALUE" x="-81.28" y="-78.74" size="1.778" layer="96" rot="R180"/>
+</instance>
+<instance part="U3" gate="G$1" x="200.66" y="137.16" smashed="yes">
+<attribute name="NAME" x="180.34" y="163.83" size="2.54" layer="95"/>
+<attribute name="VALUE" x="180.34" y="107.95" size="2.54" layer="96"/>
+</instance>
+<instance part="C30" gate="G$1" x="175.26" y="121.92" smashed="yes">
+<attribute name="NAME" x="176.276" y="122.555" size="1.778" layer="95"/>
+<attribute name="VALUE" x="176.276" y="117.729" size="1.778" layer="96"/>
+</instance>
+<instance part="VSS60" gate="G$1" x="175.26" y="114.3" smashed="yes">
+<attribute name="VALUE" x="172.72" y="109.22" size="1.778" layer="96" rot="R90"/>
+</instance>
+<instance part="OS2" gate="A" x="271.78" y="127" smashed="yes" rot="R180">
+<attribute name="NAME" x="279.4" y="118.745" size="1.778" layer="95" rot="R180"/>
+<attribute name="VALUE" x="279.4" y="137.16" size="1.778" layer="96" rot="R180"/>
+</instance>
+<instance part="C31" gate="G$1" x="292.1" y="124.46" smashed="yes" rot="R180">
+<attribute name="NAME" x="291.084" y="123.825" size="1.778" layer="95" rot="R180"/>
+<attribute name="VALUE" x="291.084" y="128.651" size="1.778" layer="96" rot="R180"/>
 </instance>
 </instances>
@@
 <junction x="-81.28" y="-76.2"/>
 </segment>
+<segment>
+<wire x1="238.76" y1="160.02" x2="226.06" y2="160.02" width="0.1524" layer="91"/>
+<pinref part="U3" gate="G$1" pin="VDD"/>
+<junction x="226.06" y="160.02"/>
+<junction x="238.76" y="160.02"/>
+<label x="246.38" y="160.02" size="1.778" layer="95"/>
+</segment>
+<segment>
+<wire x1="236.22" y1="157.48" x2="226.06" y2="157.48" width="0.1524" layer="91"/>
+<pinref part="U3" gate="G$1" pin="VDDIO"/>
+<junction x="226.06" y="157.48"/>
+<junction x="236.22" y="157.48"/>
+<label x="246.38" y="157.48" size="1.778" layer="95"/>
+</segment>
+<segment>
+<wire x1="236.22" y1="124.46" x2="226.06" y2="124.46" width="0.1524" layer="91"/>
+<pinref part="U3" gate="G$1" pin="XOUT32/CLKSEL1"/>
+<junction x="226.06" y="124.46"/>
+<junction x="236.22" y="124.46"/>
+<label x="231.14" y="121.92" size="1.778" layer="95"/>
+</segment>
+<segment>
+<wire x1="175.26" y1="152.4" x2="165.1" y2="152.4" width="0.1524" layer="91"/>
+<pinref part="U3" gate="G$1" pin="CLKSEL0"/>
+<junction x="175.26" y="152.4"/>
+<junction x="165.1" y="152.4"/>
+<label x="152.4" y="152.4" size="1.778" layer="95"/>
+</segment>
+<segment>
+<wire x1="297.18" y1="121.92" x2="292.1" y2="121.92" width="0.1524" layer="91"/>
+<pinref part="OS2" gate="A" pin="VDD"/>
+<pinref part="C31" gate="G$1" pin="1"/>
+<wire x1="292.1" y1="121.92" x2="284.48" y2="121.92" width="0.1524" layer="91"/>
+<junction x="292.1" y="121.92"/>
+<junction x="284.48" y="121.92"/>
+<label x="297.18" y="119.38" size="1.778" layer="95"/>
+</segment>
+<segment>
+<wire x1="259.08" y1="121.92" x2="248.92" y2="121.92" width="0.1524" layer="91"/>
+<pinref part="OS2" gate="A" pin="CON"/>
+<junction x="259.08" y="121.92"/>
+<junction x="248.92" y="121.92"/>
+<label x="251.46" y="119.38" size="1.778" layer="95"/>
+</segment>
 </net>
 <net name="VSS" class="2">
@@
 <label x="91.44" y="147.32" size="1.778" layer="95"/>
 <junction x="93.98" y="137.16"/>
+<junction x="93.98" y="132.08"/>
 </segment>
 <segment>
@@
 <pinref part="VSS9" gate="G$1" pin="VSS"/>
 <junction x="96.52" y="139.7"/>
+<junction x="96.52" y="132.08"/>
 </segment>
 <segment>
@@
 <junction x="-71.12" y="-27.94"/>
 </segment>
+<segment>
+<wire x1="233.68" y1="116.84" x2="226.06" y2="116.84" width="0.1524" layer="91"/>
+<pinref part="U3" gate="G$1" pin="GNDIO"/>
+<junction x="226.06" y="116.84"/>
+<junction x="233.68" y="116.84"/>
+<label x="238.76" y="116.84" size="1.778" layer="95"/>
+</segment>
+<segment>
+<wire x1="231.14" y1="114.3" x2="226.06" y2="114.3" width="0.1524" layer="91"/>
+<pinref part="U3" gate="G$1" pin="GND"/>
+<junction x="226.06" y="114.3"/>
+<junction x="231.14" y="114.3"/>
+<label x="238.76" y="114.3" size="1.778" layer="95"/>
+</segment>
+<segment>
+<pinref part="C30" gate="G$1" pin="2"/>
+<pinref part="VSS60" gate="G$1" pin="VSS"/>
+<junction x="175.26" y="116.84"/>
+</segment>
+<segment>
+<wire x1="292.1" y1="132.08" x2="284.48" y2="132.08" width="0.1524" layer="91"/>
+<pinref part="OS2" gate="A" pin="VSS"/>
+<pinref part="C31" gate="G$1" pin="2"/>
+<wire x1="292.1" y1="129.54" x2="292.1" y2="132.08" width="0.1524" layer="91"/>
+<junction x="292.1" y="129.54"/>
+<junction x="292.1" y="132.08"/>
+<junction x="284.48" y="132.08"/>
+<label x="297.18" y="132.08" size="1.778" layer="95"/>
+</segment>
 </net>
 <net name="AVDD" class="2">
@@
 <junction x="-43.18" y="-33.02"/>
 </segment>
+<segment>
+<wire x1="162.56" y1="139.7" x2="165.1" y2="139.7" width="0.1524" layer="91"/>
+<pinref part="U3" gate="G$1" pin="!H_CS"/>
+<junction x="175.26" y="139.7"/>
+<junction x="165.1" y="139.7"/>
+<wire x1="165.1" y1="139.7" x2="175.26" y2="139.7" width="0.1524" layer="91"/>
+<junction x="162.56" y="139.7"/>
+<label x="149.86" y="139.7" size="1.778" layer="95"/>
+</segment>
 </net>
 <net name="N$3" class="0">
@@
 <junction x="17.78" y="-25.4"/>
 </segment>
+<segment>
+<wire x1="226.06" y1="147.32" x2="238.76" y2="147.32" width="0.1524" layer="91"/>
+<pinref part="U3" gate="G$1" pin="H_SCL/SCK/RX"/>
+<junction x="226.06" y="147.32"/>
+<junction x="238.76" y="147.32"/>
+<label x="243.84" y="147.32" size="1.778" layer="95"/>
+</segment>
 </net>
 <net name="SDO2" class="0">
@@
 <junction x="17.78" y="-22.86"/>
 </segment>
+<segment>
+<wire x1="175.26" y1="137.16" x2="162.56" y2="137.16" width="0.1524" layer="91"/>
+<pinref part="U3" gate="G$1" pin="SA0/H_MOSI"/>
+<junction x="175.26" y="137.16"/>
+<junction x="162.56" y="137.16"/>
+<label x="149.86" y="137.16" size="1.778" layer="95"/>
+</segment>
 </net>
 <net name="SDI2" class="0">
@@
 <junction x="-30.48" y="-35.56"/>
 <junction x="-43.18" y="-35.56"/>
+</segment>
+<segment>
+<wire x1="226.06" y1="144.78" x2="238.76" y2="144.78" width="0.1524" layer="91"/>
+<pinref part="U3" gate="G$1" pin="H_SDA/H_MISO/TX"/>
+<junction x="226.06" y="144.78"/>
+<junction x="238.76" y="144.78"/>
+<label x="243.84" y="144.78" size="1.778" layer="95"/>
 </segment>
 </net>
@@
 <label x="119.38" y="114.3" size="1.778" layer="95"/>
 </segment>
+<segment>
+<wire x1="226.06" y1="152.4" x2="254" y2="152.4" width="0.1524" layer="91"/>
+<pinref part="U3" gate="G$1" pin="!H_INT"/>
+<junction x="226.06" y="152.4"/>
+<junction x="254" y="152.4"/>
+<label x="256.54" y="152.4" size="1.778" layer="95"/>
+</segment>
 </net>
 <net name="N$6" class="0">
@@
 </segment>
 </net>
+<net name="N$14" class="0">
+<segment>
+<pinref part="U3" gate="G$1" pin="CAP"/>
+<pinref part="C30" gate="G$1" pin="1"/>
+<junction x="175.26" y="124.46"/>
+</segment>
+</net>
+<net name="32KHZ" class="0">
+<segment>
+<pinref part="U3" gate="G$1" pin="XIN32"/>
+<pinref part="OS2" gate="A" pin="OUT"/>
+<wire x1="226.06" y1="127" x2="259.08" y2="127" width="0.1524" layer="91"/>
+<junction x="259.08" y="127"/>
+<junction x="226.06" y="127"/>
+<label x="243.84" y="127" size="1.778" layer="95"/>
+</segment>
+</net>

Commit message: up
Parts:
- added C32: 0.1uf, rcl:C-USC0805
- added OSCI1: PTR1PAD1-13, testpad:PTR1PAD1-13
- added R8, R9: 10k, rcl:R-US_M0805
- added SJ3: BOOT_ON, jumper:SJ
- added SJ4: IMU_RESET, jumper:SJ
Connections:
- net RB15 renamed BUZZER1
- removed net BMA_INT2: IC1.INT2, TP3.TP, U1.PGD3/VREF-/OA2IN-/AN2/C2IN1-/RPB0/CTED2/RB0, U3.!H_INT
- new net N$16: R8.1, SJ3.2, U3.!BOOT
- new net N$17: C32.1, R9.1, SJ4.2, U3.!RST
- new net TP3_SIG_WAKE: IC1.INT2, TP3.TP, U1.PGD3/VREF-/OA2IN-/AN2/C2IN1-/RPB0/CTED2/RB0, U3.PS0/WAKE
- net 32KHZ: now also OSCI1.TP
- net EXT_INT2: now also U3.!H_INT
- net VDD: now also R8.2, R9.2, U3.PS1
- net VSS: now also C32.2, SJ3.1, SJ4.1
Changed lines of the file:
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@@
 <part name="OS2" library="IQD-Frequency-Products" library_urn="urn:adsk.eagle:library:90" deviceset="OSC-OE" device="-IQXO-793" package3d_urn="urn:adsk.eagle:package:3371/1"/>
 <part name="C31" library="rcl" library_urn="urn:adsk.eagle:library:334" deviceset="C-US" device="C0805" package3d_urn="urn:adsk.eagle:package:23617/2" value="0.1uf"/>
+<part name="OSCI1" library="testpad" library_urn="urn:adsk.eagle:library:385" deviceset="PTR1" device="PAD1-13" package3d_urn="urn:adsk.eagle:package:27946/1"/>
+<part name="R8" library="rcl" library_urn="urn:adsk.eagle:library:334" deviceset="R-US_" device="M0805" package3d_urn="urn:adsk.eagle:package:23556/2" value="10k"/>
+<part name="VSS61" library="supply1" library_urn="urn:adsk.eagle:library:371" deviceset="VSS" device=""/>
+<part name="SJ3" library="jumper" library_urn="urn:adsk.eagle:library:252" deviceset="SJ" device="" package3d_urn="urn:adsk.eagle:package:15471/1" value="BOOT_ON"/>
+<part name="R9" library="rcl" library_urn="urn:adsk.eagle:library:334" deviceset="R-US_" device="M0805" package3d_urn="urn:adsk.eagle:package:23556/2" value="10k"/>
+<part name="C32" library="rcl" library_urn="urn:adsk.eagle:library:334" deviceset="C-US" device="C0805" package3d_urn="urn:adsk.eagle:package:23617/2" value="0.1uf"/>
+<part name="VSS62" library="supply1" library_urn="urn:adsk.eagle:library:371" deviceset="VSS" device=""/>
+<part name="SJ4" library="jumper" library_urn="urn:adsk.eagle:library:252" deviceset="SJ" device="" package3d_urn="urn:adsk.eagle:package:15471/1" value="IMU_RESET"/>
+<part name="VSS63" library="supply1" library_urn="urn:adsk.eagle:library:371" deviceset="VSS" device=""/>
 </parts>
 <sheets>
@@
 <attribute name="NAME" x="291.084" y="123.825" size="1.778" layer="95" rot="R180"/>
 <attribute name="VALUE" x="291.084" y="128.651" size="1.778" layer="96" rot="R180"/>
+</instance>
+<instance part="OSCI1" gate="G$1" x="231.14" y="129.54" smashed="yes" rot="R180">
+<attribute name="NAME" x="232.156" y="135.89" size="1.778" layer="95" rot="R270"/>
+<attribute name="TP_SIGNAL_NAME" x="229.87" y="132.08" size="1.778" layer="97" rot="R180"/>
+</instance>
+<instance part="R8" gate="G$1" x="139.7" y="149.86" smashed="yes" rot="R90">
+<attribute name="NAME" x="138.2014" y="146.05" size="1.778" layer="95" rot="R90"/>
+<attribute name="VALUE" x="143.002" y="146.05" size="1.778" layer="96" rot="R90"/>
+</instance>
+<instance part="VSS61" gate="G$1" x="139.7" y="132.08" smashed="yes">
+<attribute name="VALUE" x="142.24" y="129.54" size="1.778" layer="96" rot="R180"/>
+</instance>
+<instance part="SJ3" gate="1" x="139.7" y="139.7" smashed="yes" rot="R90">
+<attribute name="NAME" x="129.54" y="142.24" size="1.778" layer="95" rot="R180"/>
+<attribute name="VALUE" x="137.16" y="138.43" size="1.778" layer="96" rot="R180"/>
+</instance>
+<instance part="R9" gate="G$1" x="147.32" y="157.48" smashed="yes" rot="R90">
+<attribute name="NAME" x="145.8214" y="153.67" size="1.778" layer="95" rot="R90"/>
+<attribute name="VALUE" x="150.622" y="153.67" size="1.778" layer="96" rot="R90"/>
+</instance>
+<instance part="C32" gate="G$1" x="149.86" y="152.4" smashed="yes" rot="R90">
+<attribute name="NAME" x="149.225" y="153.416" size="1.778" layer="95" rot="R90"/>
+<attribute name="VALUE" x="154.051" y="153.416" size="1.778" layer="96" rot="R90"/>
+</instance>
+<instance part="VSS62" gate="G$1" x="157.48" y="152.4" smashed="yes" rot="R90">
+<attribute name="VALUE" x="160.02" y="154.94" size="1.778" layer="96" rot="R270"/>
+</instance>
+<instance part="SJ4" gate="1" x="121.92" y="154.94" smashed="yes" rot="R90">
+<attribute name="NAME" x="111.76" y="157.48" size="1.778" layer="95" rot="R180"/>
+<attribute name="VALUE" x="119.38" y="153.67" size="1.778" layer="96" rot="R180"/>
+</instance>
+<instance part="VSS63" gate="G$1" x="121.92" y="147.32" smashed="yes">
+<attribute name="VALUE" x="124.46" y="144.78" size="1.778" layer="96" rot="R180"/>
 </instance>
 </instances>
@@
 <junction x="165.1" y="152.4"/>
 <label x="152.4" y="152.4" size="1.778" layer="95"/>
+<label x="167.64" y="152.4" size="1.778" layer="95"/>
 </segment>
 <segment>
@@
 <junction x="248.92" y="121.92"/>
 <label x="251.46" y="119.38" size="1.778" layer="95"/>
+</segment>
+<segment>
+<wire x1="175.26" y1="129.54" x2="165.1" y2="129.54" width="0.1524" layer="91"/>
+<pinref part="U3" gate="G$1" pin="PS1"/>
+<junction x="175.26" y="129.54"/>
+<junction x="165.1" y="129.54"/>
+<label x="152.4" y="129.54" size="1.778" layer="95"/>
+</segment>
+<segment>
+<wire x1="139.7" y1="154.94" x2="129.54" y2="154.94" width="0.1524" layer="91"/>
+<pinref part="R8" gate="G$1" pin="2"/>
+<junction x="139.7" y="154.94"/>
+<junction x="129.54" y="154.94"/>
+<label x="129.54" y="152.4" size="1.778" layer="95"/>
+</segment>
+<segment>
+<wire x1="147.32" y1="162.56" x2="137.16" y2="162.56" width="0.1524" layer="91"/>
+<pinref part="R9" gate="G$1" pin="2"/>
+<junction x="137.16" y="162.56"/>
+<junction x="147.32" y="162.56"/>
+<label x="127" y="162.56" size="1.778" layer="95"/>
 </segment>
 </net>
@@
 <label x="297.18" y="132.08" size="1.778" layer="95"/>
 </segment>
+<segment>
+<pinref part="SJ3" gate="1" pin="1"/>
+<pinref part="VSS61" gate="G$1" pin="VSS"/>
+<junction x="139.7" y="134.62"/>
+</segment>
+<segment>
+<pinref part="C32" gate="G$1" pin="2"/>
+<pinref part="VSS62" gate="G$1" pin="VSS"/>
+<junction x="154.94" y="152.4"/>
+</segment>
+<segment>
+<pinref part="SJ4" gate="1" pin="1"/>
+<pinref part="VSS63" gate="G$1" pin="VSS"/>
+<junction x="121.92" y="149.86"/>
+</segment>
 </net>
 <net name="AVDD" class="2">
@@
 <junction x="121.92" y="111.76"/>
 <label x="116.84" y="109.22" size="1.778" layer="95"/>
+</segment>
+<segment>
+<wire x1="226.06" y1="152.4" x2="238.76" y2="152.4" width="0.1524" layer="91"/>
+<pinref part="U3" gate="G$1" pin="!H_INT"/>
+<junction x="226.06" y="152.4"/>
+<junction x="238.76" y="152.4"/>
+<label x="246.38" y="152.4" size="1.778" layer="95"/>
 </segment>
 </net>
@@
 </segment>
 </net>
-<net name="RB15" class="0">
+<net name="BUZZER1" class="0">
 <segment>
 <pinref part="U1" gate="A" pin="RPB15/PWM1L/RB15"/>
@@
 </segment>
 </net>
-<net name="BMA_INT2" class="0">
+<net name="TP3_SIG_WAKE" class="0">
 <segment>
 <pinref part="U1" gate="A" pin="PGD3/VREF-/OA2IN-/AN2/C2IN1-/RPB0/CTED2/RB0"/>
@@
 </segment>
 <segment>
-<wire x1="226.06" y1="152.4" x2="254" y2="152.4" width="0.1524" layer="91"/>
-<pinref part="U3" gate="G$1" pin="!H_INT"/>
-<junction x="226.06" y="152.4"/>
-<junction x="254" y="152.4"/>
-<label x="256.54" y="152.4" size="1.778" layer="95"/>
+<wire x1="147.32" y1="132.08" x2="175.26" y2="132.08" width="0.1524" layer="91"/>
+<pinref part="U3" gate="G$1" pin="PS0/WAKE"/>
+<junction x="175.26" y="132.08"/>
+<junction x="147.32" y="132.08"/>
+<label x="149.86" y="132.08" size="1.778" layer="95"/>
 </segment>
 </net>
@@
 <pinref part="U3" gate="G$1" pin="XIN32"/>
 <pinref part="OS2" gate="A" pin="OUT"/>
-<wire x1="226.06" y1="127" x2="259.08" y2="127" width="0.1524" layer="91"/>
+<wire x1="226.06" y1="127" x2="231.14" y2="127" width="0.1524" layer="91"/>
 <junction x="259.08" y="127"/>
 <junction x="226.06" y="127"/>
 <label x="243.84" y="127" size="1.778" layer="95"/>
-</segment>
-</net>
+<wire x1="231.14" y1="127" x2="259.08" y2="127" width="0.1524" layer="91"/>
+<pinref part="OSCI1" gate="G$1" pin="TP"/>
+<junction x="231.14" y="127"/>
+</segment>
+</net>
+<net name="N$16" class="0">
+<segment>
+<pinref part="U3" gate="G$1" pin="!BOOT"/>
+<wire x1="175.26" y1="144.78" x2="139.7" y2="144.78" width="0.1524" layer="91"/>
+<pinref part="R8" gate="G$1" pin="1"/>
+<pinref part="SJ3" gate="1" pin="2"/>
+<junction x="139.7" y="144.78"/>
+<junction x="175.26" y="144.78"/>
+</segment>
+</net>
+<net name="N$17" class="0">
+<segment>
+<pinref part="R9" gate="G$1" pin="1"/>
+<pinref part="C32" gate="G$1" pin="1"/>
+<wire x1="147.32" y1="152.4" x2="147.32" y2="147.32" width="0.1524" layer="91"/>
+<junction x="147.32" y="152.4"/>
+<pinref part="U3" gate="G$1" pin="!RST"/>
+<wire x1="147.32" y1="147.32" x2="175.26" y2="147.32" width="0.1524" layer="91"/>
+<junction x="175.26" y="147.32"/>
+<wire x1="147.32" y1="152.4" x2="142.24" y2="152.4" width="0.1524" layer="91"/>
+<wire x1="142.24" y1="152.4" x2="142.24" y2="160.02" width="0.1524" layer="91"/>
+<pinref part="SJ4" gate="1" pin="2"/>
+<wire x1="142.24" y1="160.02" x2="121.92" y2="160.02" width="0.1524" layer="91"/>
+<junction x="121.92" y="160.02"/>
+</segment>
+</net>
