File: ll-tester.sch (EAGLE design)
At the start: 116 parts, among them IC1 BMA490L, IC2 TCAN330GD, IC3 EM14R0D-R20-L064S, IC4 CAT4238TD-GT3, U1 PIC32MK0512MCJ048T-I/Y8XTQFP4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, U2 MAX6126B30, U3 BNO080

Commit message: p
Parts:
- added DISP_SIGS: DISP-SIG, pinhead:PINHD-1X2
- added GLORY: GLORY, pinhead:PINHD-1X2
- added SJ7: IMU_R_SIG, jumper:SJ
- SV3: value MISC0 -> MISC_SIG
Connections:
- new net MISC_0: DISP_SIGS.1, SJ5.3
- net DIS_RESET: now also DISP_SIGS.2, SJ7.2
- net INDX2: no longer SJ5.3
- net N$17: now also SJ7.1
- net VDD: now also GLORY.1, GLORY.2
Changed lines of the file:
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@@
 <part name="LS1" library="CMI-9705-0380-SMT-TR" deviceset="CMI-9705-0380-SMT-TR" device=""/>
 <part name="VSS55" library="supply1" library_urn="urn:adsk.eagle:library:371" deviceset="VSS" device=""/>
-<part name="SV3" library="con-lstb" library_urn="urn:adsk.eagle:library:162" deviceset="MA10-1" device="" package3d_urn="urn:adsk.eagle:package:8346/1" value="MISC0"/>
+<part name="SV3" library="con-lstb" library_urn="urn:adsk.eagle:library:162" deviceset="MA10-1" device="" package3d_urn="urn:adsk.eagle:package:8346/1" value="MISC_SIG"/>
 <part name="VSS56" library="supply1" library_urn="urn:adsk.eagle:library:371" deviceset="VSS" device=""/>
 <part name="VDD4" library="supply1" library_urn="urn:adsk.eagle:library:371" deviceset="VDD" device=""/>
@@
 <part name="SJ4" library="jumper" library_urn="urn:adsk.eagle:library:252" deviceset="SJ" device="" package3d_urn="urn:adsk.eagle:package:15471/1" value="IMU_RESET"/>
 <part name="VSS63" library="supply1" library_urn="urn:adsk.eagle:library:371" deviceset="VSS" device=""/>
+<part name="SJ7" library="jumper" library_urn="urn:adsk.eagle:library:252" deviceset="SJ" device="" package3d_urn="urn:adsk.eagle:package:15471/1" value="IMU_R_SIG"/>
+<part name="DISP_SIGS" library="pinhead" library_urn="urn:adsk.eagle:library:325" deviceset="PINHD-1X2" device="" package3d_urn="urn:adsk.eagle:package:22435/2" value="DISP-SIG"/>
+<part name="GLORY" library="pinhead" library_urn="urn:adsk.eagle:library:325" deviceset="PINHD-1X2" device="" package3d_urn="urn:adsk.eagle:package:22435/2" value="GLORY"/>
 </parts>
 <sheets>
@@
 <attribute name="VALUE" x="124.46" y="144.78" size="1.778" layer="96" rot="R180"/>
 </instance>
+<instance part="SJ7" gate="1" x="116.84" y="160.02" smashed="yes" rot="R180">
+<attribute name="NAME" x="114.3" y="149.86" size="1.778" layer="95" rot="R270"/>
+<attribute name="VALUE" x="109.22" y="166.37" size="1.778" layer="96"/>
+</instance>
+<instance part="DISP_SIGS" gate="G$1" x="43.18" y="-101.6" smashed="yes">
+<attribute name="NAME" x="36.83" y="-95.885" size="1.778" layer="95"/>
+<attribute name="VALUE" x="36.83" y="-106.68" size="1.778" layer="96"/>
+</instance>
+<instance part="GLORY" gate="G$1" x="160.02" y="-83.82" smashed="yes">
+<attribute name="NAME" x="153.67" y="-78.105" size="1.778" layer="95"/>
+<attribute name="VALUE" x="153.67" y="-88.9" size="1.778" layer="96"/>
+</instance>
 </instances>
 <busses>
@@
 <label x="127" y="162.56" size="1.778" layer="95"/>
 </segment>
+<segment>
+<wire x1="149.86" y1="-81.28" x2="157.48" y2="-81.28" width="0.1524" layer="91"/>
+<pinref part="GLORY" gate="G$1" pin="1"/>
+<junction x="157.48" y="-81.28"/>
+<junction x="149.86" y="-81.28"/>
+<label x="142.24" y="-81.28" size="1.778" layer="95"/>
+</segment>
+<segment>
+<wire x1="149.86" y1="-83.82" x2="157.48" y2="-83.82" width="0.1524" layer="91"/>
+<pinref part="GLORY" gate="G$1" pin="2"/>
+<junction x="157.48" y="-83.82"/>
+<junction x="149.86" y="-83.82"/>
+<label x="142.24" y="-83.82" size="1.778" layer="95"/>
+</segment>
 </net>
 <net name="VSS" class="2">
@@
 <junction x="30.48" y="-121.92"/>
 </segment>
+<segment>
+<wire x1="99.06" y1="160.02" x2="111.76" y2="160.02" width="0.1524" layer="91"/>
+<pinref part="SJ7" gate="1" pin="2"/>
+<junction x="111.76" y="160.02"/>
+<junction x="99.06" y="160.02"/>
+<label x="83.82" y="160.02" size="1.778" layer="95"/>
+</segment>
+<segment>
+<wire x1="27.94" y1="-101.6" x2="40.64" y2="-101.6" width="0.1524" layer="91"/>
+<pinref part="DISP_SIGS" gate="G$1" pin="2"/>
+<junction x="40.64" y="-101.6"/>
+<junction x="27.94" y="-101.6"/>
+<label x="12.7" y="-101.6" size="1.778" layer="95"/>
+</segment>
 </net>
 <net name="SDI1" class="0">
@@
 </segment>
 <segment>
-<wire x1="30.48" y1="-114.3" x2="43.18" y2="-114.3" width="0.1524" layer="91"/>
-<label x="15.24" y="-114.3" size="1.778" layer="95"/>
-<junction x="43.18" y="-114.3"/>
-<junction x="30.48" y="-114.3"/>
-</segment>
-<segment>
 <wire x1="27.94" y1="-71.12" x2="40.64" y2="-71.12" width="0.1524" layer="91"/>
 <pinref part="IC3" gate="G$1" pin="CHANNEL_A"/>
@@
 <junction x="-43.18" y="0"/>
 </segment>
-<segment>
-<pinref part="SJ5" gate="G$1" pin="3"/>
-<wire x1="111.76" y1="-172.72" x2="104.14" y2="-172.72" width="0.1524" layer="91"/>
-<wire x1="104.14" y1="-172.72" x2="104.14" y2="-170.18" width="0.1524" layer="91"/>
-<wire x1="104.14" y1="-170.18" x2="78.74" y2="-170.18" width="0.1524" layer="91"/>
-<wire x1="78.74" y1="-170.18" x2="78.74" y2="-111.76" width="0.1524" layer="91"/>
-<wire x1="78.74" y1="-111.76" x2="43.18" y2="-111.76" width="0.1524" layer="91"/>
-<junction x="43.18" y="-111.76"/>
-<wire x1="30.48" y1="-111.76" x2="43.18" y2="-111.76" width="0.1524" layer="91"/>
-<junction x="30.48" y="-111.76"/>
-<label x="15.24" y="-111.76" size="1.778" layer="95"/>
-<label x="88.9" y="-170.18" size="1.778" layer="95"/>
-<junction x="111.76" y="-172.72"/>
-</segment>
 </net>
 <net name="BUZZER1" class="0">
@@
 <wire x1="142.24" y1="160.02" x2="121.92" y2="160.02" width="0.1524" layer="91"/>
 <junction x="121.92" y="160.02"/>
+<pinref part="SJ7" gate="1" pin="1"/>
+</segment>
+</net>
+<net name="MISC_0" class="0">
+<segment>
+<pinref part="SJ5" gate="G$1" pin="3"/>
+<wire x1="111.76" y1="-172.72" x2="81.28" y2="-172.72" width="0.1524" layer="91"/>
+<wire x1="81.28" y1="-172.72" x2="81.28" y2="-111.76" width="0.1524" layer="91"/>
+<wire x1="81.28" y1="-111.76" x2="43.18" y2="-111.76" width="0.1524" layer="91"/>
+<junction x="111.76" y="-172.72"/>
+<junction x="43.18" y="-111.76"/>
+<wire x1="30.48" y1="-111.76" x2="43.18" y2="-111.76" width="0.1524" layer="91"/>
+<junction x="30.48" y="-111.76"/>
+<label x="15.24" y="-111.76" size="1.778" layer="95"/>
+<label x="91.44" y="-172.72" size="1.778" layer="95"/>
+</segment>
+<segment>
+<wire x1="27.94" y1="-99.06" x2="40.64" y2="-99.06" width="0.1524" layer="91"/>
+<pinref part="DISP_SIGS" gate="G$1" pin="1"/>
+<junction x="40.64" y="-99.06"/>
+<junction x="27.94" y="-99.06"/>
+<label x="17.78" y="-99.06" size="1.778" layer="95"/>
 </segment>
 </net>

Commit message: up
Parts:
- added R10, R11: 10k, rcl:R-US_M0805
- added SV4: IMU_SIG, con-lstb:MA10-1
Connections:
- new net BNO_CHIP_RESET: C32.1, R9.1, SJ4.2, SJ7.1, SV4.8, U3.!RST
- new net N$18: R11.2, U3.ENV_SCL
- net 32KHZ: now also SV4.9
- net EXT_INT2: now also SV4.6
- net IMU_CS: now also SV4.2
- net N$17: now also R10.2, U3.ENV_SDA; no longer C32.1, R9.1, SJ4.2, SJ7.1, U3.!RST
- net RED_LED: now also SV4.7
- net SCK2: now also SV4.3
- net SDI2: now also SV4.4
- net SDO2: now also SV4.5
- net TP3_SIG_WAKE: now also SV4.10
- net VDD: now also R10.1, R11.1
- net VSS: now also SV4.1
Other:
- moved on the sheet: OSCI1
Changed lines of the file:
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@@
 <part name="DISP_SIGS" library="pinhead" library_urn="urn:adsk.eagle:library:325" deviceset="PINHD-1X2" device="" package3d_urn="urn:adsk.eagle:package:22435/2" value="DISP-SIG"/>
 <part name="GLORY" library="pinhead" library_urn="urn:adsk.eagle:library:325" deviceset="PINHD-1X2" device="" package3d_urn="urn:adsk.eagle:package:22435/2" value="GLORY"/>
+<part name="SV4" library="con-lstb" library_urn="urn:adsk.eagle:library:162" deviceset="MA10-1" device="" package3d_urn="urn:adsk.eagle:package:8346/1" value="IMU_SIG"/>
+<part name="VSS64" library="supply1" library_urn="urn:adsk.eagle:library:371" deviceset="VSS" device=""/>
+<part name="R10" library="rcl" library_urn="urn:adsk.eagle:library:334" deviceset="R-US_" device="M0805" package3d_urn="urn:adsk.eagle:package:23556/2" value="10k"/>
+<part name="R11" library="rcl" library_urn="urn:adsk.eagle:library:334" deviceset="R-US_" device="M0805" package3d_urn="urn:adsk.eagle:package:23556/2" value="10k"/>
+<part name="VDD19" library="supply1" library_urn="urn:adsk.eagle:library:371" deviceset="VDD" device=""/>
+<part name="VDD24" library="supply1" library_urn="urn:adsk.eagle:library:371" deviceset="VDD" device=""/>
 </parts>
 <sheets>
@@
 <attribute name="VALUE" x="291.084" y="128.651" size="1.778" layer="96" rot="R180"/>
 </instance>
-<instance part="OSCI1" gate="G$1" x="231.14" y="129.54" smashed="yes" rot="R180">
-<attribute name="NAME" x="232.156" y="135.89" size="1.778" layer="95" rot="R270"/>
-<attribute name="TP_SIGNAL_NAME" x="229.87" y="132.08" size="1.778" layer="97" rot="R180"/>
+<instance part="OSCI1" gate="G$1" x="238.76" y="129.54" smashed="yes" rot="R180">
+<attribute name="NAME" x="239.776" y="135.89" size="1.778" layer="95" rot="R270"/>
+<attribute name="TP_SIGNAL_NAME" x="237.49" y="132.08" size="1.778" layer="97" rot="R180"/>
 </instance>
 <instance part="R8" gate="G$1" x="139.7" y="149.86" smashed="yes" rot="R90">
@@
 <attribute name="VALUE" x="153.67" y="-88.9" size="1.778" layer="96"/>
 </instance>
+<instance part="SV4" gate="1" x="248.92" y="86.36" smashed="yes">
+<attribute name="VALUE" x="247.65" y="71.12" size="1.778" layer="96"/>
+<attribute name="NAME" x="247.65" y="102.362" size="1.778" layer="95"/>
+</instance>
+<instance part="VSS64" gate="G$1" x="256.54" y="73.66" smashed="yes">
+<attribute name="VALUE" x="254" y="68.58" size="1.778" layer="96" rot="R90"/>
+</instance>
+<instance part="R10" gate="G$1" x="231.14" y="137.16" smashed="yes" rot="R180">
+<attribute name="NAME" x="229.87" y="135.6614" size="1.778" layer="95" rot="R180"/>
+<attribute name="VALUE" x="234.95" y="135.382" size="1.778" layer="96" rot="R180"/>
+</instance>
+<instance part="R11" gate="G$1" x="231.14" y="139.7" smashed="yes" rot="R180">
+<attribute name="NAME" x="229.87" y="143.2814" size="1.778" layer="95" rot="R180"/>
+<attribute name="VALUE" x="234.95" y="143.002" size="1.778" layer="96" rot="R180"/>
+</instance>
+<instance part="VDD19" gate="G$1" x="238.76" y="139.7" smashed="yes" rot="R270">
+<attribute name="VALUE" x="236.22" y="142.24" size="1.778" layer="96"/>
+</instance>
+<instance part="VDD24" gate="G$1" x="238.76" y="137.16" smashed="yes" rot="R270">
+<attribute name="VALUE" x="236.22" y="139.7" size="1.778" layer="96"/>
+</instance>
 </instances>
 <busses>
@@
 <label x="142.24" y="-83.82" size="1.778" layer="95"/>
 </segment>
+<segment>
+<pinref part="R11" gate="G$1" pin="1"/>
+<pinref part="VDD19" gate="G$1" pin="VDD"/>
+<junction x="236.22" y="139.7"/>
+</segment>
+<segment>
+<pinref part="R10" gate="G$1" pin="1"/>
+<pinref part="VDD24" gate="G$1" pin="VDD"/>
+<junction x="236.22" y="137.16"/>
+</segment>
 </net>
 <net name="VSS" class="2">
@@
 <junction x="121.92" y="149.86"/>
 </segment>
+<segment>
+<pinref part="SV4" gate="1" pin="1"/>
+<pinref part="VSS64" gate="G$1" pin="VSS"/>
+<junction x="256.54" y="76.2"/>
+</segment>
 </net>
 <net name="AVDD" class="2">
@@
 <junction x="15.24" y="101.6"/>
 </segment>
+<segment>
+<wire x1="269.24" y1="91.44" x2="256.54" y2="91.44" width="0.1524" layer="91"/>
+<pinref part="SV4" gate="1" pin="7"/>
+<label x="264.16" y="91.44" size="1.778" layer="95"/>
+<junction x="256.54" y="91.44"/>
+</segment>
 </net>
 <net name="IMU_CS" class="0">
@@
 <label x="149.86" y="139.7" size="1.778" layer="95"/>
 </segment>
+<segment>
+<wire x1="256.54" y1="78.74" x2="266.7" y2="78.74" width="0.1524" layer="91"/>
+<pinref part="SV4" gate="1" pin="2"/>
+<label x="259.08" y="78.74" size="1.778" layer="95"/>
+<junction x="256.54" y="78.74"/>
+</segment>
 </net>
 <net name="N$3" class="0">
@@
 <label x="243.84" y="147.32" size="1.778" layer="95"/>
 </segment>
+<segment>
+<wire x1="256.54" y1="81.28" x2="269.24" y2="81.28" width="0.1524" layer="91"/>
+<pinref part="SV4" gate="1" pin="3"/>
+<label x="259.08" y="81.28" size="1.778" layer="95"/>
+<junction x="256.54" y="81.28"/>
+</segment>
 </net>
 <net name="SDO2" class="0">
@@
 <label x="149.86" y="137.16" size="1.778" layer="95"/>
 </segment>
+<segment>
+<wire x1="269.24" y1="86.36" x2="256.54" y2="86.36" width="0.1524" layer="91"/>
+<pinref part="SV4" gate="1" pin="5"/>
+<label x="259.08" y="86.36" size="1.778" layer="95"/>
+<junction x="256.54" y="86.36"/>
+</segment>
 </net>
 <net name="SDI2" class="0">
@@
 <label x="243.84" y="144.78" size="1.778" layer="95"/>
 </segment>
+<segment>
+<wire x1="256.54" y1="83.82" x2="269.24" y2="83.82" width="0.1524" layer="91"/>
+<pinref part="SV4" gate="1" pin="4"/>
+<label x="259.08" y="83.82" size="1.778" layer="95"/>
+<junction x="256.54" y="83.82"/>
+</segment>
 </net>
 <net name="EXT_INT2" class="0">
@@
 <label x="246.38" y="152.4" size="1.778" layer="95"/>
 </segment>
+<segment>
+<wire x1="256.54" y1="88.9" x2="269.24" y2="88.9" width="0.1524" layer="91"/>
+<pinref part="SV4" gate="1" pin="6"/>
+<label x="259.08" y="88.9" size="1.778" layer="95"/>
+<junction x="256.54" y="88.9"/>
+</segment>
 </net>
 <net name="PGD_C1TX" class="0">
@@
 <label x="149.86" y="132.08" size="1.778" layer="95"/>
 </segment>
+<segment>
+<wire x1="256.54" y1="99.06" x2="284.48" y2="99.06" width="0.1524" layer="91"/>
+<pinref part="SV4" gate="1" pin="10"/>
+<label x="276.86" y="99.06" size="1.778" layer="95"/>
+<junction x="256.54" y="99.06"/>
+</segment>
 </net>
 <net name="N$6" class="0">
@@
 <pinref part="U3" gate="G$1" pin="XIN32"/>
 <pinref part="OS2" gate="A" pin="OUT"/>
-<wire x1="226.06" y1="127" x2="231.14" y2="127" width="0.1524" layer="91"/>
+<wire x1="226.06" y1="127" x2="238.76" y2="127" width="0.1524" layer="91"/>
 <junction x="259.08" y="127"/>
 <junction x="226.06" y="127"/>
 <label x="243.84" y="127" size="1.778" layer="95"/>
-<wire x1="231.14" y1="127" x2="259.08" y2="127" width="0.1524" layer="91"/>
+<wire x1="238.76" y1="127" x2="259.08" y2="127" width="0.1524" layer="91"/>
 <pinref part="OSCI1" gate="G$1" pin="TP"/>
-<junction x="231.14" y="127"/>
+<junction x="238.76" y="127"/>
+</segment>
+<segment>
+<wire x1="256.54" y1="96.52" x2="284.48" y2="96.52" width="0.1524" layer="91"/>
+<pinref part="SV4" gate="1" pin="9"/>
+<label x="276.86" y="96.52" size="1.778" layer="95"/>
+<junction x="256.54" y="96.52"/>
 </segment>
 </net>
@@
 </segment>
 </net>
-<net name="N$17" class="0">
+<net name="BNO_CHIP_RESET" class="0">
 <segment>
 <pinref part="R9" gate="G$1" pin="1"/>
@@
 <junction x="121.92" y="160.02"/>
 <pinref part="SJ7" gate="1" pin="1"/>
+<label x="149.86" y="147.32" size="1.778" layer="95"/>
+</segment>
+<segment>
+<wire x1="256.54" y1="93.98" x2="284.48" y2="93.98" width="0.1524" layer="91"/>
+<pinref part="SV4" gate="1" pin="8"/>
+<label x="276.86" y="93.98" size="1.778" layer="95"/>
+<junction x="256.54" y="93.98"/>
 </segment>
 </net>
@@
 </segment>
 </net>
+<net name="N$17" class="0">
+<segment>
+<pinref part="U3" gate="G$1" pin="ENV_SDA"/>
+<pinref part="R10" gate="G$1" pin="2"/>
+<junction x="226.06" y="137.16"/>
+</segment>
+</net>
+<net name="N$18" class="0">
+<segment>
+<pinref part="U3" gate="G$1" pin="ENV_SCL"/>
+<pinref part="R11" gate="G$1" pin="2"/>
+<junction x="226.06" y="139.7"/>
+</segment>
+</net>
