File: ll-tester.sch (EAGLE design)
At the start: 122 parts, among them IC1 BMA490L, IC2 TCAN330GD, IC3 EM14R0D-R20-L064S, IC4 CAT4238TD-GT3, U1 PIC32MK0512MCJ048T-I/Y8XTQFP4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, U2 MAX6126B30, U3 BNO080

Commit message: up
Parts:
- added PS1: MYRBP500080B21RE, MYRBP500080B21RE:MYRBP500080B21RE
- added PS2: MYRLP330015F21RE, MYRLP330015F21RE:MYRLP330015F21RE
Changed lines of the file:
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@@
 <part name="VDD19" library="supply1" library_urn="urn:adsk.eagle:library:371" deviceset="VDD" device=""/>
 <part name="VDD24" library="supply1" library_urn="urn:adsk.eagle:library:371" deviceset="VDD" device=""/>
+<part name="PS1" library="MYRBP500080B21RE" deviceset="MYRBP500080B21RE" device=""/>
+<part name="PS2" library="MYRLP330015F21RE" deviceset="MYRLP330015F21RE" device=""/>
 </parts>
 <sheets>
@@
 <attribute name="VALUE" x="236.22" y="139.7" size="1.778" layer="96"/>
 </instance>
+<instance part="PS1" gate="G$1" x="220.98" y="-96.52" smashed="yes">
+<attribute name="NAME" x="240.03" y="-78.74" size="1.778" layer="95" align="center-left"/>
+<attribute name="VALUE" x="240.03" y="-81.28" size="1.778" layer="96" align="center-left"/>
+</instance>
+<instance part="PS2" gate="G$1" x="220.98" y="-149.86" smashed="yes">
+<attribute name="NAME" x="240.03" y="-132.08" size="1.778" layer="95" align="center-left"/>
+<attribute name="VALUE" x="240.03" y="-134.62" size="1.778" layer="96" align="center-left"/>
+</instance>
 </instances>

Commit message: up
Parts:
- added +5VDC: +5VDC, pinhead:PINHD-1X2
- added C33, C44: 10uf, rcl:C-USC0805
- added SJ8: BLANK_ON, jumper:SJ
Connections:
- removed net DC_INPUT: 3.3VDC.VI, C20.1, C21.1, R6.1
- new net +5V: +5VDC.1, +5VDC.2, C33.1, IC3.POWER_(+), PS1.VOUT
- new net N$20: PS2.L1, PS2.LX
- new net N$23: PS1.L2, PS1.LX
- new net V+: 3.3VDC.VI, C20.1, C21.1, PS2.CE, PS2.VIN, R6.1
- net MISC_0: now also SJ8.1
- net RB11: now also SJ8.2
- net VDD: now also C44.1, PS1.CE, PS1.L1, PS1.VBAT, PS2.L2, PS2.VOUT; no longer IC3.POWER_(+)
- net VSS: now also C33.2, C44.2, PS1.EP, PS1.GND_1, PS1.GND_2, PS2.EP, PS2.GND_1, PS2.GND_2
Other:
- moved on the sheet: PS1
