File: ll-tester.sch (EAGLE design)
At the start: 128 parts, among them IC1 BMA490L, IC2 TCAN330GD, IC3 EM14R0D-R20-L064S, IC4 CAT4238TD-GT3, U1 PIC32MK0512MCJ048T-I/Y8XTQFP4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, U2 MAX6126B30, U3 BNO080

Commit message: up
Parts:
- added C45, C46: 0.1uf, rcl:C-USC0805
- added C47: 10uf, rcl:C-USC0805
- added U4: BME280, BME280:BME280
- added U5: VCNL4040M3OE, VCNL4040M3OE:VCNL4040M3OE
Connections:
- removed net N$17: R10.2, U3.ENV_SDA
- removed net N$18: R11.2, U3.ENV_SCL
- new net BSCL: R11.2, U3.ENV_SCL, U4.SCK, U5.SCL
- new net BSDA: R10.2, U3.ENV_SDA, U4.SDI, U5.SDA
- new net N$22: U5.C-LED, U5.C-SENSOR
- net VDD: now also C45.1, C46.1, C47.1, U4.CSB, U4.VDD, U4.VDDIO, U5.VDD, U5.VDD-LED
- net VSS: now also C45.2, C46.2, C47.2, U4.GND, U5.GND
Changed lines of the file:
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@@
 <part name="+5VDC" library="pinhead" library_urn="urn:adsk.eagle:library:325" deviceset="PINHD-1X2" device="" package3d_urn="urn:adsk.eagle:package:22435/2" value="+5VDC"/>
 <part name="P+3" library="supply1" library_urn="urn:adsk.eagle:library:371" deviceset="+5V" device=""/>
+<part name="U4" library="BME280" deviceset="BME280" device=""/>
+<part name="U5" library="VCNL4040M3OE" deviceset="VCNL4040M3OE" device=""/>
+<part name="VSS73" library="supply1" library_urn="urn:adsk.eagle:library:371" deviceset="VSS" device=""/>
+<part name="VSS74" library="supply1" library_urn="urn:adsk.eagle:library:371" deviceset="VSS" device=""/>
+<part name="C45" library="rcl" library_urn="urn:adsk.eagle:library:334" deviceset="C-US" device="C0805" package3d_urn="urn:adsk.eagle:package:23617/2" value="0.1uf"/>
+<part name="VSS75" library="supply1" library_urn="urn:adsk.eagle:library:371" deviceset="VSS" device=""/>
+<part name="C46" library="rcl" library_urn="urn:adsk.eagle:library:334" deviceset="C-US" device="C0805" package3d_urn="urn:adsk.eagle:package:23617/2" value="0.1uf"/>
+<part name="VSS76" library="supply1" library_urn="urn:adsk.eagle:library:371" deviceset="VSS" device=""/>
+<part name="C47" library="rcl" library_urn="urn:adsk.eagle:library:334" deviceset="C-US" device="C0805" package3d_urn="urn:adsk.eagle:package:23617/2" value="10uf"/>
+<part name="VSS77" library="supply1" library_urn="urn:adsk.eagle:library:371" deviceset="VSS" device=""/>
 </parts>
 <sheets>
@@
 <attribute name="VALUE" x="208.28" y="-55.88" size="1.778" layer="96"/>
 </instance>
+<instance part="U4" gate="G$1" x="287.02" y="43.18" smashed="yes">
+<attribute name="NAME" x="276.8538" y="56.5231" size="1.786590625" layer="95"/>
+<attribute name="VALUE" x="276.8517" y="27.9276" size="1.782940625" layer="96"/>
+</instance>
+<instance part="U5" gate="_VCNL4040" x="294.64" y="-2.54" smashed="yes">
+<attribute name="NAME" x="289.552159375" y="11.4515" size="1.780740625" layer="95"/>
+<attribute name="VALUE" x="289.55508125" y="-17.7948" size="1.77971875" layer="96"/>
+</instance>
+<instance part="VSS73" gate="G$1" x="276.86" y="7.62" smashed="yes" rot="R180">
+<attribute name="VALUE" x="279.4" y="12.7" size="1.778" layer="96" rot="R270"/>
+</instance>
+<instance part="VSS74" gate="G$1" x="302.26" y="30.48" smashed="yes">
+<attribute name="VALUE" x="299.72" y="25.4" size="1.778" layer="96" rot="R90"/>
+</instance>
+<instance part="C45" gate="G$1" x="312.42" y="55.88" smashed="yes">
+<attribute name="NAME" x="313.436" y="56.515" size="1.778" layer="95"/>
+<attribute name="VALUE" x="313.436" y="51.689" size="1.778" layer="96"/>
+</instance>
+<instance part="VSS75" gate="G$1" x="312.42" y="48.26" smashed="yes">
+<attribute name="VALUE" x="309.88" y="43.18" size="1.778" layer="96" rot="R90"/>
+</instance>
+<instance part="C46" gate="G$1" x="276.86" y="-17.78" smashed="yes">
+<attribute name="NAME" x="277.876" y="-17.145" size="1.778" layer="95"/>
+<attribute name="VALUE" x="277.876" y="-21.971" size="1.778" layer="96"/>
+</instance>
+<instance part="VSS76" gate="G$1" x="276.86" y="-25.4" smashed="yes">
+<attribute name="VALUE" x="274.32" y="-30.48" size="1.778" layer="96" rot="R90"/>
+</instance>
+<instance part="C47" gate="G$1" x="266.7" y="-17.78" smashed="yes">
+<attribute name="NAME" x="267.716" y="-17.145" size="1.778" layer="95"/>
+<attribute name="VALUE" x="267.716" y="-21.971" size="1.778" layer="96"/>
+</instance>
+<instance part="VSS77" gate="G$1" x="266.7" y="-25.4" smashed="yes">
+<attribute name="VALUE" x="264.16" y="-30.48" size="1.778" layer="96" rot="R90"/>
+</instance>
 </instances>
 <busses>
@@
 <pinref part="VDD26" gate="G$1" pin="VDD"/>
 </segment>
+<segment>
+<pinref part="U4" gate="G$1" pin="VDD"/>
+<wire x1="302.26" y1="50.8" x2="302.26" y2="53.34" width="0.1524" layer="91"/>
+<pinref part="U4" gate="G$1" pin="VDDIO"/>
+<wire x1="302.26" y1="53.34" x2="302.26" y2="58.42" width="0.1524" layer="91"/>
+<junction x="302.26" y="53.34"/>
+<junction x="302.26" y="58.42"/>
+<wire x1="312.42" y1="58.42" x2="302.26" y2="58.42" width="0.1524" layer="91"/>
+<junction x="312.42" y="58.42"/>
+<junction x="302.26" y="50.8"/>
+<label x="304.8" y="58.42" size="1.778" layer="95"/>
+<pinref part="C45" gate="G$1" pin="1"/>
+</segment>
+<segment>
+<wire x1="271.78" y1="45.72" x2="261.62" y2="45.72" width="0.1524" layer="91"/>
+<pinref part="U4" gate="G$1" pin="CSB"/>
+<junction x="271.78" y="45.72"/>
+<junction x="261.62" y="45.72"/>
+<label x="266.7" y="45.72" size="1.778" layer="95"/>
+</segment>
+<segment>
+<pinref part="U5" gate="_VCNL4040" pin="VDD"/>
+<wire x1="276.86" y1="-5.08" x2="276.86" y2="-10.16" width="0.1524" layer="91"/>
+<pinref part="U5" gate="_VCNL4040" pin="VDD-LED"/>
+<wire x1="276.86" y1="-10.16" x2="276.86" y2="-15.24" width="0.1524" layer="91"/>
+<junction x="276.86" y="-10.16"/>
+<junction x="276.86" y="-5.08"/>
+<wire x1="276.86" y1="-15.24" x2="266.7" y2="-15.24" width="0.1524" layer="91"/>
+<junction x="266.7" y="-15.24"/>
+<label x="266.7" y="-17.78" size="1.778" layer="95"/>
+<pinref part="C46" gate="G$1" pin="1"/>
+<junction x="276.86" y="-15.24"/>
+<pinref part="C47" gate="G$1" pin="1"/>
+</segment>
 </net>
 <net name="VSS" class="1">
@@
 <junction x="236.22" y="-60.96"/>
 </segment>
+<segment>
+<pinref part="U5" gate="_VCNL4040" pin="GND"/>
+<pinref part="VSS73" gate="G$1" pin="VSS"/>
+<junction x="276.86" y="5.08"/>
+</segment>
+<segment>
+<pinref part="U4" gate="G$1" pin="GND"/>
+<pinref part="VSS74" gate="G$1" pin="VSS"/>
+<junction x="302.26" y="33.02"/>
+</segment>
+<segment>
+<pinref part="C45" gate="G$1" pin="2"/>
+<pinref part="VSS75" gate="G$1" pin="VSS"/>
+<junction x="312.42" y="50.8"/>
+</segment>
+<segment>
+<pinref part="C46" gate="G$1" pin="2"/>
+<pinref part="VSS76" gate="G$1" pin="VSS"/>
+<junction x="276.86" y="-22.86"/>
+</segment>
+<segment>
+<pinref part="C47" gate="G$1" pin="2"/>
+<pinref part="VSS77" gate="G$1" pin="VSS"/>
+<junction x="266.7" y="-22.86"/>
+</segment>
 </net>
 <net name="AVDD" class="2">
@@
 </segment>
 </net>
-<net name="N$17" class="0">
+<net name="BSDA" class="0">
 <segment>
 <pinref part="U3" gate="G$1" pin="ENV_SDA"/>
 <pinref part="R10" gate="G$1" pin="2"/>
 <junction x="226.06" y="137.16"/>
+<wire x1="226.06" y1="137.16" x2="226.06" y2="132.08" width="0.1524" layer="91"/>
+<wire x1="226.06" y1="132.08" x2="233.68" y2="132.08" width="0.1524" layer="91"/>
+<junction x="233.68" y="132.08"/>
+<label x="243.84" y="137.16" size="1.778" layer="95"/>
+</segment>
+<segment>
+<wire x1="264.16" y1="40.64" x2="271.78" y2="40.64" width="0.1524" layer="91"/>
+<pinref part="U4" gate="G$1" pin="SDI"/>
+<junction x="271.78" y="40.64"/>
+<junction x="264.16" y="40.64"/>
+<label x="266.7" y="40.64" size="1.778" layer="95"/>
+</segment>
+<segment>
+<wire x1="312.42" y1="0" x2="320.04" y2="0" width="0.1524" layer="91"/>
+<pinref part="U5" gate="_VCNL4040" pin="SDA"/>
+<junction x="320.04" y="0"/>
+<junction x="312.42" y="0"/>
+<label x="314.96" y="0" size="1.778" layer="95"/>
 </segment>
 </net>
-<net name="N$18" class="0">
+<net name="BSCL" class="0">
 <segment>
 <pinref part="U3" gate="G$1" pin="ENV_SCL"/>
 <pinref part="R11" gate="G$1" pin="2"/>
 <junction x="226.06" y="139.7"/>
+<wire x1="226.06" y1="139.7" x2="226.06" y2="142.24" width="0.1524" layer="91"/>
+<wire x1="226.06" y1="142.24" x2="233.68" y2="142.24" width="0.1524" layer="91"/>
+<junction x="233.68" y="142.24"/>
+<label x="243.84" y="139.7" size="1.778" layer="95"/>
+</segment>
+<segment>
+<wire x1="264.16" y1="43.18" x2="271.78" y2="43.18" width="0.1524" layer="91"/>
+<pinref part="U4" gate="G$1" pin="SCK"/>
+<junction x="271.78" y="43.18"/>
+<junction x="264.16" y="43.18"/>
+<label x="266.7" y="43.18" size="1.778" layer="95"/>
+</segment>
+<segment>
+<wire x1="312.42" y1="5.08" x2="320.04" y2="5.08" width="0.1524" layer="91"/>
+<pinref part="U5" gate="_VCNL4040" pin="SCL"/>
+<junction x="320.04" y="5.08"/>
+<junction x="312.42" y="5.08"/>
+<label x="314.96" y="5.08" size="1.778" layer="95"/>
 </segment>
 </net>
@@
 </segment>
 </net>
+<net name="N$22" class="0">
+<segment>
+<pinref part="U5" gate="_VCNL4040" pin="C-SENSOR"/>
+<wire x1="276.86" y1="0" x2="269.24" y2="0" width="0.1524" layer="91"/>
+<wire x1="269.24" y1="0" x2="269.24" y2="17.78" width="0.1524" layer="91"/>
+<wire x1="269.24" y1="17.78" x2="330.2" y2="17.78" width="0.1524" layer="91"/>
+<wire x1="330.2" y1="17.78" x2="330.2" y2="-10.16" width="0.1524" layer="91"/>
+<pinref part="U5" gate="_VCNL4040" pin="C-LED"/>
+<wire x1="330.2" y1="-10.16" x2="312.42" y2="-10.16" width="0.1524" layer="91"/>
+<junction x="276.86" y="0"/>
+<junction x="312.42" y="-10.16"/>
+</segment>
+</net>

Commit message: up
Parts:
- C32: value 0.1uf -> 0.47uf
- R10, R11: value 10k -> 2.2k
- U3: value BNO080 -> BNO086
Changed lines of the file:
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@@
 <part name="R7" library="rcl" library_urn="urn:adsk.eagle:library:334" deviceset="R-US_" device="M0805" package3d_urn="urn:adsk.eagle:package:23556/2" value="10k"/>
 <part name="VDD18" library="supply1" library_urn="urn:adsk.eagle:library:371" deviceset="VDD" device=""/>
-<part name="U3" library="BNO080" deviceset="BNO080" device=""/>
+<part name="U3" library="BNO080" deviceset="BNO080" device="" value="BNO086"/>
 <part name="C30" library="rcl" library_urn="urn:adsk.eagle:library:334" deviceset="C-US" device="C0805" package3d_urn="urn:adsk.eagle:package:23617/2" value="0.1uf"/>
 <part name="VSS60" library="supply1" library_urn="urn:adsk.eagle:library:371" deviceset="VSS" device=""/>
@@
 <part name="SJ3" library="jumper" library_urn="urn:adsk.eagle:library:252" deviceset="SJ" device="" package3d_urn="urn:adsk.eagle:package:15471/1" value="BOOT_ON"/>
 <part name="R9" library="rcl" library_urn="urn:adsk.eagle:library:334" deviceset="R-US_" device="M0805" package3d_urn="urn:adsk.eagle:package:23556/2" value="10k"/>
-<part name="C32" library="rcl" library_urn="urn:adsk.eagle:library:334" deviceset="C-US" device="C0805" package3d_urn="urn:adsk.eagle:package:23617/2" value="0.1uf"/>
+<part name="C32" library="rcl" library_urn="urn:adsk.eagle:library:334" deviceset="C-US" device="C0805" package3d_urn="urn:adsk.eagle:package:23617/2" value="0.47uf"/>
 <part name="VSS62" library="supply1" library_urn="urn:adsk.eagle:library:371" deviceset="VSS" device=""/>
 <part name="SJ4" library="jumper" library_urn="urn:adsk.eagle:library:252" deviceset="SJ" device="" package3d_urn="urn:adsk.eagle:package:15471/1" value="IMU_RESET"/>
@@
 <part name="SV4" library="con-lstb" library_urn="urn:adsk.eagle:library:162" deviceset="MA10-1" device="" package3d_urn="urn:adsk.eagle:package:8346/1" value="IMU_SIG"/>
 <part name="VSS64" library="supply1" library_urn="urn:adsk.eagle:library:371" deviceset="VSS" device=""/>
-<part name="R10" library="rcl" library_urn="urn:adsk.eagle:library:334" deviceset="R-US_" device="M0805" package3d_urn="urn:adsk.eagle:package:23556/2" value="10k"/>
-<part name="R11" library="rcl" library_urn="urn:adsk.eagle:library:334" deviceset="R-US_" device="M0805" package3d_urn="urn:adsk.eagle:package:23556/2" value="10k"/>
+<part name="R10" library="rcl" library_urn="urn:adsk.eagle:library:334" deviceset="R-US_" device="M0805" package3d_urn="urn:adsk.eagle:package:23556/2" value="2.2k"/>
+<part name="R11" library="rcl" library_urn="urn:adsk.eagle:library:334" deviceset="R-US_" device="M0805" package3d_urn="urn:adsk.eagle:package:23556/2" value="2.2k"/>
 <part name="VDD19" library="supply1" library_urn="urn:adsk.eagle:library:371" deviceset="VDD" device=""/>
 <part name="VDD24" library="supply1" library_urn="urn:adsk.eagle:library:371" deviceset="VDD" device=""/>

Commit message: up
Parts:
- added R12, R13: 0 ohms, rcl:R-US_R0805
- added R21, R22: 1k, rcl:R-US_R0805
- added SJ9: QEI_PWR, jumper:SJ2W
Connections:
- new net CHANA: IC3.CHANNEL_A, R12.1
- new net CHANB: IC3.CHANNEL_B, R13.1
- new net CHANP: IC3.POWER_(+), SJ9.2
- net +5V: now also SJ9.3; no longer IC3.POWER_(+)
- net QEA2: now also R12.2, R22.1; no longer IC3.CHANNEL_A
- net QEB2: now also R13.2, R21.2; no longer IC3.CHANNEL_B
- net VDD: now also SJ9.1
- net VSS: now also R21.1, R22.2
Changed lines of the file:
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@@
 <part name="PS2" library="MYRLP330015F21RE" deviceset="MYRLP330015F21RE" device=""/>
 <part name="P+1" library="supply1" library_urn="urn:adsk.eagle:library:371" deviceset="+5V" device=""/>
-<part name="P+2" library="supply1" library_urn="urn:adsk.eagle:library:371" deviceset="+5V" device=""/>
 <part name="C33" library="rcl" library_urn="urn:adsk.eagle:library:334" deviceset="C-US" device="C0805" package3d_urn="urn:adsk.eagle:package:23617/2" value="10uf"/>
 <part name="C44" library="rcl" library_urn="urn:adsk.eagle:library:334" deviceset="C-US" device="C0805" package3d_urn="urn:adsk.eagle:package:23617/2" value="10uf"/>
@@
 <part name="C47" library="rcl" library_urn="urn:adsk.eagle:library:334" deviceset="C-US" device="C0805" package3d_urn="urn:adsk.eagle:package:23617/2" value="10uf"/>
 <part name="VSS77" library="supply1" library_urn="urn:adsk.eagle:library:371" deviceset="VSS" device=""/>
+<part name="SJ9" library="jumper" library_urn="urn:adsk.eagle:library:252" deviceset="SJ2W" device="" package3d_urn="urn:adsk.eagle:package:15474/1" value="QEI_PWR"/>
+<part name="P+4" library="supply1" library_urn="urn:adsk.eagle:library:371" deviceset="+5V" device=""/>
+<part name="VDD27" library="supply1" library_urn="urn:adsk.eagle:library:371" deviceset="VDD" device=""/>
+<part name="R12" library="rcl" library_urn="urn:adsk.eagle:library:334" deviceset="R-US_" device="R0805" package3d_urn="urn:adsk.eagle:package:23553/2" value="0 ohms"/>
+<part name="R13" library="rcl" library_urn="urn:adsk.eagle:library:334" deviceset="R-US_" device="R0805" package3d_urn="urn:adsk.eagle:package:23553/2" value="0 ohms"/>
+<part name="R21" library="rcl" library_urn="urn:adsk.eagle:library:334" deviceset="R-US_" device="R0805" package3d_urn="urn:adsk.eagle:package:23553/2" value="1k"/>
+<part name="R22" library="rcl" library_urn="urn:adsk.eagle:library:334" deviceset="R-US_" device="R0805" package3d_urn="urn:adsk.eagle:package:23553/2" value="1k"/>
+<part name="VSS78" library="supply1" library_urn="urn:adsk.eagle:library:371" deviceset="VSS" device=""/>
+<part name="VSS79" library="supply1" library_urn="urn:adsk.eagle:library:371" deviceset="VSS" device=""/>
 </parts>
 <sheets>
@@
 <attribute name="VALUE" x="233.68" y="-58.42" size="1.778" layer="96" rot="R180"/>
 </instance>
-<instance part="P+2" gate="1" x="22.86" y="-78.74" smashed="yes" rot="R90">
-<attribute name="VALUE" x="27.94" y="-81.28" size="1.778" layer="96" rot="R180"/>
-</instance>
 <instance part="C33" gate="G$1" x="233.68" y="-50.8" smashed="yes" rot="R90">
 <attribute name="NAME" x="233.045" y="-49.784" size="1.778" layer="95" rot="R90"/>
@@
 <attribute name="VALUE" x="264.16" y="-30.48" size="1.778" layer="96" rot="R90"/>
 </instance>
+<instance part="SJ9" gate="G$1" x="10.16" y="-78.74" smashed="yes" rot="R180">
+<attribute name="NAME" x="7.62" y="-79.121" size="1.778" layer="95" rot="R180"/>
+<attribute name="VALUE" x="15.24" y="-84.455" size="1.778" layer="96" rot="R180"/>
+</instance>
+<instance part="P+4" gate="1" x="10.16" y="-71.12" smashed="yes">
+<attribute name="VALUE" x="7.62" y="-76.2" size="1.778" layer="96" rot="R90"/>
+</instance>
+<instance part="VDD27" gate="G$1" x="10.16" y="-91.44" smashed="yes" rot="R180">
+<attribute name="VALUE" x="12.7" y="-88.9" size="1.778" layer="96" rot="R270"/>
+</instance>
+<instance part="R12" gate="G$1" x="12.7" y="-48.26" smashed="yes" rot="R180">
+<attribute name="NAME" x="16.51" y="-49.7586" size="1.778" layer="95" rot="R180"/>
+<attribute name="VALUE" x="16.51" y="-44.958" size="1.778" layer="96" rot="R180"/>
+</instance>
+<instance part="R13" gate="G$1" x="12.7" y="-63.5" smashed="yes" rot="R180">
+<attribute name="NAME" x="16.51" y="-64.9986" size="1.778" layer="95" rot="R180"/>
+<attribute name="VALUE" x="16.51" y="-60.198" size="1.778" layer="96" rot="R180"/>
+</instance>
+<instance part="R21" gate="G$1" x="2.54" y="-63.5" smashed="yes">
+<attribute name="NAME" x="-1.27" y="-62.0014" size="1.778" layer="95"/>
+<attribute name="VALUE" x="-1.27" y="-66.802" size="1.778" layer="96"/>
+</instance>
+<instance part="R22" gate="G$1" x="2.54" y="-48.26" smashed="yes" rot="R180">
+<attribute name="NAME" x="6.35" y="-49.7586" size="1.778" layer="95" rot="R180"/>
+<attribute name="VALUE" x="6.35" y="-44.958" size="1.778" layer="96" rot="R180"/>
+</instance>
+<instance part="VSS78" gate="G$1" x="-5.08" y="-63.5" smashed="yes" rot="R270">
+<attribute name="VALUE" x="-10.16" y="-60.96" size="1.778" layer="96"/>
+</instance>
+<instance part="VSS79" gate="G$1" x="-5.08" y="-48.26" smashed="yes" rot="R270">
+<attribute name="VALUE" x="-10.16" y="-45.72" size="1.778" layer="96"/>
+</instance>
 </instances>
 <busses>
@@
 <pinref part="C47" gate="G$1" pin="1"/>
 </segment>
+<segment>
+<pinref part="SJ9" gate="G$1" pin="1"/>
+<pinref part="VDD27" gate="G$1" pin="VDD"/>
+<wire x1="10.16" y1="-88.9" x2="10.16" y2="-83.82" width="0.1524" layer="91"/>
+<junction x="10.16" y="-88.9"/>
+<junction x="10.16" y="-83.82"/>
+</segment>
 </net>
 <net name="VSS" class="1">
@@
 <junction x="266.7" y="-22.86"/>
 </segment>
+<segment>
+<pinref part="R21" gate="G$1" pin="1"/>
+<pinref part="VSS78" gate="G$1" pin="VSS"/>
+<junction x="-2.54" y="-63.5"/>
+</segment>
+<segment>
+<pinref part="R22" gate="G$1" pin="2"/>
+<pinref part="VSS79" gate="G$1" pin="VSS"/>
+<junction x="-2.54" y="-48.26"/>
+</segment>
 </net>
 <net name="AVDD" class="2">
@@
 </segment>
 <segment>
-<wire x1="27.94" y1="-71.12" x2="40.64" y2="-71.12" width="0.1524" layer="91"/>
-<pinref part="IC3" gate="G$1" pin="CHANNEL_A"/>
-<junction x="40.64" y="-71.12"/>
-<label x="27.94" y="-71.12" size="1.778" layer="95"/>
+<wire x1="7.62" y1="-60.96" x2="7.62" y2="-48.26" width="0.1524" layer="91"/>
+<label x="0" y="-55.88" size="1.778" layer="95"/>
+<pinref part="R12" gate="G$1" pin="2"/>
+<pinref part="R22" gate="G$1" pin="1"/>
+<junction x="7.62" y="-48.26"/>
+<junction x="7.62" y="-60.96"/>
 </segment>
 </net>
@@
 </segment>
 <segment>
-<wire x1="27.94" y1="-81.28" x2="40.64" y2="-81.28" width="0.1524" layer="91"/>
-<pinref part="IC3" gate="G$1" pin="CHANNEL_B"/>
-<junction x="40.64" y="-81.28"/>
-<label x="30.48" y="-81.28" size="1.778" layer="95"/>
+<wire x1="7.62" y1="-76.2" x2="7.62" y2="-63.5" width="0.1524" layer="91"/>
+<label x="0" y="-71.12" size="1.778" layer="95"/>
+<pinref part="R13" gate="G$1" pin="2"/>
+<pinref part="R21" gate="G$1" pin="2"/>
+<junction x="7.62" y="-63.5"/>
+<junction x="7.62" y="-76.2"/>
 </segment>
 </net>
@@
 </segment>
 <segment>
-<wire x1="40.64" y1="-78.74" x2="25.4" y2="-78.74" width="0.1524" layer="91"/>
-<pinref part="IC3" gate="G$1" pin="POWER_(+)"/>
-<junction x="40.64" y="-78.74"/>
-<junction x="25.4" y="-78.74"/>
-<label x="17.78" y="-78.74" size="1.778" layer="95"/>
-<pinref part="P+2" gate="1" pin="+5V"/>
-</segment>
-<segment>
 <pinref part="+5VDC" gate="G$1" pin="2"/>
 <wire x1="203.2" y1="-58.42" x2="210.82" y2="-58.42" width="0.1524" layer="91"/>
@@
 <junction x="203.2" y="-60.96"/>
 </segment>
+<segment>
+<pinref part="SJ9" gate="G$1" pin="3"/>
+<pinref part="P+4" gate="1" pin="+5V"/>
+<junction x="10.16" y="-73.66"/>
+</segment>
 </net>
 <net name="N$22" class="0">
@@
 </segment>
 </net>
+<net name="CHANP" class="1">
+<segment>
+<wire x1="40.64" y1="-78.74" x2="15.24" y2="-78.74" width="0.1524" layer="91"/>
+<pinref part="IC3" gate="G$1" pin="POWER_(+)"/>
+<junction x="40.64" y="-78.74"/>
+<label x="17.78" y="-78.74" size="1.778" layer="95"/>
+<pinref part="SJ9" gate="G$1" pin="2"/>
+<junction x="15.24" y="-78.74"/>
+</segment>
+</net>
+<net name="CHANA" class="0">
+<segment>
+<pinref part="IC3" gate="G$1" pin="CHANNEL_A"/>
+<wire x1="40.64" y1="-71.12" x2="30.48" y2="-71.12" width="0.1524" layer="91"/>
+<junction x="30.48" y="-71.12"/>
+<label x="33.02" y="-71.12" size="1.778" layer="95"/>
+<junction x="40.64" y="-71.12"/>
+</segment>
+<segment>
+<wire x1="27.94" y1="-48.26" x2="17.78" y2="-48.26" width="0.1524" layer="91"/>
+<pinref part="R12" gate="G$1" pin="1"/>
+<junction x="27.94" y="-48.26"/>
+<wire x1="38.1" y1="-48.26" x2="27.94" y2="-48.26" width="0.1524" layer="91"/>
+<junction x="38.1" y="-48.26"/>
+<label x="30.48" y="-48.26" size="1.778" layer="95"/>
+<junction x="17.78" y="-48.26"/>
+</segment>
+</net>
+<net name="CHANB" class="0">
+<segment>
+<pinref part="IC3" gate="G$1" pin="CHANNEL_B"/>
+<wire x1="40.64" y1="-81.28" x2="33.02" y2="-81.28" width="0.1524" layer="91"/>
+<junction x="33.02" y="-81.28"/>
+<label x="35.56" y="-81.28" size="1.778" layer="95"/>
+<junction x="40.64" y="-81.28"/>
+</segment>
+<segment>
+<wire x1="25.4" y1="-63.5" x2="17.78" y2="-63.5" width="0.1524" layer="91"/>
+<pinref part="R13" gate="G$1" pin="1"/>
+<junction x="25.4" y="-63.5"/>
+<wire x1="33.02" y1="-63.5" x2="25.4" y2="-63.5" width="0.1524" layer="91"/>
+<junction x="33.02" y="-63.5"/>
+<label x="22.86" y="-63.5" size="1.778" layer="95"/>
+<junction x="17.78" y="-63.5"/>
+</segment>
+</net>
