File: ll-tester.sch (EAGLE design)
At the start: 138 parts, among them IC1 BMA490L, IC2 TCAN330GD, IC3 EM14R0D-R20-L064S, IC4 CAT4238TD-GT3, U1 PIC32MK0512MCJ048T-I/Y8XTQFP4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, U2 MAX6126B30, U3 BNO086, U4 BME280, U5 VCNL4040M3OE

Commit message: up
Connections:
- removed net N$66: IC4.FB, PAD8.P, R19.1
- removed net N$67: C43.1, D2.C, PAD7.P
- removed net N$68: PAD10.P, PAD9.P
- removed net N$69: PAD11.P, PAD12.P
- new net CA1: C43.1, D2.C, LCD2.CAT1, PAD7.P
- new net CA2: LCD2.CAT2, LCD2.CAT4, PAD10.P, PAD9.P
- new net CA3: LCD2.CAT3, LCD2.CAT5, PAD11.P, PAD12.P
- new net CA6: IC4.FB, LCD2.CAT6, PAD8.P, R19.1
Changed lines of the file:
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@@
-</segment>
-</net>
-<net name="N$66" class="2">
-<segment>
-<pinref part="IC4" gate="G$1" pin="FB"/>
-<wire x1="71.12" y1="-190.5" x2="71.12" y2="-210.82" width="0.1524" layer="91"/>
-<junction x="71.12" y="-190.5"/>
-<pinref part="R19" gate="G$1" pin="1"/>
-<wire x1="71.12" y1="-210.82" x2="17.78" y2="-210.82" width="0.1524" layer="91"/>
-<junction x="71.12" y="-210.82"/>
-<pinref part="PAD8" gate="P" pin="P"/>
-<junction x="17.78" y="-210.82"/>
-</segment>
-</net>
-<net name="N$67" class="2">
-<segment>
-<pinref part="D2" gate="G$1" pin="C"/>
-<wire x1="40.64" y1="-185.42" x2="38.1" y2="-185.42" width="0.1524" layer="91"/>
-<pinref part="C43" gate="G$1" pin="1"/>
-<wire x1="38.1" y1="-185.42" x2="30.48" y2="-185.42" width="0.1524" layer="91"/>
-<wire x1="30.48" y1="-185.42" x2="17.78" y2="-185.42" width="0.1524" layer="91"/>
-<junction x="30.48" y="-185.42"/>
-<pinref part="PAD7" gate="P" pin="P"/>
-<junction x="17.78" y="-185.42"/>
-<junction x="38.1" y="-185.42"/>
-</segment>
-</net>
-<net name="N$68" class="2">
-<segment>
-<pinref part="PAD10" gate="P" pin="P"/>
-<wire x1="17.78" y1="-157.48" x2="27.94" y2="-157.48" width="0.1524" layer="91"/>
-<wire x1="27.94" y1="-157.48" x2="27.94" y2="-149.86" width="0.1524" layer="91"/>
-<pinref part="PAD9" gate="P" pin="P"/>
-<wire x1="27.94" y1="-149.86" x2="17.78" y2="-149.86" width="0.1524" layer="91"/>
-<junction x="17.78" y="-149.86"/>
-<junction x="17.78" y="-157.48"/>
-</segment>
-</net>
-<net name="N$69" class="2">
-<segment>
-<pinref part="PAD12" gate="P" pin="P"/>
-<wire x1="17.78" y1="-172.72" x2="27.94" y2="-172.72" width="0.1524" layer="91"/>
-<wire x1="27.94" y1="-172.72" x2="27.94" y2="-165.1" width="0.1524" layer="91"/>
-<pinref part="PAD11" gate="P" pin="P"/>
-<wire x1="27.94" y1="-165.1" x2="17.78" y2="-165.1" width="0.1524" layer="91"/>
-<junction x="17.78" y="-165.1"/>
-<junction x="17.78" y="-172.72"/>
 </segment>
 </net>
@@
 </segment>
 </net>
+<net name="CA1" class="1">
+<segment>
+<pinref part="LCD2" gate="G$1" pin="CAT1"/>
+<wire x1="111.76" y1="-147.32" x2="111.76" y2="-154.94" width="0.1524" layer="91"/>
+<junction x="111.76" y="-147.32"/>
+<junction x="111.76" y="-154.94"/>
+<label x="111.76" y="-157.48" size="1.778" layer="95" rot="R90"/>
+</segment>
+<segment>
+<pinref part="D2" gate="G$1" pin="C"/>
+<wire x1="40.64" y1="-185.42" x2="38.1" y2="-185.42" width="0.1524" layer="91"/>
+<pinref part="C43" gate="G$1" pin="1"/>
+<wire x1="38.1" y1="-185.42" x2="30.48" y2="-185.42" width="0.1524" layer="91"/>
+<wire x1="30.48" y1="-185.42" x2="17.78" y2="-185.42" width="0.1524" layer="91"/>
+<junction x="30.48" y="-185.42"/>
+<pinref part="PAD7" gate="P" pin="P"/>
+<junction x="17.78" y="-185.42"/>
+<junction x="38.1" y="-185.42"/>
+<wire x1="17.78" y1="-185.42" x2="10.16" y2="-185.42" width="0.1524" layer="91"/>
+<label x="12.7" y="-185.42" size="1.778" layer="95" rot="R90"/>
+<junction x="10.16" y="-185.42"/>
+</segment>
+</net>
+<net name="CA2" class="1">
+<segment>
+<pinref part="LCD2" gate="G$1" pin="CAT2"/>
+<wire x1="114.3" y1="-147.32" x2="114.3" y2="-154.94" width="0.1524" layer="91"/>
+<junction x="114.3" y="-147.32"/>
+<junction x="114.3" y="-154.94"/>
+<label x="114.3" y="-157.48" size="1.778" layer="95" rot="R90"/>
+</segment>
+<segment>
+<pinref part="PAD10" gate="P" pin="P"/>
+<wire x1="17.78" y1="-157.48" x2="27.94" y2="-157.48" width="0.1524" layer="91"/>
+<wire x1="27.94" y1="-157.48" x2="27.94" y2="-149.86" width="0.1524" layer="91"/>
+<pinref part="PAD9" gate="P" pin="P"/>
+<wire x1="27.94" y1="-149.86" x2="17.78" y2="-149.86" width="0.1524" layer="91"/>
+<wire x1="10.16" y1="-157.48" x2="17.78" y2="-157.48" width="0.1524" layer="91"/>
+<wire x1="10.16" y1="-149.86" x2="17.78" y2="-149.86" width="0.1524" layer="91"/>
+<label x="7.62" y="-157.48" size="1.778" layer="95" rot="R180"/>
+<label x="7.62" y="-149.86" size="1.778" layer="95" rot="R180"/>
+<junction x="10.16" y="-149.86"/>
+<junction x="10.16" y="-157.48"/>
+<junction x="17.78" y="-149.86"/>
+<junction x="17.78" y="-157.48"/>
+</segment>
+<segment>
+<wire x1="119.38" y1="-147.32" x2="119.38" y2="-154.94" width="0.1524" layer="91"/>
+<pinref part="LCD2" gate="G$1" pin="CAT4"/>
+<label x="119.38" y="-157.48" size="1.778" layer="95" rot="R90"/>
+<junction x="119.38" y="-154.94"/>
+<junction x="119.38" y="-147.32"/>
+</segment>
+</net>
+<net name="CA3" class="1">
+<segment>
+<pinref part="LCD2" gate="G$1" pin="CAT3"/>
+<wire x1="116.84" y1="-147.32" x2="116.84" y2="-154.94" width="0.1524" layer="91"/>
+<junction x="116.84" y="-147.32"/>
+<junction x="116.84" y="-154.94"/>
+<wire x1="116.84" y1="-147.32" x2="116.84" y2="-154.94" width="0.1524" layer="91"/>
+<label x="116.84" y="-157.48" size="1.778" layer="95" rot="R90"/>
+</segment>
+<segment>
+<pinref part="PAD12" gate="P" pin="P"/>
+<wire x1="17.78" y1="-172.72" x2="27.94" y2="-172.72" width="0.1524" layer="91"/>
+<wire x1="27.94" y1="-172.72" x2="27.94" y2="-165.1" width="0.1524" layer="91"/>
+<pinref part="PAD11" gate="P" pin="P"/>
+<wire x1="27.94" y1="-165.1" x2="17.78" y2="-165.1" width="0.1524" layer="91"/>
+<wire x1="10.16" y1="-172.72" x2="17.78" y2="-172.72" width="0.1524" layer="91"/>
+<wire x1="10.16" y1="-165.1" x2="17.78" y2="-165.1" width="0.1524" layer="91"/>
+<label x="7.62" y="-172.72" size="1.778" layer="95" rot="R180"/>
+<label x="7.62" y="-165.1" size="1.778" layer="95" rot="R180"/>
+<junction x="10.16" y="-165.1"/>
+<junction x="10.16" y="-172.72"/>
+<junction x="17.78" y="-165.1"/>
+<junction x="17.78" y="-172.72"/>
+</segment>
+<segment>
+<wire x1="121.92" y1="-147.32" x2="121.92" y2="-154.94" width="0.1524" layer="91"/>
+<pinref part="LCD2" gate="G$1" pin="CAT5"/>
+<label x="121.92" y="-157.48" size="1.778" layer="95" rot="R90"/>
+<junction x="121.92" y="-154.94"/>
+<junction x="121.92" y="-147.32"/>
+</segment>
+</net>
+<net name="CA6" class="1">
+<segment>
+<pinref part="LCD2" gate="G$1" pin="CAT6"/>
+<wire x1="124.46" y1="-147.32" x2="124.46" y2="-154.94" width="0.1524" layer="91"/>
+<junction x="124.46" y="-147.32"/>
+<junction x="124.46" y="-154.94"/>
+<label x="124.46" y="-157.48" size="1.778" layer="95" rot="R90"/>
+</segment>
+<segment>
+<pinref part="IC4" gate="G$1" pin="FB"/>
+<wire x1="71.12" y1="-190.5" x2="71.12" y2="-210.82" width="0.1524" layer="91"/>
+<junction x="71.12" y="-190.5"/>
+<pinref part="R19" gate="G$1" pin="1"/>
+<wire x1="71.12" y1="-210.82" x2="17.78" y2="-210.82" width="0.1524" layer="91"/>
+<junction x="71.12" y="-210.82"/>
+<pinref part="PAD8" gate="P" pin="P"/>
+<junction x="17.78" y="-210.82"/>
+<wire x1="10.16" y1="-210.82" x2="17.78" y2="-210.82" width="0.1524" layer="91"/>
+<label x="12.7" y="-210.82" size="1.778" layer="95" rot="R90"/>
+<junction x="10.16" y="-210.82"/>
+</segment>
+</net>

Commit message: up
Parts:
- added I2C: I2C, pinhead:PINHD-1X2
Connections:
- net BSCL: now also I2C.1
- net BSDA: now also I2C.2
Changed lines of the file:
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@@
 <part name="VSS78" library="supply1" library_urn="urn:adsk.eagle:library:371" deviceset="VSS" device=""/>
 <part name="VSS79" library="supply1" library_urn="urn:adsk.eagle:library:371" deviceset="VSS" device=""/>
+<part name="I2C" library="pinhead" library_urn="urn:adsk.eagle:library:325" deviceset="PINHD-1X2" device="" package3d_urn="urn:adsk.eagle:package:22435/2" value="I2C"/>
 </parts>
 <sheets>
@@
 <attribute name="VALUE" x="-10.16" y="-45.72" size="1.778" layer="96"/>
 </instance>
+<instance part="I2C" gate="G$1" x="261.62" y="25.4" smashed="yes">
+<attribute name="NAME" x="255.27" y="31.115" size="1.778" layer="95"/>
+<attribute name="VALUE" x="255.27" y="20.32" size="1.778" layer="96"/>
+</instance>
 </instances>
 <busses>
@@
 <label x="314.96" y="0" size="1.778" layer="95"/>
 </segment>
+<segment>
+<wire x1="251.46" y1="25.4" x2="259.08" y2="25.4" width="0.1524" layer="91"/>
+<pinref part="I2C" gate="G$1" pin="2"/>
+<junction x="251.46" y="25.4"/>
+<junction x="259.08" y="25.4"/>
+<label x="243.84" y="25.4" size="1.778" layer="95"/>
+</segment>
 </net>
 <net name="BSCL" class="0">
@@
 <label x="314.96" y="5.08" size="1.778" layer="95"/>
 </segment>
+<segment>
+<wire x1="251.46" y1="27.94" x2="259.08" y2="27.94" width="0.1524" layer="91"/>
+<pinref part="I2C" gate="G$1" pin="1"/>
+<junction x="259.08" y="27.94"/>
+<junction x="251.46" y="27.94"/>
+<label x="243.84" y="27.94" size="1.778" layer="95"/>
+</segment>
 </net>
