File: mate_a.brd (EAGLE design)
At the start: 92.7 x 100 mm, 8 parts, among them IC1 PIC18F47Q84-E_P, X1 GLX-S-88M

Commit message: up
Parts:
- added OS1_10MHZ: OSC-OE-CFPS-72, IQD-Frequency-Products:7.2X5.2-4-PAD
- added U1: REF3440IDBVR, REF3440IDBVR:SOT95P280X145-6N
- moved R1 30.1 mm to (133.3, 43.2)
- moved R3 29.5 mm to (125.7, 52.1), turned to 90 degrees
- moved OK1 28.0 mm to (132.1, 50.8)
- moved R4 25.7 mm to (125.7, 62.2), turned to 90 degrees
- moved OK2 25.4 mm to (132.1, 62.2)
- moved R2 20.4 mm to (127.0, 43.2)
- moved X1 19.1 mm to (132.1, 31.8)
- moved IC1 2.54 mm to (106.7, 45.7)
Connections:
- new net CPU_CLK: IC1.13, OS1_10MHZ.3
- new net VREF: IC1.5, U1.5, U1.6
- net VDD: now also OS1_10MHZ.1, OS1_10MHZ.4, U1.4
- net VSS: now also OS1_10MHZ.2, U1.1, U1.2, U1.3
Routing:
- net +24V: track 21.1 -> 59.5 mm
- net VREF: track 0.00 -> 29.9 mm
- net PC_TX: track 16.6 -> 40.8 mm
- net 0V: track 41.6 -> 17.6 mm
- net MX_TX: track 28.5 -> 47.0 mm
- net VDD: track 56.4 -> 72.2 mm
- net CPU_CLK: track 0.00 -> 15.2 mm
- net VSS: track 15.1 -> 29.0 mm, vias 1 -> 2
- net N$1: track 16.3 -> 3.11 mm
- net MX_RX: track 22.5 -> 20.6 mm
- net N$3: track 9.86 -> 8.67 mm
Other:
- board size 92.7 x 100 mm -> 64.8 x 55.5 mm

Commit message: up
Parts:
- added C1, C2, C3, C5: 0.1uf, rcl:C0805
- added C4, C6: 10uf, rcl:C0805
- added ICSP: ICSP, con-lstb:MA06-1
- added R5: 56ohm, rcl:R0805
- added R6: 10k, rcl:R0805
- added SV1: Analog, con-lstb:MA10-1
- added SV2: Digtal, con-lstb:MA10-1
- moved U1 8.98 mm to (87.6, 30.5)
- moved OS1_10MHZ 6.35 mm to (88.9, 22.9)
Connections:
- new net AN0: IC1.2, SV1.1
- new net AN1: IC1.3, SV1.2
- new net AN2: IC1.4, SV1.3
- new net MCLR_SIG: IC1.1, ICSP.1, R5.2
- new net N$2: C1.1, R5.1, R6.1
- new net PGC: IC1.39, ICSP.5
- new net PGD: IC1.40, ICSP.4
- new net RD0: IC1.19, SV2.1
- new net RD1: IC1.20, SV2.2
- new net RD2: IC1.21, SV2.3
- new net RD3: IC1.22, SV2.4
- net VDD: now also C2.1, C3.1, C4.1, C5.1, C6.1, ICSP.2, R6.2, SV1.10, SV2.10
- net VSS: now also C1.2, C2.2, C3.2, C4.2, C5.2, C6.2, ICSP.3, SV1.9, SV2.9
Routing:
- net VDD: track 72.2 -> 165.5 mm, vias 0 -> 1
- net PGC: track 0.00 -> 62.8 mm
- net PGD: track 0.00 -> 41.2 mm
- net VSS: track 29.0 -> 59.0 mm, vias 2 -> 1
- net AN1: track 0.00 -> 29.9 mm
- net AN2: track 0.00 -> 29.9 mm
- net AN0: track 0.00 -> 29.9 mm
- net RD1: track 0.00 -> 28.0 mm
- net MCLR_SIG: track 0.00 -> 23.8 mm
- net RD0: track 0.00 -> 23.5 mm
- net +24V: track 59.5 -> 37.3 mm
- net MX_TX: track 47.0 -> 61.9 mm
- net N$2: track 0.00 -> 9.12 mm
- net RD2: track 0.00 -> 8.36 mm
- net RD3: track 0.00 -> 8.35 mm
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
Commit message: up
Parts:
- moved C6 12.7 mm to (121.9, 48.3), flipped to the bottom, turned to 270 degrees
- moved C5 9.67 mm to (118.1, 48.3), flipped to the bottom, turned to 270 degrees
- flipped C1 to the bottom
- flipped C3 to the bottom
- flipped C4 to the bottom
- flipped R5 to the bottom
- flipped R6 to the bottom
Routing:
- net PGC: track 62.8 -> 41.1 mm
- net VSS: track 59.0 -> 38.9 mm
- net PC_RX: track 39.5 -> 59.1 mm
- net VDD: track 165.5 -> 153.8 mm
- net AN0: track 29.9 -> 40.2 mm
- net MCLR_SIG: track 23.8 -> 31.3 mm
- net MX_TX: track 61.9 -> 55.0 mm, vias 0 -> 2
- net N$2: track 9.12 -> 14.8 mm

Commit message: up
Parts:
- added C10, C13, C15, C8: 10uf, rcl:C0805
- added C11, C12, C14, C7, C9: 0.1uf, rcl:C0805
- added CANBUS: CANBUS, con-lstb:MA04-1
- added CAN_PWR: CAN_PWR, jumper:SJ
- added IC2: 7805TV, linear:TO220V
- added LED1: run, led:CHIPLED_0805
- added LED2: error, led:CHIPLED_0805
- added LED3: comm, led:CHIPLED_0805
- added MISC_IO: misc-io, con-lstb:MA10-1
- added R7, R8, R9: 1k, rcl:R0805
- added RESET: reset, jumper:SJ
- added TP1: PTR1PAD1-13, testpad:P1-13
- added TTL_SERIAL: TTL Serial, con-lstb:MA04-1
- added U2: TCAN330GDR, TCAN330GDR:SOIC127P600X175-8N
- added X2: 22-23-2021, con-molex:22-23-2021
- R1, R2: value (none) -> 1.5k
- R3: value (none) -> 330ohm
- R4: value (none) -> 220ohm
- moved SV2 41.0 mm to (85.1, 53.3), turned to 270 degrees
- moved C4 6.35 mm to (95.2, 38.1)
Connections:
- removed net RD0: IC1.19, SV2.1
- new net AN3: IC1.6, SV1.4
- new net AN4: IC1.7, SV1.5
- new net CANRX: IC1.33, U2.4
- new net CANTX: IC1.37, U2.1
- new net CAN_N: CANBUS.1, U2.6
- new net CAN_P: CANBUS.3, U2.7
- new net CAN_VCC: C7.1, C8.1, CANBUS.4, CAN_PWR.1, U2.3
- new net CLOCKO: IC1.14, MISC_IO.10
- new net LED1: IC1.34, R7.2
- new net LED2: IC1.35, R8.2
- new net LED3: IC1.36, R9.2
- new net LO_PWR: IC1.17, TP1.TP
- new net N$4: LED1.A, R7.1
- new net N$5: LED2.A, R8.1
- new net N$6: LED3.A, R9.1
- new net RB5: IC1.38, MISC_IO.6
- new net RC0: IC1.15, SV1.6
- new net RC1: IC1.16, SV1.7
- new net RD4: IC1.27, MISC_IO.4
- new net RD5: IC1.28, MISC_IO.5
- new net RD7: IC1.30, MISC_IO.7
- new net RE0: IC1.8, MISC_IO.1
- new net RE1: IC1.9, MISC_IO.2
- new net RE2: IC1.10, MISC_IO.3
- new net RX2: IC1.19, SV2.8
- new net SCK1: IC1.18, SV2.4
- new net SDI1: IC1.23, SV2.5
- new net SDO1: IC1.24, SV2.6
- new net TX2: IC1.29, SV2.7
- new net V+: C14.1, C15.1, IC2.1, X2.1
- net MCLR_SIG: now also MISC_IO.8
- net N$2: now also RESET.1
- net PC_RX: now also TTL_SERIAL.3
- net PC_TX: now also TTL_SERIAL.2
- net RD1: now also SV2.1; no longer SV2.2
- net RD2: now also SV2.2; no longer SV2.3
- net RD3: now also SV2.3; no longer SV2.4
- net VDD: now also C10.1, C11.1, C12.1, C13.1, C9.1, CAN_PWR.2, IC2.3
- net VREF: now also SV1.8
- net VSS: now also C10.2, C11.2, C12.2, C13.2, C14.2, C15.2, C7.2, C8.2, C9.2, CANBUS.2, IC2.2, LED1.C, LED2.C, LED3.C, MISC_IO.9, RESET.2, TTL_SERIAL.1, U2.2, U2.5, U2.8, X2.2
Routing:
- net SDO1: track 0.00 -> 78.7 mm
- net RD2: track 8.36 -> 70.9 mm, vias 0 -> 1
- net RD3: track 8.35 -> 70.8 mm, vias 0 -> 1
- net VDD: track 153.8 -> 212.2 mm, vias 1 -> 4
- net SDI1: track 0.00 -> 51.7 mm, vias 0 -> 2
- net AN3: track 0.00 -> 46.8 mm, vias 0 -> 2
- net RB5: track 0.00 -> 41.0 mm, vias 0 -> 1
- net SCK1: track 0.00 -> 40.3 mm, vias 0 -> 2
- net RD4: track 0.00 -> 38.8 mm, vias 0 -> 2
- net RX2: track 0.00 -> 38.4 mm
- net RD5: track 0.00 -> 38.0 mm, vias 0 -> 1
- net AN4: track 0.00 -> 35.3 mm, vias 0 -> 1
- net TX2: track 0.00 -> 33.5 mm, vias 0 -> 1
- net CAN_VCC: track 0.00 -> 31.0 mm, vias 0 -> 1
- net MCLR_SIG: track 31.3 -> 59.9 mm, vias 0 -> 1
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
Commit message: up
Parts:
- added C16: 0.1uf, rcl:C0805
- added C17: 10uf, rcl:C0805
Connections:
- net VDD: now also TTL_SERIAL.4
- net VREF: now also C16.1, C17.1
- net VSS: now also C16.2, C17.2
Routing:
- net SDI1: track 51.7 -> 68.8 mm
- net SCK1: track 40.3 -> 57.5 mm
- net +24V: track 55.3 -> 38.2 mm
- net AN3: track 46.8 -> 29.8 mm
- net MCLR_SIG: track 59.9 -> 45.2 mm, vias 1 -> 0
- net VDD: track 212.2 -> 226.0 mm, vias 4 -> 5
- net PC_RX: track 63.9 -> 77.7 mm, vias 1 -> 2
- net RE2: track 15.8 -> 28.6 mm, vias 1 -> 0
- net PGC: track 42.4 -> 52.8 mm
- net RD3: track 70.8 -> 62.0 mm
- net RB5: track 41.0 -> 33.5 mm, vias 1 -> 0
- net RD5: track 38.0 -> 32.5 mm
- net VREF: track 49.3 -> 54.0 mm
- net RD1: track 55.2 -> 59.8 mm, vias 2 -> 0
- net 0V: track 24.4 -> 28.5 mm
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Other:
- board text added: "Outback FM interface 1.0"

Commit message: up
Parts:
- added R10: 120ohm, rcl:R0805
- R1, R2: value 1.5k -> 2.2k
- R3: value 330ohm -> 1k
- R4: value 220ohm -> 470ohm
Connections:
- net CAN_N: now also R10.1
- net CAN_P: now also R10.2
- net PC_RX: now also SV2.8; no longer TTL_SERIAL.3
- net PC_TX: now also SV2.7; no longer TTL_SERIAL.2
- net RX2: now also TTL_SERIAL.3; no longer SV2.8
- net TX2: now also TTL_SERIAL.2; no longer SV2.7
Routing:
- net PC_TX: track 57.9 -> 88.0 mm, vias 1 -> 2
- net SDO1: track 80.4 -> 55.9 mm, vias 1 -> 0
- net VDD: track 226.0 -> 247.8 mm
- net SDI1: track 68.8 -> 56.9 mm
- net PC_RX: track 77.7 -> 88.6 mm
- net PGC: track 52.8 -> 42.3 mm, vias 0 -> 1
- net RE2: track 28.6 -> 18.3 mm, vias 0 -> 1
- net SCK1: track 57.5 -> 67.4 mm, vias 2 -> 1
- net CPU_CLK: track 21.4 -> 30.9 mm
- net RD2: track 67.4 -> 58.3 mm
- net VREF: track 54.0 -> 62.7 mm, vias 1 -> 2
- net VSS: track 62.3 -> 54.0 mm
- net RD4: track 39.9 -> 31.7 mm, vias 2 -> 0
- net AN2: track 32.8 -> 40.4 mm, vias 2 -> 1
- net RD1: track 59.8 -> 67.0 mm
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
Commit message: up
Parts:
- added VREF_PWR: 5vdc_vref_pwr, con-molex:22-23-2021
- added ZENER: 5.6V, diode:SMB
- 24VDC_PWR: value 22-23-2021 -> 24vdc power
- moved U1 7.73 mm to (95.2, 31.8)
- moved C11 1.80 mm to (92.7, 31.8)
- moved C16 1.80 mm to (90.2, 36.8)
- moved C17 1.80 mm to (86.4, 36.8)
- turned ICSP to 90 degrees
- turned MISC_IO to 90 degrees
- turned R7 to 270 degrees
- turned SV1 to 90 degrees
- turned SV2 to 90 degrees
- renumbered X2 to 24VDC_PWR
Connections:
- net RX2 renamed PC_RX2
- net TX2 renamed PC_TX2
- removed net PC_RX: IC1.26, OK1.4, R3.1, SV2.8
- removed net PC_TX: IC1.25, OK2.1, SV2.7
- net AN0: now also SV1.10; no longer SV1.1
- net AN1: now also SV1.1; no longer SV1.2
- net AN2: now also SV1.2; no longer SV1.3
- net MX_RX: now also IC1.26, OK1.4, R3.1, SV2.10
- net MX_TX: now also IC1.25, OK2.1, SV2.7
- net VDD: now also SV1.8, SV2.8, ZENER.C; no longer SV1.10, SV2.10
- net VREF: now also SV1.3, VREF_PWR.1; no longer SV1.8
- net VSS: now also VREF_PWR.2, ZENER.A
Routing:
- net MX_TX: track 49.6 -> 139.5 mm
- net PC_RX: track 88.6 -> 0.00 mm, vias 2 -> 0
- net PC_TX: track 88.0 -> 0.00 mm, vias 2 -> 0
- net MX_RX: track 16.9 -> 98.1 mm, vias 0 -> 4
- net AN1: track 32.4 -> 78.1 mm, vias 2 -> 1
- net CLOCKO: track 9.63 -> 47.8 mm, vias 0 -> 2
- net SCK1: track 67.4 -> 33.0 mm, vias 1 -> 3
- net VDD: track 247.8 -> 223.6 mm, vias 5 -> 3
- net AN2: track 40.4 -> 63.3 mm, vias 1 -> 0
- net RD3: track 59.5 -> 41.6 mm
- net AN3: track 35.8 -> 49.0 mm, vias 3 -> 1
- net SDI1: track 56.9 -> 45.7 mm, vias 2 -> 3
- net RE2: track 18.3 -> 7.56 mm, vias 1 -> 0
- net MCLR_SIG: track 45.2 -> 34.5 mm, vias 0 -> 1
- net 0V: track 28.0 -> 17.6 mm
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