File: mate_a.brd (EAGLE design)
At the start: 64.8 x 55.5 mm, 50 parts, among them IC1 PIC18F47Q84-E_P, IC2 7805TV, U1 REF3440IDBVR, U2 TCAN330GDR, X1 GLX-S-88M

Commit message: up
Connections:
- net LED1 renamed MLED
- net LED2 renamed RLED
- net LED3 renamed DLED
- net RD1 renamed DB0
- net RD2 renamed DB1
- net RD3 renamed CS
- net RE0 renamed RELAY
- net RE1 renamed MISC
Changed lines of the file:
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@@
 <via x="123.2916" y="22.1742" extent="1-16" drill="0.35"/>
 </signal>
-<signal name="RD1">
+<signal name="DB0">
 <contactref element="IC1" pad="20"/>
 <contactref element="SV2" pad="1"/>
@@
 <wire x1="85.0392" y1="41.91" x2="85.09" y2="41.91" width="0.1524" layer="1"/>
 </signal>
-<signal name="RD2">
+<signal name="DB1">
 <contactref element="IC1" pad="21"/>
 <contactref element="SV2" pad="2"/>
@@
 <via x="84.8106" y="37.4904" extent="1-16" drill="0.35"/>
 </signal>
-<signal name="RD3">
+<signal name="CS">
 <contactref element="IC1" pad="22"/>
 <contactref element="SV2" pad="3"/>
@@
 <via x="104.394" y="56.769" extent="1-16" drill="0.35"/>
 </signal>
-<signal name="RE0">
+<signal name="RELAY">
 <contactref element="IC1" pad="8"/>
 <contactref element="MISC_IO" pad="1"/>
@@
 <wire x1="98.9076" y1="52.0446" x2="98.965" y2="52.07" width="0.1524" layer="1"/>
 </signal>
-<signal name="RE1">
+<signal name="MISC">
 <contactref element="IC1" pad="9"/>
 <contactref element="MISC_IO" pad="2"/>
@@
 <wire x1="123.2154" y1="44.196" x2="123.19" y2="44.13" width="0.1524" layer="1"/>
 </signal>
-<signal name="LED1">
+<signal name="MLED">
 <contactref element="IC1" pad="34"/>
 <contactref element="R7" pad="2"/>
@@
 <wire x1="114.3762" y1="54.5592" x2="114.395" y2="54.61" width="0.1524" layer="1"/>
 </signal>
-<signal name="LED2">
+<signal name="RLED">
 <contactref element="IC1" pad="35"/>
 <contactref element="R8" pad="2"/>
@@
 <wire x1="120.7008" y1="42.291" x2="120.65" y2="42.23" width="0.1524" layer="1"/>
 </signal>
-<signal name="LED3">
+<signal name="DLED">
 <contactref element="IC1" pad="36"/>
 <contactref element="R9" pad="2"/>

Commit message: up
Parts:
- moved ICSP 1.27 mm to (77.5, 59.7), turned to 270 degrees
Connections:
- removed net RD4: IC1.27, MISC_IO.4
- new net UC_RX: IC1.26, OK1.4, R3.1, SV2.10
- new net UC_TX: IC1.25, OK2.1, SV2.7
- net DLED: now also IC1.27, MISC_IO.4
- net MX_RX: no longer IC1.26, OK1.4, R3.1, SV2.10
- net MX_TX: no longer IC1.25, OK2.1, SV2.7
Routing:
- net UC_TX: track 0.00 -> 101.5 mm, vias 0 -> 2
- net UC_RX: track 0.00 -> 95.6 mm, vias 0 -> 3
- net MX_RX: track 98.1 -> 16.9 mm, vias 4 -> 0
- net MX_TX: track 139.5 -> 61.0 mm, vias 2 -> 0
- net DLED: track 26.6 -> 68.5 mm, vias 1 -> 2
- net RD4: track 29.0 -> 0.00 mm, vias 1 -> 0
- net VDD: track 223.6 -> 247.9 mm, vias 3 -> 4
- net RD7: track 28.2 -> 47.3 mm, vias 1 -> 0
- net AN1: track 78.1 -> 64.4 mm
- net VREF: track 66.7 -> 79.9 mm, vias 2 -> 1
- net AN3: track 49.0 -> 37.7 mm, vias 1 -> 0
- net CS: track 41.6 -> 52.8 mm
- net SDI1: track 45.7 -> 56.6 mm, vias 3 -> 1
- net PGD: track 40.1 -> 49.7 mm
- net SDO1: track 47.4 -> 55.9 mm
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Other:
- board text added: "Outback FM interface 1.1"
- board text removed: "Outback FM interface 1.0"

Commit message: up
Parts:
- added C18: 0.1uf, rcl:C0805
- added C19: 10uf, rcl:C0805
- added IC3: ADM3095EBRZ, ADM3095EBRZ:SOIC127P600X175-16N
- added JP1: MODBUS, pinhead:1X05
- added R11: 120, rcl:R0805
- moved R6 7.41 mm to (81.3, 66.0), turned to 270 degrees
- moved C3 6.35 mm to (101.6, 43.2)
- moved RESET 5.39 mm to (78.7, 73.7)
- moved C1 2.54 mm to (85.1, 69.8)
- moved C16 1.27 mm to (90.2, 38.1)
- moved C17 1.27 mm to (86.4, 38.1)
- moved R5 1.27 mm to (91.4, 69.8)
Connections:
- removed net LO_PWR: IC1.17, TP1.TP
- new net DERE: IC1.17, IC3.5, IC3.6, TP1.TP
- new net N$11: IC3.14, JP1.2, R11.2
- new net N$8: IC3.11, JP1.3, R11.1
- net RC0: now also IC3.7
- net RC1: now also IC3.4
- net VDD: now also C18.1, C19.1, IC3.2, IC3.3, JP1.5
- net VSS: now also C18.2, C19.2, IC3.1, IC3.10, IC3.12, IC3.13, IC3.15, IC3.16, IC3.8, IC3.9, JP1.1, JP1.4
Routing:
- net DERE: track 0.00 -> 61.6 mm, vias 0 -> 2
- net RC1: track 30.7 -> 73.2 mm, vias 1 -> 3
- net RC0: track 29.9 -> 64.8 mm, vias 0 -> 3
- net N$8: track 0.00 -> 30.8 mm, vias 0 -> 1
- net DB0: track 61.3 -> 34.4 mm
- net N$11: track 0.00 -> 25.1 mm
- net LO_PWR: track 21.4 -> 0.00 mm
- net SCK1: track 30.8 -> 50.7 mm, vias 2 -> 0
- net AN2: track 69.7 -> 51.9 mm, vias 2 -> 1
- net UC_RX: track 95.6 -> 109.9 mm
- net SDI1: track 56.6 -> 43.4 mm
- net CS: track 52.8 -> 41.1 mm, vias 3 -> 1
- net AN1: track 64.4 -> 53.6 mm
- net VREF: track 79.9 -> 70.2 mm, vias 1 -> 0
- net UC_TX: track 101.5 -> 91.9 mm
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Other:
- board size 64.8 x 55.5 mm -> 64.8 x 59.4 mm

Commit message: up
Parts:
- renumbered JP1 to MODBUS, SV1 to ANALOG, SV2 to DIGITAL, X1 to MATE
Connections:
- net N$11 renamed MB_B
- net N$8 renamed MB_A
- net RC0 renamed MB_RX
- net RC1 renamed MB_TX
Other:
- board size 64.8 x 59.4 mm -> 64.8 x 61.9 mm

Commit message: up
Parts:
- removed IC1: PIC18F47Q84-E_P, PIC18F47Q84-E_P:DIP1543W58P254L5175H635Q40N
- added IC4: PIC18F47Q84-I_PT, PIC18F47Q84-I_PT:QFP80P1200X1200X120-44N
- moved OS1_10MHZ 20.7 mm to (109.2, 26.7)
- moved IC3 7.73 mm to (99.1, 64.8)
- moved C18 7.62 mm to (99.1, 57.1)
- moved C19 7.62 mm to (99.1, 54.6)
- moved ZENER 7.62 mm to (108.0, 41.9)
- moved R11 7.41 mm to (100.3, 73.7)
- moved U1 6.35 mm to (95.2, 25.4)
- moved VREF_PWR 6.35 mm to (87.6, 25.4)
- moved C2 5.68 mm to (100.3, 25.4)
- flipped U2 to the bottom
Connections:
- net AN0: now also IC4.19; no longer IC1.2
- net AN1: now also IC4.20; no longer IC1.3
- net AN2: now also IC4.21; no longer IC1.4
- net AN3: now also IC4.23; no longer IC1.6
- net AN4: now also IC4.24; no longer IC1.7
- net CANRX: now also IC4.8; no longer IC1.33
- net CANTX: now also IC4.14; no longer IC1.37
- net CLOCKO: now also IC4.31; no longer IC1.14
- net CPU_CLK: now also IC4.30; no longer IC1.13
- net CS: now also IC4.41; no longer IC1.22
- net DB0: now also IC4.39; no longer IC1.20
- net DB1: now also IC4.40; no longer IC1.21
- net DERE: now also IC4.36; no longer IC1.17
- net DLED: now also IC4.11, IC4.2; no longer IC1.27, IC1.36
- net MB_RX: now also IC4.32; no longer IC1.15
- net MB_TX: now also IC4.35; no longer IC1.16
- net MCLR_SIG: now also IC4.18; no longer IC1.1
- net MISC: now also IC4.26; no longer IC1.9
- net MLED: now also IC4.9; no longer IC1.34
- net PC_RX2: now also IC4.38; no longer IC1.19
- net PC_TX2: now also IC4.4; no longer IC1.29
- net PGC: now also IC4.16; no longer IC1.39
- net PGD: now also IC4.17; no longer IC1.40
- net RB5: now also IC4.15; no longer IC1.38
- net RD5: now also IC4.3; no longer IC1.28
- net RD7: now also IC4.5; no longer IC1.30
- net RE2: now also IC4.27; no longer IC1.10
- net RELAY: now also IC4.25; no longer IC1.8
- net RLED: now also IC4.10; no longer IC1.35
- net SCK1: now also IC4.37; no longer IC1.18
- net SDI1: now also IC4.42; no longer IC1.23
- net SDO1: now also IC4.43; no longer IC1.24
- net UC_RX: now also IC4.1; no longer IC1.26
- net UC_TX: now also IC4.44; no longer IC1.25
- net VDD: now also IC4.28, IC4.7; no longer IC1.11, IC1.32
- net VREF: now also IC4.22; no longer IC1.5
- net VSS: now also IC4.29, IC4.6; no longer IC1.12, IC1.31
Routing:
- net CANTX: track 5.49 -> 37.4 mm, vias 0 -> 1
- net RD7: track 50.3 -> 24.2 mm, vias 1 -> 0
- net SDO1: track 46.8 -> 24.0 mm, vias 3 -> 0
- net MCLR_SIG: track 39.5 -> 61.3 mm, vias 0 -> 2
- net SDI1: track 43.4 -> 22.4 mm
- net SCK1: track 50.7 -> 30.0 mm, vias 0 -> 1
- net PC_RX2: track 39.6 -> 58.5 mm, vias 1 -> 0
- net RELAY: track 19.2 -> 38.0 mm, vias 0 -> 1
- net DERE: track 61.6 -> 80.3 mm
- net UC_TX: track 91.9 -> 74.8 mm
- net RD5: track 29.0 -> 13.5 mm
- net RE2: track 7.56 -> 22.9 mm, vias 0 -> 1
- net PGD: track 53.4 -> 38.3 mm, vias 0 -> 1
- net CANRX: track 13.3 -> 28.4 mm, vias 0 -> 2
- net AN1: track 53.6 -> 38.6 mm
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Other:
- board text added: "Outback FM interface 1.2"
- board text removed: "Outback FM interface 1.1"

Commit message: up
Parts:
- added EXT_IO: EXT_IO, con-lstb:MA06-1
- added R_RESET: remote_reset, pinhead:1X02
- moved CANBUS 4.02 mm to (124.5, 73.7)
- moved IC2 1.27 mm to (115.6, 31.8)
- moved RESET 1.27 mm to (80.0, 73.7)
- moved 24VDC_PWR 1.27 mm to (119.4, 21.6)
Connections:
- removed net N$2: C1.1, R5.1, R6.1, RESET.1
- new net R_RESET: C1.1, R5.1, R6.1, RESET.1, R_RESET.2
- net PGC: now also EXT_IO.5
- net PGD: now also EXT_IO.6
- net RB5: now also EXT_IO.4
- net RD5: now also EXT_IO.2
- net RD7: now also EXT_IO.3
- net VSS: now also EXT_IO.1, R_RESET.1
Routing:
- net R_RESET: track 0.00 -> 52.2 mm, vias 0 -> 1
- net PGD: track 38.3 -> 75.7 mm
- net PGC: track 40.6 -> 67.0 mm, vias 0 -> 1
- net SCK1: track 30.0 -> 53.3 mm, vias 1 -> 0
- net VDD: track 249.7 -> 271.7 mm, vias 4 -> 2
- net RD5: track 13.5 -> 35.0 mm
- net N$2: track 20.9 -> 0.00 mm, vias 1 -> 0
- net MISC: track 22.2 -> 42.9 mm, vias 1 -> 0
- net PC_RX2: track 58.5 -> 38.0 mm, vias 0 -> 1
- net RB5: track 32.0 -> 48.6 mm
- net RELAY: track 38.0 -> 23.7 mm, vias 1 -> 0
- net RD7: track 24.2 -> 36.6 mm, vias 0 -> 2
- net DB1: track 30.5 -> 42.2 mm
- net UC_TX: track 74.8 -> 63.2 mm
- net UC_RX: track 107.4 -> 116.2 mm
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
Commit message: up
Parts:
- added R12: 0 ohm fuse, rcl:R1206
- added TP2: PTR1PAD1-13, testpad:P1-13
Connections:
- new net N$2: C14.1, C15.1, IC2.1, R12.1
- net CPU_CLK: now also TP2.TP
- net V+: now also R12.2; no longer C14.1, C15.1, IC2.1
Routing:
- net RLED: track 21.6 -> 85.0 mm, vias 2 -> 0
- net UC_RX: track 116.2 -> 87.3 mm
- net SCK1: track 53.3 -> 26.5 mm, vias 0 -> 1
- net N$2: track 0.00 -> 20.5 mm
- net RE2: track 22.9 -> 42.7 mm
- net MISC: track 42.9 -> 24.0 mm, vias 0 -> 1
- net DB1: track 42.2 -> 25.1 mm
- net PGC: track 67.0 -> 82.5 mm
- net VDD: track 271.7 -> 256.8 mm, vias 2 -> 3
- net RD7: track 36.6 -> 51.5 mm, vias 2 -> 0
- net V+: track 17.8 -> 3.76 mm
- net PC_RX2: track 38.0 -> 47.8 mm, vias 1 -> 0
- net DERE: track 73.4 -> 64.0 mm
- net RB5: track 48.6 -> 41.7 mm
- net CLOCKO: track 32.0 -> 38.1 mm
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- added copper zone on layer 1, net VSS

Commit message: up
Connections:
- removed net AN3: ANALOG.4, IC4.23
- new net AN5: ANALOG.5, IC4.24
- net AN4: now also ANALOG.4, IC4.23; no longer ANALOG.5, IC4.24
Routing:
- net AN5: track 0.00 -> 40.2 mm, vias 0 -> 1
- net AN3: track 38.0 -> 0.00 mm, vias 1 -> 0
- net AN4: track 40.2 -> 38.0 mm
Changed lines of the file:
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@@
 <via x="119.8626" y="60.96" extent="1-16" drill="0.35"/>
 </signal>
-<signal name="AN3">
+<signal name="AN4">
 <contactref element="ANALOG" pad="4"/>
 <contactref element="IC4" pad="23"/>
@@
 <via x="111.5568" y="38.3286" extent="1-16" drill="0.35"/>
 </signal>
-<signal name="AN4">
+<signal name="AN5">
 <contactref element="ANALOG" pad="5"/>
 <contactref element="IC4" pad="24"/>
