File: isoamp.sch (EAGLE design)
At the start: 13 parts, among them IC1 AD210JN, IC2 7815T, X2 PS-in, X3 PS-out

Commit message: up
Parts:
- added 24VDC_PWR: 22-23-2021, con-molex:22-23-2021
- added JP3: isoV+, pinhead:PINHD-1X1
- added JP4: iosV-, pinhead:PINHD-1X1
- added R3: 6200 ohm, rcl:R-US_M1206
- added SENSE_PWR_ON: pwr_led, led:LEDCHIPLED_1206
- added SJ1: GND_SHORT, jumper:SJW
- added TP1, TP2, TP3, TP4, TP5, TP6, TP7: TPPAD1-13, testpad:TPPAD1-13
- R1: value (none) -> 5100 ohm
- R2: value (none) -> 160000 ohm
Connections:
- new net 0V: IC1.PWR_COM, JP4.1, SJ1.2
- new net N$6: R3.2, SENSE_PWR_ON.A
- net +15V: now also JP3.1, TP3.TP
- net +24V: now also 24VDC_PWR-1.S, TP4.TP
- net 0-5VOUT: now also TP1.TP
- net GND: now also 24VDC_PWR-2.S, SJ1.1, TP2.TP, TP7.TP; no longer IC1.PWR_COM
- net N$1: now also SENSE_PWR_ON.C
- net N$3: now also R3.1
- net PV-NEG: now also TP6.TP
- net PV-SCALE: now also TP5.TP
