File: mate_a.sch (EAGLE design)
At the start: 8 parts, among them IC1 PIC18F47Q84-E_P, X1 GLX-S-88M

Commit message: up
Parts:
- added OS1_10MHZ: OSC-OE-CFPS-72, IQD-Frequency-Products:OSC-OE-CFPS-72
- added U1: REF3440IDBVR, REF3440IDBVR:REF3440IDBVR
Connections:
- new net CPU_CLK: IC1.RA7, OS1_10MHZ.OUT
- new net VREF: IC1.RA3, U1.OUT_F, U1.OUT_S
- net VDD: now also OS1_10MHZ.CON, OS1_10MHZ.VDD, U1.IN
- net VSS: now also OS1_10MHZ.VSS, U1.ENABLE, U1.GND_F, U1.GND_S
Changed lines of the file:
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@@
 <part name="X1" library="con-kycon" library_urn="urn:adsk.eagle:library:157" deviceset="GLX-S-88M" device="" package3d_urn="urn:adsk.eagle:package:7680/1"/>
 <part name="GND3" library="supply1" library_urn="urn:adsk.eagle:library:371" deviceset="0V" device=""/>
+<part name="OS1_10MHZ" library="IQD-Frequency-Products" library_urn="urn:adsk.eagle:library:90" deviceset="OSC-OE" device="-CFPS-72" package3d_urn="urn:adsk.eagle:package:3365/1"/>
+<part name="U1" library="REF3440IDBVR" deviceset="REF3440IDBVR" device=""/>
+<part name="VDD2" library="supply1" library_urn="urn:adsk.eagle:library:371" deviceset="VDD" device=""/>
+<part name="VSS3" library="supply1" library_urn="urn:adsk.eagle:library:371" deviceset="VSS" device=""/>
+<part name="VDD3" library="supply1" library_urn="urn:adsk.eagle:library:371" deviceset="VDD" device=""/>
+<part name="VSS4" library="supply1" library_urn="urn:adsk.eagle:library:371" deviceset="VSS" device=""/>
+<part name="VDD4" library="supply1" library_urn="urn:adsk.eagle:library:371" deviceset="VDD" device=""/>
+<part name="VSS5" library="supply1" library_urn="urn:adsk.eagle:library:371" deviceset="VSS" device=""/>
 </parts>
 <sheets>
@@
 <attribute name="VALUE" x="-29.845" y="-17.78" size="1.778" layer="96"/>
 </instance>
+<instance part="OS1_10MHZ" gate="A" x="134.62" y="-27.94" smashed="yes">
+<attribute name="NAME" x="127" y="-19.685" size="1.778" layer="95"/>
+<attribute name="VALUE" x="127" y="-38.1" size="1.778" layer="96"/>
+</instance>
+<instance part="U1" gate="G$1" x="137.16" y="7.62" smashed="yes">
+<attribute name="NAME" x="124.46" y="16.24" size="2.0828" layer="95" ratio="10" rot="SR0"/>
+<attribute name="VALUE" x="124.46" y="-4" size="2.0828" layer="96" ratio="10" rot="SR0"/>
+</instance>
+<instance part="VDD2" gate="G$1" x="119.38" y="7.62" smashed="yes" rot="R180">
+<attribute name="VALUE" x="116.84" y="2.54" size="1.778" layer="96"/>
+</instance>
+<instance part="VSS3" gate="G$1" x="119.38" y="15.24" smashed="yes" rot="R180">
+<attribute name="VALUE" x="116.84" y="20.32" size="1.778" layer="96"/>
+</instance>
+<instance part="VDD3" gate="G$1" x="121.92" y="-20.32" smashed="yes">
+<attribute name="VALUE" x="124.46" y="-15.24" size="1.778" layer="96" rot="R180"/>
+</instance>
+<instance part="VSS4" gate="G$1" x="121.92" y="-35.56" smashed="yes">
+<attribute name="VALUE" x="124.46" y="-40.64" size="1.778" layer="96" rot="R180"/>
+</instance>
+<instance part="VDD4" gate="G$1" x="147.32" y="-20.32" smashed="yes">
+<attribute name="VALUE" x="149.86" y="-15.24" size="1.778" layer="96" rot="R180"/>
+</instance>
+<instance part="VSS5" gate="G$1" x="154.94" y="-5.08" smashed="yes">
+<attribute name="VALUE" x="157.48" y="-10.16" size="1.778" layer="96" rot="R180"/>
+</instance>
 </instances>
 <busses>
@@
 <label x="25.4" y="40.64" size="1.778" layer="95"/>
 <junction x="-7.62" y="40.64"/>
+</segment>
+<segment>
+<pinref part="U1" gate="G$1" pin="IN"/>
+<pinref part="VDD2" gate="G$1" pin="VDD"/>
+<junction x="119.38" y="10.16"/>
+</segment>
+<segment>
+<pinref part="OS1_10MHZ" gate="A" pin="VDD"/>
+<pinref part="VDD3" gate="G$1" pin="VDD"/>
+<junction x="121.92" y="-22.86"/>
+</segment>
+<segment>
+<pinref part="OS1_10MHZ" gate="A" pin="CON"/>
+<pinref part="VDD4" gate="G$1" pin="VDD"/>
+<junction x="147.32" y="-22.86"/>
 </segment>
 </net>
@@
 <junction x="-7.62" y="38.1"/>
 </segment>
+<segment>
+<pinref part="U1" gate="G$1" pin="ENABLE"/>
+<pinref part="VSS3" gate="G$1" pin="VSS"/>
+<junction x="119.38" y="12.7"/>
+</segment>
+<segment>
+<pinref part="OS1_10MHZ" gate="A" pin="VSS"/>
+<pinref part="VSS4" gate="G$1" pin="VSS"/>
+<junction x="121.92" y="-33.02"/>
+</segment>
+<segment>
+<pinref part="U1" gate="G$1" pin="GND_F"/>
+<wire x1="154.94" y1="5.08" x2="154.94" y2="2.54" width="0.1524" layer="91"/>
+<pinref part="U1" gate="G$1" pin="GND_S"/>
+<wire x1="154.94" y1="2.54" x2="154.94" y2="-2.54" width="0.1524" layer="91"/>
+<junction x="154.94" y="2.54"/>
+<junction x="154.94" y="5.08"/>
+<pinref part="VSS5" gate="G$1" pin="VSS"/>
+<junction x="154.94" y="-2.54"/>
+</segment>
+</net>
+<net name="CPU_CLK" class="0">
+<segment>
+<pinref part="OS1_10MHZ" gate="A" pin="OUT"/>
+<wire x1="147.32" y1="-27.94" x2="157.48" y2="-27.94" width="0.1524" layer="91"/>
+<label x="149.86" y="-33.02" size="1.778" layer="95"/>
+<junction x="147.32" y="-27.94"/>
+<junction x="157.48" y="-27.94"/>
+</segment>
+<segment>
+<wire x1="27.94" y1="35.56" x2="38.1" y2="35.56" width="0.1524" layer="91"/>
+<pinref part="IC1" gate="G$1" pin="RA7"/>
+<junction x="38.1" y="35.56"/>
+<junction x="27.94" y="35.56"/>
+<label x="15.24" y="35.56" size="1.778" layer="95"/>
+</segment>
+</net>
+<net name="VREF" class="0">
+<segment>
+<wire x1="38.1" y1="55.88" x2="-7.62" y2="55.88" width="0.1524" layer="91"/>
+<pinref part="IC1" gate="G$1" pin="RA3"/>
+<junction x="38.1" y="55.88"/>
+<junction x="-7.62" y="55.88"/>
+<label x="-10.16" y="58.42" size="1.778" layer="95"/>
+</segment>
+<segment>
+<pinref part="U1" gate="G$1" pin="OUT_S"/>
+<wire x1="154.94" y1="10.16" x2="154.94" y2="12.7" width="0.1524" layer="91"/>
+<pinref part="U1" gate="G$1" pin="OUT_F"/>
+<wire x1="154.94" y1="12.7" x2="154.94" y2="17.78" width="0.1524" layer="91"/>
+<junction x="154.94" y="12.7"/>
+<junction x="154.94" y="17.78"/>
+<junction x="154.94" y="10.16"/>
+<label x="157.48" y="15.24" size="1.778" layer="95"/>
+</segment>
 </net>
 </nets>
 </sheet>
 </sheets>
+<errors>
+</errors>
 </schematic>
 </drawing>

Commit message: up
Parts:
- added C1, C2, C3, C5: 0.1uf, rcl:C-USC0805
- added C4, C6: 10uf, rcl:C-USC0805
- added ICSP: ICSP, con-lstb:MA06-1
- added R5: 56ohm, rcl:R-US_R0805
- added R6: 10k, rcl:R-US_R0805
- added SV1: Analog, con-lstb:MA10-1
- added SV2: Digtal, con-lstb:MA10-1
Connections:
- new net AN0: IC1.RA0, SV1.1
- new net AN1: IC1.RA1, SV1.2
- new net AN2: IC1.RA2, SV1.3
- new net MCLR_SIG: IC1.!MCLR!/VPP/RE3, ICSP.1, R5.2
- new net N$2: C1.1, R5.1, R6.1
- new net PGC: IC1.RB6/ICSPCLK, ICSP.5
- new net PGD: IC1.RB7/ICSPDAT, ICSP.4
- new net RD0: IC1.RD0, SV2.1
- new net RD1: IC1.RD1, SV2.2
- new net RD2: IC1.RD2, SV2.3
- new net RD3: IC1.RD3, SV2.4
- net VDD: now also C2.1, C3.1, C4.1, C5.1, C6.1, ICSP.2, R6.2, SV1.10, SV2.10
- net VSS: now also C1.2, C2.2, C3.2, C4.2, C5.2, C6.2, ICSP.3, SV1.9, SV2.9

Commit message: up
Parts:
- added C10, C13, C15, C8: 10uf, rcl:C-USC0805
- added C11, C12, C14, C7, C9: 0.1uf, rcl:C-USC0805
- added CANBUS: CANBUS, con-lstb:MA04-1
- added CAN_PWR: CAN_PWR, jumper:SJ
- added IC2: 7805TV, linear:7805TV
- added LED1: run, led:LEDCHIPLED_0805
- added LED2: error, led:LEDCHIPLED_0805
- added LED3: comm, led:LEDCHIPLED_0805
- added MISC_IO: misc-io, con-lstb:MA10-1
- added R7, R8, R9: 1k, rcl:R-US_R0805
- added RESET: reset, jumper:SJ
- added TP1: PTR1PAD1-13, testpad:PTR1PAD1-13
- added TTL_SERIAL: TTL Serial, con-lstb:MA04-1
- added U2: TCAN330GDR, TCAN330GDR:TCAN330GDR
- added X2: 22-23-2021, con-molex:22-23-2021
- R1, R2: value (none) -> 1.5k
- R3: value (none) -> 330ohm
- R4: value (none) -> 220ohm
Connections:
- removed net RD0: IC1.RD0, SV2.1
- new net AN3: IC1.RA4, SV1.4
- new net AN4: IC1.RA5, SV1.5
- new net CANRX: IC1.RB0, U2.RXD
- new net CANTX: IC1.RB4, U2.TXD
- new net CAN_N: CANBUS.1, U2.CANL
- new net CAN_P: CANBUS.3, U2.CANH
- new net CAN_VCC: C7.1, C8.1, CANBUS.4, CAN_PWR.1, U2.VCC
- new net CLOCKO: IC1.RA6, MISC_IO.10
- new net LED1: IC1.RB1, R7.2
- new net LED2: IC1.RB2, R8.2
- new net LED3: IC1.RB3, R9.2
- new net LO_PWR: IC1.RC2, TP1.TP
- new net N$4: LED1.A, R7.1
- new net N$5: LED2.A, R8.1
- new net N$6: LED3.A, R9.1
- new net RB5: IC1.RB5, MISC_IO.6
- new net RC0: IC1.RC0, SV1.6
- new net RC1: IC1.RC1, SV1.7
- new net RD4: IC1.RD4, MISC_IO.4
- new net RD5: IC1.RD5, MISC_IO.5
- new net RD7: IC1.RD7, MISC_IO.7
- new net RE0: IC1.RE0, MISC_IO.1
- new net RE1: IC1.RE1, MISC_IO.2
- new net RE2: IC1.RE2, MISC_IO.3
- new net RX2: IC1.RD0, SV2.8
- new net SCK1: IC1.RC3, SV2.4
- new net SDI1: IC1.RC4, SV2.5
- new net SDO1: IC1.RC5, SV2.6
- new net TX2: IC1.RD6, SV2.7
- new net V+: C14.1, C15.1, IC2.VI, X2-1.S
- net MCLR_SIG: now also MISC_IO.8
- net N$2: now also RESET.1
- net PC_RX: now also TTL_SERIAL.3
- net PC_TX: now also TTL_SERIAL.2
- net RD1: now also SV2.1; no longer SV2.2
- net RD2: now also SV2.2; no longer SV2.3
- net RD3: now also SV2.3; no longer SV2.4
- net VDD: now also C10.1, C11.1, C12.1, C13.1, C9.1, CAN_PWR.2, IC2.VO
- net VREF: now also SV1.8
- net VSS: now also C10.2, C11.2, C12.2, C13.2, C14.2, C15.2, C7.2, C8.2, C9.2, CANBUS.2, IC2.GND, LED1.C, LED2.C, LED3.C, MISC_IO.9, RESET.2, TTL_SERIAL.1, U2.GND, U2.S, U2.SHDN, X2-2.S

Commit message: up
Parts:
- added C16: 0.1uf, rcl:C-USC0805
- added C17: 10uf, rcl:C-USC0805
Connections:
- net VDD: now also TTL_SERIAL.4
- net VREF: now also C16.1, C17.1
- net VSS: now also C16.2, C17.2
Changed lines of the file:
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@@
 <part name="RESET" library="jumper" library_urn="urn:adsk.eagle:library:252" deviceset="SJ" device="" package3d_urn="urn:adsk.eagle:package:15471/1" value="reset"/>
 <part name="VSS31" library="supply1" library_urn="urn:adsk.eagle:library:371" deviceset="VSS" device=""/>
+<part name="VDD9" library="supply1" library_urn="urn:adsk.eagle:library:371" deviceset="VDD" device=""/>
+<part name="C16" library="rcl" library_urn="urn:adsk.eagle:library:334" deviceset="C-US" device="C0805" package3d_urn="urn:adsk.eagle:package:23617/2" value="0.1uf"/>
+<part name="C17" library="rcl" library_urn="urn:adsk.eagle:library:334" deviceset="C-US" device="C0805" package3d_urn="urn:adsk.eagle:package:23617/2" value="10uf"/>
+<part name="VSS32" library="supply1" library_urn="urn:adsk.eagle:library:371" deviceset="VSS" device=""/>
+<part name="VSS33" library="supply1" library_urn="urn:adsk.eagle:library:371" deviceset="VSS" device=""/>
 </parts>
 <sheets>
@@
 <instance part="VSS31" gate="G$1" x="0" y="78.74" smashed="yes">
 <attribute name="VALUE" x="2.54" y="73.66" size="1.778" layer="96" rot="R180"/>
+</instance>
+<instance part="VDD9" gate="G$1" x="170.18" y="86.36" smashed="yes">
+<attribute name="VALUE" x="172.72" y="91.44" size="1.778" layer="96" rot="R180"/>
+</instance>
+<instance part="C16" gate="G$1" x="165.1" y="10.16" smashed="yes">
+<attribute name="NAME" x="166.116" y="10.795" size="1.778" layer="95"/>
+<attribute name="VALUE" x="166.116" y="5.969" size="1.778" layer="96"/>
+</instance>
+<instance part="C17" gate="G$1" x="175.26" y="10.16" smashed="yes">
+<attribute name="NAME" x="176.276" y="10.795" size="1.778" layer="95"/>
+<attribute name="VALUE" x="176.276" y="5.969" size="1.778" layer="96"/>
+</instance>
+<instance part="VSS32" gate="G$1" x="165.1" y="2.54" smashed="yes">
+<attribute name="VALUE" x="167.64" y="-2.54" size="1.778" layer="96" rot="R180"/>
+</instance>
+<instance part="VSS33" gate="G$1" x="175.26" y="2.54" smashed="yes">
+<attribute name="VALUE" x="177.8" y="-2.54" size="1.778" layer="96" rot="R180"/>
 </instance>
 </instances>
@@
 <junction x="-40.64" y="-20.32"/>
 </segment>
+<segment>
+<pinref part="TTL_SERIAL" gate="1" pin="4"/>
+<pinref part="VDD9" gate="G$1" pin="VDD"/>
+<junction x="170.18" y="83.82"/>
+</segment>
 </net>
 <net name="+24V" class="1">
@@
 <junction x="0" y="81.28"/>
 </segment>
+<segment>
+<pinref part="C16" gate="G$1" pin="2"/>
+<pinref part="VSS32" gate="G$1" pin="VSS"/>
+<junction x="165.1" y="5.08"/>
+</segment>
+<segment>
+<pinref part="C17" gate="G$1" pin="2"/>
+<pinref part="VSS33" gate="G$1" pin="VSS"/>
+<junction x="175.26" y="5.08"/>
+</segment>
 </net>
 <net name="CPU_CLK" class="0">
@@
 <junction x="154.94" y="10.16"/>
 <label x="157.48" y="15.24" size="1.778" layer="95"/>
-</segment>
-<segment>
+<pinref part="C17" gate="G$1" pin="1"/>
+<wire x1="154.94" y1="12.7" x2="165.1" y2="12.7" width="0.1524" layer="91"/>
+<pinref part="C16" gate="G$1" pin="1"/>
+<wire x1="165.1" y1="12.7" x2="175.26" y2="12.7" width="0.1524" layer="91"/>
+<junction x="165.1" y="12.7"/>
+<junction x="175.26" y="12.7"/>
+</segment>
+<segment>

Commit message: up
Parts:
- added R10: 120ohm, rcl:R-US_R0805
- R1, R2: value 1.5k -> 2.2k
- R3: value 330ohm -> 1k
- R4: value 220ohm -> 470ohm
Connections:
- net CAN_N: now also R10.1
- net CAN_P: now also R10.2
- net PC_RX: now also SV2.8; no longer TTL_SERIAL.3
- net PC_TX: now also SV2.7; no longer TTL_SERIAL.2
- net RX2: now also TTL_SERIAL.3; no longer SV2.8
- net TX2: now also TTL_SERIAL.2; no longer SV2.7
Changed lines of the file:
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@@
 <part name="OK1" library="optocoupler" library_urn="urn:adsk.eagle:library:320" deviceset="4N*?M" device="S" package3d_urn="urn:adsk.eagle:package:21970/1" technology="25"/>
 <part name="OK2" library="optocoupler" library_urn="urn:adsk.eagle:library:320" deviceset="4N*?M" device="S" package3d_urn="urn:adsk.eagle:package:21970/1" technology="25"/>
-<part name="R1" library="rcl" library_urn="urn:adsk.eagle:library:334" deviceset="R-US_" device="R0805" package3d_urn="urn:adsk.eagle:package:23553/2" value="1.5k"/>
-<part name="R2" library="rcl" library_urn="urn:adsk.eagle:library:334" deviceset="R-US_" device="R0805" package3d_urn="urn:adsk.eagle:package:23553/2" value="1.5k"/>
-<part name="R3" library="rcl" library_urn="urn:adsk.eagle:library:334" deviceset="R-US_" device="R0805" package3d_urn="urn:adsk.eagle:package:23553/2" value="330ohm"/>
-<part name="R4" library="rcl" library_urn="urn:adsk.eagle:library:334" deviceset="R-US_" device="R0805" package3d_urn="urn:adsk.eagle:package:23553/2" value="220ohm"/>
+<part name="R1" library="rcl" library_urn="urn:adsk.eagle:library:334" deviceset="R-US_" device="R0805" package3d_urn="urn:adsk.eagle:package:23553/2" value="2.2k"/>
+<part name="R2" library="rcl" library_urn="urn:adsk.eagle:library:334" deviceset="R-US_" device="R0805" package3d_urn="urn:adsk.eagle:package:23553/2" value="2.2k"/>
+<part name="R3" library="rcl" library_urn="urn:adsk.eagle:library:334" deviceset="R-US_" device="R0805" package3d_urn="urn:adsk.eagle:package:23553/2" value="1k"/>
+<part name="R4" library="rcl" library_urn="urn:adsk.eagle:library:334" deviceset="R-US_" device="R0805" package3d_urn="urn:adsk.eagle:package:23553/2" value="470ohm"/>
 <part name="P+1" library="supply1" library_urn="urn:adsk.eagle:library:371" deviceset="+24V" device=""/>
 <part name="GND1" library="supply1" library_urn="urn:adsk.eagle:library:371" deviceset="0V" device=""/>
@@
 <part name="VSS32" library="supply1" library_urn="urn:adsk.eagle:library:371" deviceset="VSS" device=""/>
 <part name="VSS33" library="supply1" library_urn="urn:adsk.eagle:library:371" deviceset="VSS" device=""/>
+<part name="R10" library="rcl" library_urn="urn:adsk.eagle:library:334" deviceset="R-US_" device="R0805" package3d_urn="urn:adsk.eagle:package:23553/2" value="120ohm"/>
 </parts>
 <sheets>
@@
 </instance>
 <instance part="VSS12" gate="G$1" x="-38.1" y="20.32" smashed="yes" rot="R90">
-<attribute name="VALUE" x="-33.02" y="22.86" size="1.778" layer="96" rot="R270"/>
+<attribute name="VALUE" x="-35.56" y="20.32" size="1.778" layer="96"/>
 </instance>
 <instance part="VDD7" gate="G$1" x="-38.1" y="22.86" smashed="yes" rot="R270">
-<attribute name="VALUE" x="-33.02" y="20.32" size="1.778" layer="96" rot="R90"/>
+<attribute name="VALUE" x="-30.48" y="25.4" size="1.778" layer="96" rot="R180"/>
 </instance>
 <instance part="CANBUS" gate="1" x="-48.26" y="-33.02" smashed="yes">
@@
 <instance part="VSS33" gate="G$1" x="175.26" y="2.54" smashed="yes">
 <attribute name="VALUE" x="177.8" y="-2.54" size="1.778" layer="96" rot="R180"/>
+</instance>
+<instance part="R10" gate="G$1" x="198.12" y="43.18" smashed="yes" rot="R90">
+<attribute name="NAME" x="196.6214" y="39.37" size="1.778" layer="95" rot="R90"/>
+<attribute name="VALUE" x="201.422" y="39.37" size="1.778" layer="96" rot="R90"/>
 </instance>
 </instances>
@@
 </segment>
 <segment>
-<wire x1="170.18" y1="81.28" x2="195.58" y2="81.28" width="0.1524" layer="91"/>
-<pinref part="TTL_SERIAL" gate="1" pin="3"/>
-<junction x="170.18" y="81.28"/>
-<junction x="195.58" y="81.28"/>
-<label x="185.42" y="81.28" size="1.778" layer="95"/>
+<wire x1="-40.64" y1="17.78" x2="-27.94" y2="17.78" width="0.1524" layer="91"/>
+<pinref part="SV2" gate="1" pin="8"/>
+<junction x="-40.64" y="17.78"/>
+<junction x="-27.94" y="17.78"/>
+<label x="-35.56" y="17.78" size="1.778" layer="95"/>
 </segment>
 </net>
@@
 </segment>
 <segment>
-<wire x1="170.18" y1="78.74" x2="195.58" y2="78.74" width="0.1524" layer="91"/>
-<pinref part="TTL_SERIAL" gate="1" pin="2"/>
-<junction x="170.18" y="78.74"/>
-<junction x="195.58" y="78.74"/>
-<label x="185.42" y="78.74" size="1.778" layer="95"/>
+<wire x1="-40.64" y1="15.24" x2="-27.94" y2="15.24" width="0.1524" layer="91"/>
+<pinref part="SV2" gate="1" pin="7"/>
+<junction x="-40.64" y="15.24"/>
+<junction x="-27.94" y="15.24"/>
+<label x="-35.56" y="15.24" size="1.778" layer="95"/>
 </segment>
 </net>
@@
 </segment>
 <segment>
-<wire x1="-27.94" y1="17.78" x2="-40.64" y2="17.78" width="0.1524" layer="91"/>
-<pinref part="SV2" gate="1" pin="8"/>
-<junction x="-40.64" y="17.78"/>
-<junction x="-27.94" y="17.78"/>
-<label x="-35.56" y="17.78" size="1.778" layer="95"/>
+<wire x1="182.88" y1="81.28" x2="170.18" y2="81.28" width="0.1524" layer="91"/>
+<pinref part="TTL_SERIAL" gate="1" pin="3"/>
+<junction x="170.18" y="81.28"/>
+<junction x="182.88" y="81.28"/>
+<label x="175.26" y="81.28" size="1.778" layer="95"/>
 </segment>
 </net>
@@
 </segment>
 <segment>
-<wire x1="-40.64" y1="15.24" x2="-27.94" y2="15.24" width="0.1524" layer="91"/>
-<pinref part="SV2" gate="1" pin="7"/>
-<junction x="-40.64" y="15.24"/>
-<junction x="-27.94" y="15.24"/>
-<label x="-35.56" y="15.24" size="1.778" layer="95"/>
-</segment>
-</net>
-<net name="CAN_N" class="0">
+<wire x1="170.18" y1="78.74" x2="182.88" y2="78.74" width="0.1524" layer="91"/>
+<pinref part="TTL_SERIAL" gate="1" pin="2"/>
+<junction x="170.18" y="78.74"/>
+<junction x="182.88" y="78.74"/>
+<label x="175.26" y="78.74" size="1.778" layer="95"/>
+</segment>
+</net>
+<net name="CAN_N" class="1">
 <segment>
 <pinref part="U2" gate="G$1" pin="CANL"/>
@@
 <junction x="180.34" y="43.18"/>
 <junction x="193.04" y="43.18"/>
+<wire x1="193.04" y1="43.18" x2="193.04" y2="38.1" width="0.1524" layer="91"/>
+<pinref part="R10" gate="G$1" pin="1"/>
+<wire x1="193.04" y1="38.1" x2="198.12" y2="38.1" width="0.1524" layer="91"/>
+<junction x="198.12" y="38.1"/>
 </segment>
 <segment>
@@
 </segment>
 </net>
-<net name="CAN_P" class="0">
+<net name="CAN_P" class="1">
 <segment>
 <pinref part="U2" gate="G$1" pin="CANH"/>
@@
 <junction x="180.34" y="45.72"/>
 <junction x="193.04" y="45.72"/>
-</segment>
-<segment>
+<wire x1="193.04" y1="45.72" x2="193.04" y2="48.26" width="0.1524" layer="91"/>
+<pinref part="R10" gate="G$1" pin="2"/>
+<wire x1="193.04" y1="48.26" x2="198.12" y2="48.26" width="0.1524" layer="91"/>
+<junction x="198.12" y="48.26"/>
+</segment>
+<segment>

Commit message: up
Parts:
- added VREF_PWR: 5vdc_vref_pwr, con-molex:22-23-2021
- added ZENER: 5.6V, diode:ZENER-DIODESMB
- 24VDC_PWR: value 22-23-2021 -> 24vdc power
- renumbered X2 to 24VDC_PWR
Connections:
- net RX2 renamed PC_RX2
- net TX2 renamed PC_TX2
- removed net PC_RX: IC1.RC7, OK1.EMI, R3.1, SV2.8
- removed net PC_TX: IC1.RC6, OK2.A, SV2.7
- net AN0: now also SV1.10; no longer SV1.1
- net AN1: now also SV1.1; no longer SV1.2
- net AN2: now also SV1.2; no longer SV1.3
- net MX_RX: now also IC1.RC7, OK1.EMI, R3.1, SV2.10
- net MX_TX: now also IC1.RC6, OK2.A, SV2.7
- net VDD: now also SV1.8, SV2.8, ZENER.C; no longer SV1.10, SV2.10
- net VREF: now also SV1.3, VREF_PWR-1.S; no longer SV1.8
- net VSS: now also VREF_PWR-2.S, ZENER.A

Commit message: up
Connections:
- net LED1 renamed MLED
- net LED2 renamed RLED
- net LED3 renamed DLED
- net RD1 renamed DB0
- net RD2 renamed DB1
- net RD3 renamed CS
- net RE0 renamed RELAY
- net RE1 renamed MISC
Changed lines of the file:
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@@
 </segment>
 </net>
-<net name="RD1" class="0">
+<net name="DB0" class="0">
 <segment>
 <pinref part="IC1" gate="G$1" pin="RD1"/>
@@
 </segment>
 </net>
-<net name="RD2" class="0">
+<net name="DB1" class="0">
 <segment>
 <pinref part="IC1" gate="G$1" pin="RD2"/>
@@
 </segment>
 </net>
-<net name="RD3" class="0">
+<net name="CS" class="0">
 <segment>
 <pinref part="IC1" gate="G$1" pin="RD3"/>
@@
 </segment>
 </net>
-<net name="RE0" class="0">
+<net name="RELAY" class="0">
 <segment>
 <pinref part="IC1" gate="G$1" pin="RE0"/>
@@
 </segment>
 </net>
-<net name="RE1" class="0">
+<net name="MISC" class="0">
 <segment>
 <pinref part="IC1" gate="G$1" pin="RE1"/>
@@
 </segment>
 </net>
-<net name="LED1" class="0">
+<net name="MLED" class="0">
 <segment>
 <pinref part="IC1" gate="G$1" pin="RB1"/>
@@
 </segment>
 </net>
-<net name="LED2" class="0">
+<net name="RLED" class="0">
 <segment>
 <pinref part="IC1" gate="G$1" pin="RB2"/>
@@
 </segment>
 </net>
-<net name="LED3" class="0">
+<net name="DLED" class="0">
 <segment>
 <pinref part="IC1" gate="G$1" pin="RB3"/>
