File: mate_a.sch (EAGLE design)
At the start: 50 parts, among them IC1 PIC18F47Q84-E_P, IC2 7805TV, U1 REF3440IDBVR, U2 TCAN330GDR, X1 GLX-S-88M

Commit message: up
Connections:
- removed net RD4: IC1.RD4, MISC_IO.4
- new net UC_RX: IC1.RC7, OK1.EMI, R3.1, SV2.10
- new net UC_TX: IC1.RC6, OK2.A, SV2.7
- net DLED: now also IC1.RD4, MISC_IO.4
- net MX_RX: no longer IC1.RC7, OK1.EMI, R3.1, SV2.10
- net MX_TX: no longer IC1.RC6, OK2.A, SV2.7
Changed lines of the file:
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@@
 <label x="-2.54" y="-22.86" size="1.778" layer="95"/>
-</segment>
-<segment>
-<pinref part="OK1" gate="G$1" pin="EMI"/>
-<pinref part="R3" gate="G$1" pin="1"/>
-<wire x1="76.2" y1="-7.62" x2="76.2" y2="-15.24" width="0.1524" layer="91"/>
-<junction x="76.2" y="-7.62"/>
-<wire x1="76.2" y1="-15.24" x2="99.06" y2="-15.24" width="0.1524" layer="91"/>
-<label x="91.44" y="-15.24" size="1.778" layer="95"/>
-<junction x="99.06" y="-15.24"/>
-</segment>
-<segment>
-<wire x1="86.36" y1="30.48" x2="111.76" y2="30.48" width="0.1524" layer="91"/>
-<pinref part="IC1" gate="G$1" pin="RC7"/>
-<junction x="86.36" y="30.48"/>
-<label x="93.98" y="30.48" size="1.778" layer="95"/>
-<junction x="111.76" y="30.48"/>
-</segment>
-<segment>
-<wire x1="-40.64" y1="22.86" x2="-27.94" y2="22.86" width="0.1524" layer="91"/>
-<pinref part="SV2" gate="1" pin="10"/>
-<label x="-35.56" y="22.86" size="1.778" layer="95"/>
-<junction x="-40.64" y="22.86"/>
-<junction x="-27.94" y="22.86"/>
 </segment>
 </net>
@@
 <junction x="-22.86" y="-15.24"/>
 <label x="-20.32" y="-15.24" size="1.778" layer="95"/>
-</segment>
-<segment>
-<pinref part="OK2" gate="G$1" pin="A"/>
-<wire x1="58.42" y1="-25.4" x2="58.42" y2="-20.32" width="0.1524" layer="91"/>
-<wire x1="58.42" y1="-20.32" x2="99.06" y2="-20.32" width="0.1524" layer="91"/>
-<label x="91.44" y="-22.86" size="1.778" layer="95"/>
-<junction x="58.42" y="-25.4"/>
-<junction x="99.06" y="-20.32"/>
-</segment>
-<segment>
-<wire x1="86.36" y1="27.94" x2="111.76" y2="27.94" width="0.1524" layer="91"/>
-<pinref part="IC1" gate="G$1" pin="RC6"/>
-<junction x="86.36" y="27.94"/>
-<label x="93.98" y="27.94" size="1.778" layer="95"/>
-<junction x="111.76" y="27.94"/>
-</segment>
-<segment>
-<wire x1="-40.64" y1="15.24" x2="-27.94" y2="15.24" width="0.1524" layer="91"/>
-<pinref part="SV2" gate="1" pin="7"/>
-<junction x="-40.64" y="15.24"/>
-<junction x="-27.94" y="15.24"/>
-<label x="-35.56" y="15.24" size="1.778" layer="95"/>
 </segment>
 </net>
@@
 </segment>
 </net>
-<net name="RD4" class="0">
-<segment>
-<pinref part="IC1" gate="G$1" pin="RD4"/>
-<wire x1="86.36" y1="33.02" x2="111.76" y2="33.02" width="0.1524" layer="91"/>
-<junction x="86.36" y="33.02"/>
-<junction x="111.76" y="33.02"/>
-<label x="93.98" y="33.02" size="1.778" layer="95"/>
-</segment>
-<segment>
-<wire x1="-7.62" y1="7.62" x2="17.78" y2="7.62" width="0.1524" layer="91"/>
-<pinref part="MISC_IO" gate="1" pin="4"/>
-<junction x="-7.62" y="7.62"/>
-<junction x="17.78" y="7.62"/>
-<label x="5.08" y="7.62" size="1.778" layer="95"/>
-</segment>
-</net>
 <net name="RD5" class="0">
 <segment>
@@
 <junction x="109.22" y="60.96"/>
 <label x="99.06" y="60.96" size="1.778" layer="95"/>
+<junction x="86.36" y="60.96"/>
 </segment>
 <segment>
@@
 <segment>
 <pinref part="IC1" gate="G$1" pin="RB3"/>
-<wire x1="86.36" y1="55.88" x2="111.76" y2="55.88" width="0.1524" layer="91"/>
+<wire x1="86.36" y1="55.88" x2="99.06" y2="55.88" width="0.1524" layer="91"/>
 <junction x="86.36" y="55.88"/>
 <junction x="111.76" y="55.88"/>
 <label x="101.6" y="55.88" size="1.778" layer="95"/>
+<junction x="99.06" y="55.88"/>
+<wire x1="99.06" y1="55.88" x2="111.76" y2="55.88" width="0.1524" layer="91"/>
 </segment>
 <segment>
@@
 <label x="144.78" y="76.2" size="1.778" layer="95"/>
 </segment>
-</net>
+<segment>
+<wire x1="-7.62" y1="7.62" x2="17.78" y2="7.62" width="0.1524" layer="91"/>
+<pinref part="MISC_IO" gate="1" pin="4"/>
+<junction x="-7.62" y="7.62"/>
+<junction x="17.78" y="7.62"/>
+<label x="5.08" y="7.62" size="1.778" layer="95"/>
+</segment>
+<segment>
+<pinref part="IC1" gate="G$1" pin="RD4"/>
+<wire x1="86.36" y1="33.02" x2="111.76" y2="33.02" width="0.1524" layer="91"/>
+<junction x="86.36" y="33.02"/>
+<junction x="111.76" y="33.02"/>
+<label x="93.98" y="33.02" size="1.778" layer="95"/>
+</segment>
+</net>
+<net name="UC_TX" class="0">
+<segment>
+<pinref part="OK2" gate="G$1" pin="A"/>
+<wire x1="58.42" y1="-25.4" x2="58.42" y2="-20.32" width="0.1524" layer="91"/>
+<wire x1="58.42" y1="-20.32" x2="99.06" y2="-20.32" width="0.1524" layer="91"/>
+<label x="91.44" y="-22.86" size="1.778" layer="95"/>
+<junction x="58.42" y="-25.4"/>
+<junction x="99.06" y="-20.32"/>
+</segment>
+<segment>
+<wire x1="86.36" y1="27.94" x2="111.76" y2="27.94" width="0.1524" layer="91"/>
+<pinref part="IC1" gate="G$1" pin="RC6"/>
+<junction x="86.36" y="27.94"/>
+<label x="93.98" y="27.94" size="1.778" layer="95"/>
+<junction x="111.76" y="27.94"/>
+</segment>
+<segment>
+<wire x1="-40.64" y1="15.24" x2="-27.94" y2="15.24" width="0.1524" layer="91"/>
+<pinref part="SV2" gate="1" pin="7"/>
+<junction x="-40.64" y="15.24"/>
+<junction x="-27.94" y="15.24"/>
+<label x="-35.56" y="15.24" size="1.778" layer="95"/>
+</segment>
+</net>
+<net name="UC_RX" class="0">
+<segment>
+<pinref part="OK1" gate="G$1" pin="EMI"/>
+<pinref part="R3" gate="G$1" pin="1"/>
+<wire x1="76.2" y1="-7.62" x2="76.2" y2="-15.24" width="0.1524" layer="91"/>
+<junction x="76.2" y="-7.62"/>
+<wire x1="76.2" y1="-15.24" x2="99.06" y2="-15.24" width="0.1524" layer="91"/>
+<label x="91.44" y="-15.24" size="1.778" layer="95"/>
+<junction x="99.06" y="-15.24"/>
+</segment>
+<segment>
+<wire x1="86.36" y1="30.48" x2="111.76" y2="30.48" width="0.1524" layer="91"/>
+<pinref part="IC1" gate="G$1" pin="RC7"/>
+<junction x="86.36" y="30.48"/>
+<label x="93.98" y="30.48" size="1.778" layer="95"/>
+<junction x="111.76" y="30.48"/>
+</segment>
+<segment>
+<wire x1="-40.64" y1="22.86" x2="-27.94" y2="22.86" width="0.1524" layer="91"/>
+<pinref part="SV2" gate="1" pin="10"/>
+<label x="-35.56" y="22.86" size="1.778" layer="95"/>
+<junction x="-40.64" y="22.86"/>
+<junction x="-27.94" y="22.86"/>
+</segment>
+</net>
