File: mate_a.sch (EAGLE design)
At the start: 50 parts, among them IC1 PIC18F47Q84-E_P, IC2 7805TV, U1 REF3440IDBVR, U2 TCAN330GDR, X1 GLX-S-88M

Commit message: up
Parts:
- added C18: 0.1uf, rcl:C-USC0805
- added C19: 10uf, rcl:C-USC0805
- added IC3: ADM3095EBRZ, ADM3095EBRZ:ADM3095EBRZ
- added JP1: MODBUS, pinhead:PINHD-1X5
- added R11: 120, rcl:R-US_R0805
Connections:
- removed net LO_PWR: IC1.RC2, TP1.TP
- new net DERE: IC1.RC2, IC3.!RE, IC3.DE, TP1.TP
- new net N$11: IC3.B, JP1.2, R11.2
- new net N$8: IC3.A, JP1.3, R11.1
- net RC0: now also IC3.RXD
- net RC1: now also IC3.TXD
- net VDD: now also C18.1, C19.1, IC3.VCC, IC3.VIO, JP1.5
- net VSS: now also C18.2, C19.2, IC3.GND_1, IC3.GND_2, IC3.GND_3, IC3.GND_4, IC3.GND_5, IC3.GND_6, IC3.GND_7, IC3.GND_8, JP1.1, JP1.4

Commit message: up
Parts:
- renumbered JP1 to MODBUS, SV1 to ANALOG, SV2 to DIGITAL, X1 to MATE
Connections:
- net N$11 renamed MB_B
- net N$8 renamed MB_A
- net RC0 renamed MB_RX
- net RC1 renamed MB_TX

Commit message: up
Parts:
- removed IC1: PIC18F47Q84-E_P, PIC18F47Q84-E_P:PIC18F47Q84-E_P
- added IC4: PIC18F47Q84-I_PT, PIC18F47Q84-I_PT:PIC18F47Q84-I_PT
Connections:
- net AN0: now also IC4.RA0; no longer IC1.RA0
- net AN1: now also IC4.RA1; no longer IC1.RA1
- net AN2: now also IC4.RA2; no longer IC1.RA2
- net AN3: now also IC4.RA4; no longer IC1.RA4
- net AN4: now also IC4.RA5; no longer IC1.RA5
- net CANRX: now also IC4.RB0; no longer IC1.RB0
- net CANTX: now also IC4.RB4; no longer IC1.RB4
- net CLOCKO: now also IC4.RA6; no longer IC1.RA6
- net CPU_CLK: now also IC4.RA7; no longer IC1.RA7
- net CS: now also IC4.RD3; no longer IC1.RD3
- net DB0: now also IC4.RD1; no longer IC1.RD1
- net DB1: now also IC4.RD2; no longer IC1.RD2
- net DERE: now also IC4.RC2; no longer IC1.RC2
- net DLED: now also IC4.RB3, IC4.RD4; no longer IC1.RB3, IC1.RD4
- net MB_RX: now also IC4.RC0; no longer IC1.RC0
- net MB_TX: now also IC4.RC1; no longer IC1.RC1
- net MCLR_SIG: now also IC4.VPP/!MCLR!/RE3; no longer IC1.!MCLR!/VPP/RE3
- net MISC: now also IC4.RE1; no longer IC1.RE1
- net MLED: now also IC4.RB1; no longer IC1.RB1
- net PC_RX2: now also IC4.RD0; no longer IC1.RD0
- net PC_TX2: now also IC4.RD6; no longer IC1.RD6
- net PGC: now also IC4.ICSPCLK/RB6; no longer IC1.RB6/ICSPCLK
- net PGD: now also IC4.ICSPDAT/RB7; no longer IC1.RB7/ICSPDAT
- net RB5: now also IC4.RB5; no longer IC1.RB5
- net RD5: now also IC4.RD5; no longer IC1.RD5
- net RD7: now also IC4.RD7; no longer IC1.RD7
- net RE2: now also IC4.RE2; no longer IC1.RE2
- net RELAY: now also IC4.RE0; no longer IC1.RE0
- net RLED: now also IC4.RB2; no longer IC1.RB2
- net SCK1: now also IC4.RC3; no longer IC1.RC3
- net SDI1: now also IC4.RC4; no longer IC1.RC4
- net SDO1: now also IC4.RC5; no longer IC1.RC5
- net UC_RX: now also IC4.RC7; no longer IC1.RC7
- net UC_TX: now also IC4.RC6; no longer IC1.RC6
- net VDD: now also IC4.VDD_1, IC4.VDD_2; no longer IC1.VDD_1, IC1.VDD_2
- net VREF: now also IC4.RA3; no longer IC1.RA3
- net VSS: now also IC4.VSS_1, IC4.VSS_2; no longer IC1.VSS_1, IC1.VSS_2

Commit message: up
Parts:
- added EXT_IO: EXT_IO, con-lstb:MA06-1
- added R_RESET: remote_reset, pinhead:PINHD-1X2
Connections:
- removed net N$2: C1.1, R5.1, R6.1, RESET.1
- new net R_RESET: C1.1, R5.1, R6.1, RESET.1, R_RESET.2
- net PGC: now also EXT_IO.5
- net PGD: now also EXT_IO.6
- net RB5: now also EXT_IO.4
- net RD5: now also EXT_IO.2
- net RD7: now also EXT_IO.3
- net VSS: now also EXT_IO.1, R_RESET.1
Changed lines of the file:
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@@
 <part name="VSS42" library="supply1" library_urn="urn:adsk.eagle:library:371" deviceset="VSS" device=""/>
 <part name="IC4" library="PIC18F47Q84-I_PT" deviceset="PIC18F47Q84-I_PT" device=""/>
+<part name="R_RESET" library="pinhead" library_urn="urn:adsk.eagle:library:325" deviceset="PINHD-1X2" device="" package3d_urn="urn:adsk.eagle:package:22435/2" value="remote_reset"/>
+<part name="EXT_IO" library="con-lstb" library_urn="urn:adsk.eagle:library:162" deviceset="MA06-1" device="" package3d_urn="urn:adsk.eagle:package:8340/1" value="EXT_IO"/>
+<part name="VSS43" library="supply1" library_urn="urn:adsk.eagle:library:371" deviceset="VSS" device=""/>
 </parts>
 <sheets>
@@
 <attribute name="NAME" x="229.87" y="12.7" size="1.778" layer="95" align="center-left"/>
 <attribute name="VALUE" x="229.87" y="10.16" size="1.778" layer="96" align="center-left"/>
+</instance>
+<instance part="R_RESET" gate="G$1" x="-33.02" y="78.74" smashed="yes" rot="R180">
+<attribute name="NAME" x="-26.67" y="73.025" size="1.778" layer="95" rot="R180"/>
+<attribute name="VALUE" x="-36.83" y="78.74" size="1.778" layer="96" rot="R180"/>
+</instance>
+<instance part="EXT_IO" gate="1" x="215.9" y="48.26" smashed="yes">
+<attribute name="VALUE" x="214.63" y="35.56" size="1.778" layer="96"/>
+<attribute name="NAME" x="214.63" y="56.642" size="1.778" layer="95"/>
+</instance>
+<instance part="VSS43" gate="G$1" x="223.52" y="38.1" smashed="yes">
+<attribute name="VALUE" x="231.14" y="40.64" size="1.778" layer="96" rot="R180"/>
 </instance>
 </instances>
@@
 <pinref part="VSS31" gate="G$1" pin="VSS"/>
 <junction x="0" y="81.28"/>
+<pinref part="R_RESET" gate="G$1" pin="1"/>
+<wire x1="-30.48" y1="76.2" x2="-7.62" y2="76.2" width="0.1524" layer="91"/>
+<wire x1="-7.62" y1="76.2" x2="-7.62" y2="81.28" width="0.1524" layer="91"/>
+<wire x1="-7.62" y1="81.28" x2="0" y2="81.28" width="0.1524" layer="91"/>
+<junction x="-30.48" y="76.2"/>
+<label x="-22.86" y="73.66" size="1.778" layer="95"/>
 </segment>
 <segment>
@@
 <label x="236.22" y="-12.7" size="1.778" layer="95"/>
 </segment>
+<segment>
+<pinref part="EXT_IO" gate="1" pin="1"/>
+<pinref part="VSS43" gate="G$1" pin="VSS"/>
+<junction x="223.52" y="40.64"/>
+</segment>
 </net>
 <net name="CPU_CLK" class="0">
@@
 <label x="213.36" y="-66.04" size="1.778" layer="95" rot="R90"/>
 </segment>
+<segment>
+<wire x1="236.22" y1="53.34" x2="223.52" y2="53.34" width="0.1524" layer="91"/>
+<pinref part="EXT_IO" gate="1" pin="6"/>
+<junction x="223.52" y="53.34"/>
+<junction x="236.22" y="53.34"/>
+<label x="226.06" y="53.34" size="1.778" layer="95"/>
+</segment>
 </net>
 <net name="PGC" class="0">
@@
 <label x="210.82" y="-66.04" size="1.778" layer="95" rot="R90"/>
 </segment>
-</net>
-<net name="N$2" class="0">
+<segment>
+<wire x1="236.22" y1="50.8" x2="223.52" y2="50.8" width="0.1524" layer="91"/>
+<pinref part="EXT_IO" gate="1" pin="5"/>
+<junction x="223.52" y="50.8"/>
+<junction x="236.22" y="50.8"/>
+<label x="226.06" y="50.8" size="1.778" layer="95"/>
+</segment>
+</net>
+<net name="R_RESET" class="0">
 <segment>
 <pinref part="R5" gate="G$1" pin="1"/>
@@
 <junction x="15.24" y="66.04"/>
 <pinref part="RESET" gate="1" pin="1"/>
+<label x="15.24" y="71.12" size="1.778" layer="95"/>
+</segment>
+<segment>
+<wire x1="-17.78" y1="78.74" x2="-30.48" y2="78.74" width="0.1524" layer="91"/>
+<pinref part="R_RESET" gate="G$1" pin="2"/>
+<junction x="-17.78" y="78.74"/>
+<junction x="-30.48" y="78.74"/>
+<label x="-22.86" y="81.28" size="1.778" layer="95"/>
 </segment>
 </net>
@@
 <label x="182.88" y="-7.62" size="1.778" layer="95"/>
 </segment>
+<segment>
+<wire x1="223.52" y1="43.18" x2="236.22" y2="43.18" width="0.1524" layer="91"/>
+<pinref part="EXT_IO" gate="1" pin="2"/>
+<junction x="223.52" y="43.18"/>
+<junction x="236.22" y="43.18"/>
+<label x="226.06" y="43.18" size="1.778" layer="95"/>
+</segment>
 </net>
 <net name="RD7" class="0">
@@
 <label x="182.88" y="-12.7" size="1.778" layer="95"/>
 </segment>
+<segment>
+<wire x1="223.52" y1="45.72" x2="236.22" y2="45.72" width="0.1524" layer="91"/>
+<pinref part="EXT_IO" gate="1" pin="3"/>
+<junction x="223.52" y="45.72"/>
+<junction x="236.22" y="45.72"/>
+<label x="226.06" y="45.72" size="1.778" layer="95"/>
+</segment>
 </net>
 <net name="RB5" class="0">
@@
 <label x="208.28" y="-66.04" size="1.778" layer="95" rot="R90"/>
 </segment>
-</net>
+<segment>
+<wire x1="236.22" y1="48.26" x2="223.52" y2="48.26" width="0.1524" layer="91"/>
+<pinref part="EXT_IO" gate="1" pin="4"/>
+<junction x="223.52" y="48.26"/>
+<junction x="236.22" y="48.26"/>
+<label x="226.06" y="48.26" size="1.778" layer="95"/>
+</segment>
+</net>

Commit message: up
Parts:
- added R12: 0 ohm fuse, rcl:R-US_R1206
- added TP2: PTR1PAD1-13, testpad:PTR1PAD1-13
Connections:
- new net N$2: C14.1, C15.1, IC2.VI, R12.1
- net CPU_CLK: now also TP2.TP
- net V+: now also R12.2; no longer C14.1, C15.1, IC2.VI
Changed lines of the file:
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@@
 <part name="MISC_IO" library="con-lstb" library_urn="urn:adsk.eagle:library:162" deviceset="MA10-1" device="" package3d_urn="urn:adsk.eagle:package:8346/1" value="misc-io"/>
 <part name="VSS26" library="supply1" library_urn="urn:adsk.eagle:library:371" deviceset="VSS" device=""/>
-<part name="SUPPLY1" library="supply2" library_urn="urn:adsk.eagle:library:372" deviceset="V+" device=""/>
 <part name="24VDC_PWR" library="con-molex" library_urn="urn:adsk.eagle:library:165" deviceset="22-23-2021" device="" package3d_urn="urn:adsk.eagle:package:8078633/1" value="24vdc power"/>
 <part name="SUPPLY2" library="supply2" library_urn="urn:adsk.eagle:library:372" deviceset="V+" device=""/>
@@
 <part name="EXT_IO" library="con-lstb" library_urn="urn:adsk.eagle:library:162" deviceset="MA06-1" device="" package3d_urn="urn:adsk.eagle:package:8340/1" value="EXT_IO"/>
 <part name="VSS43" library="supply1" library_urn="urn:adsk.eagle:library:371" deviceset="VSS" device=""/>
+<part name="TP2" library="testpad" library_urn="urn:adsk.eagle:library:385" deviceset="PTR1" device="PAD1-13" package3d_urn="urn:adsk.eagle:package:27946/1"/>
+<part name="R12" library="rcl" library_urn="urn:adsk.eagle:library:334" deviceset="R-US_" device="R1206" package3d_urn="urn:adsk.eagle:package:23540/2" value="0 ohm fuse"/>
+<part name="SUPPLY3" library="supply2" library_urn="urn:adsk.eagle:library:372" deviceset="V+" device=""/>
 </parts>
 <sheets>
@@
 <attribute name="VALUE" x="0" y="22.86" size="1.778" layer="96" rot="R270"/>
 </instance>
-<instance part="SUPPLY1" gate="1" x="-15.24" y="-40.64" smashed="yes">
-<attribute name="VALUE" x="-16.51" y="-39.37" size="1.778" layer="96"/>
-</instance>
 <instance part="24VDC_PWR" gate="-1" x="-35.56" y="-50.8" smashed="yes">
 <attribute name="NAME" x="-33.02" y="-51.562" size="1.524" layer="95"/>
@@
 <instance part="VSS43" gate="G$1" x="223.52" y="38.1" smashed="yes">
 <attribute name="VALUE" x="231.14" y="40.64" size="1.778" layer="96" rot="R180"/>
+</instance>
+<instance part="TP2" gate="G$1" x="157.48" y="-25.4" smashed="yes" rot="R180">
+<attribute name="NAME" x="158.496" y="-19.05" size="1.778" layer="95" rot="R270"/>
+<attribute name="TP_SIGNAL_NAME" x="156.21" y="-22.86" size="1.778" layer="97" rot="R180"/>
+</instance>
+<instance part="R12" gate="G$1" x="-10.16" y="-38.1" smashed="yes" rot="R90">
+<attribute name="NAME" x="-11.6586" y="-41.91" size="1.778" layer="95" rot="R90"/>
+<attribute name="VALUE" x="-6.858" y="-41.91" size="1.778" layer="96" rot="R90"/>
+</instance>
+<instance part="SUPPLY3" gate="1" x="-10.16" y="-30.48" smashed="yes">
+<attribute name="VALUE" x="-11.43" y="-29.21" size="1.778" layer="96"/>
 </instance>
 </instances>
@@
 <junction x="147.32" y="-27.94"/>
 <junction x="157.48" y="-27.94"/>
+<pinref part="TP2" gate="G$1" pin="TP"/>
 </segment>
 <segment>
@@
 <net name="V+" class="1">
 <segment>
-<pinref part="IC2" gate="A1" pin="VI"/>
-<wire x1="2.54" y1="-43.18" x2="0" y2="-43.18" width="0.1524" layer="91"/>
-<junction x="2.54" y="-43.18"/>
-<pinref part="C14" gate="G$1" pin="1"/>
-<junction x="0" y="-43.18"/>
-<wire x1="0" y1="-43.18" x2="-10.16" y2="-43.18" width="0.1524" layer="91"/>
-<pinref part="C15" gate="G$1" pin="1"/>
-<junction x="-10.16" y="-43.18"/>
-<wire x1="-10.16" y1="-43.18" x2="-15.24" y2="-43.18" width="0.1524" layer="91"/>
-<pinref part="SUPPLY1" gate="1" pin="V+"/>
-<junction x="-15.24" y="-43.18"/>
-</segment>
-<segment>
 <pinref part="24VDC_PWR" gate="-1" pin="S"/>
 <pinref part="SUPPLY2" gate="1" pin="V+"/>
 <junction x="-38.1" y="-50.8"/>
+</segment>
+<segment>
+<pinref part="R12" gate="G$1" pin="2"/>
+<pinref part="SUPPLY3" gate="1" pin="V+"/>
 </segment>
 </net>
@@
 </segment>
 </net>
+<net name="N$2" class="1">
+<segment>
+<pinref part="IC2" gate="A1" pin="VI"/>
+<wire x1="2.54" y1="-43.18" x2="0" y2="-43.18" width="0.1524" layer="91"/>
+<junction x="2.54" y="-43.18"/>
+<pinref part="C14" gate="G$1" pin="1"/>
+<junction x="0" y="-43.18"/>
+<wire x1="0" y1="-43.18" x2="-10.16" y2="-43.18" width="0.1524" layer="91"/>
+<pinref part="C15" gate="G$1" pin="1"/>
+<junction x="-10.16" y="-43.18"/>
+<pinref part="R12" gate="G$1" pin="1"/>
+</segment>
+</net>

Commit message: up
Connections:
- removed net AN3: ANALOG.4, IC4.RA4
- new net AN5: ANALOG.5, IC4.RA5
- net AN4: now also ANALOG.4, IC4.RA4; no longer ANALOG.5, IC4.RA5
Changed lines of the file:
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@@
 </segment>
 </net>
-<net name="AN3" class="0">
+<net name="AN4" class="0">
 <segment>
 <wire x1="38.1" y1="53.34" x2="25.4" y2="53.34" width="0.1524" layer="91"/>
@@
 </segment>
 </net>
-<net name="AN4" class="0">
+<net name="AN5" class="0">
 <segment>
 <wire x1="38.1" y1="50.8" x2="25.4" y2="50.8" width="0.1524" layer="91"/>
